File: Teensy36_I2S_Proto/wildly_teensy_proto.sch (EAGLE design)
At the start: 22 parts, among them CON1 MIKROE_BUS_CONN, SW1 SPST_TACT-KMR2, X1 ANTENNA

Commit message: Add files via upload
Connections:
- new net 3V: JP3.1, U$1.3V3
- new net BCLK: JP3.3, U$1.9/PWM/RX2/CS0-1
- new net CTS_OF_GSM: U$1.33/A14/CAN1TX/TX5/ALT-SCL0
- new net DOUT: JP3.4, U$1.13/LED/ALT-PWM/SCK0
- new net GND: JP3.2, U$1.GND
- new net LRCLK: JP3.5, U$1.23/A9/PWM/T
- new net RESET_GSM: U$1.20/A6/PWM/CS0-2/ALT-SCK1
- new net RTS_OF_GSM: U$1.34/A15/CAN1RX/RX5/ALT-SDA0
- new net RX_OF_GSM: U$1.1/TX1/MISO1/T
- new net TX_OF_GSM: U$1.0/RX1/MOSI1/T
Other:
- moved on the sheet: JP3, SW2
Changed lines of the file:
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@@
 <?xml version="1.0" encoding="utf-8"?>
 <!DOCTYPE eagle SYSTEM "eagle.dtd">
-<eagle version="9.3.0">
+<eagle version="9.2.2">
 <drawing>
 <settings>
@@
 <setting verticaltext="up"/>
 </settings>
-<grid distance="0.1" unitdist="inch" unit="inch" style="lines" multiple="1" display="no" altdistance="0.01" altunitdist="inch" altunit="inch"/>
+<grid distance="0.1" unitdist="inch" unit="inch" style="dots" multiple="1" display="yes" altdistance="0.01" altunitdist="inch" altunit="inch"/>
 <layers>
 <layer number="1" name="Top" color="4" fill="1" visible="no" active="no"/>
@@
 <sheet>
 <plain>
-<text x="58.42" y="-25.4" size="1.778" layer="91">Microphone In</text>
+<text x="71.12" y="-27.94" size="1.778" layer="91">Microphone In</text>
 <text x="55.88" y="106.68" size="1.778" layer="91">5V Boost 500mA</text>
 <text x="129.54" y="10.16" size="1.778" layer="91">5V Boost 1A</text>
@@
 <attribute name="VALUE" x="-0.635" y="92.71" size="1.778" layer="96" rot="R180"/>
 </instance>
-<instance part="SW2" gate="G$1" x="15.24" y="78.74" smashed="yes">
-<attribute name="NAME" x="12.7" y="82.296" size="1.27" layer="95"/>
-<attribute name="VALUE" x="12.7" y="76.454" size="1.27" layer="96"/>
+<instance part="SW2" gate="G$1" x="2.54" y="78.74" smashed="yes">
+<attribute name="NAME" x="-2.54" y="82.296" size="1.27" layer="95"/>
+<attribute name="VALUE" x="0" y="76.454" size="1.27" layer="96"/>
 </instance>
 <instance part="JP2" gate="G$1" x="137.16" y="15.24" smashed="yes" rot="R270">
@@
 <attribute name="VALUE" x="121.92" y="21.59" size="1.778" layer="96" rot="R270"/>
 </instance>
-<instance part="JP3" gate="A" x="66.04" y="-15.24" smashed="yes" rot="R90">
-<attribute name="NAME" x="55.245" y="-21.59" size="1.778" layer="95" rot="R90"/>
-<attribute name="VALUE" x="76.2" y="-21.59" size="1.778" layer="96" rot="R90"/>
+<instance part="JP3" gate="A" x="66.04" y="-17.78" smashed="yes" rot="R90">
+<attribute name="NAME" x="55.245" y="-24.13" size="1.778" layer="95" rot="R90"/>
+<attribute name="VALUE" x="76.2" y="-24.13" size="1.778" layer="96" rot="R90"/>
 </instance>
 <instance part="R8" gate="G$1" x="10.16" y="17.78" smashed="yes">
@@
 </segment>
 </net>
+<net name="3V" class="0">
+<segment>
+<pinref part="JP3" gate="A" pin="1"/>
+<wire x1="58.42" y1="-20.32" x2="58.42" y2="-27.94" width="0.1524" layer="91"/>
+<wire x1="58.42" y1="-27.94" x2="22.86" y2="-27.94" width="0.1524" layer="91"/>
+<wire x1="22.86" y1="-27.94" x2="22.86" y2="91.44" width="0.1524" layer="91"/>
+<pinref part="U$1" gate="G$1" pin="3V3"/>
+<wire x1="22.86" y1="91.44" x2="30.48" y2="91.44" width="0.1524" layer="91"/>
+<label x="58.42" y="-15.24" size="1.778" layer="95" rot="R90"/>
+</segment>
+</net>
+<net name="GND" class="0">
+<segment>
+<pinref part="JP3" gate="A" pin="2"/>
+<wire x1="60.96" y1="-20.32" x2="60.96" y2="-30.48" width="0.1524" layer="91"/>
+<wire x1="60.96" y1="-30.48" x2="25.4" y2="-30.48" width="0.1524" layer="91"/>
+<wire x1="25.4" y1="-30.48" x2="25.4" y2="88.9" width="0.1524" layer="91"/>
+<pinref part="U$1" gate="G$1" pin="GND"/>
+<wire x1="25.4" y1="88.9" x2="30.48" y2="88.9" width="0.1524" layer="91"/>
+<label x="60.96" y="-15.24" size="1.778" layer="95" rot="R90"/>
+</segment>
+</net>
+<net name="BCLK" class="0">
+<segment>
+<pinref part="JP3" gate="A" pin="3"/>
+<wire x1="63.5" y1="-20.32" x2="63.5" y2="-33.02" width="0.1524" layer="91"/>
+<wire x1="63.5" y1="-33.02" x2="27.94" y2="-33.02" width="0.1524" layer="91"/>
+<pinref part="U$1" gate="G$1" pin="9/PWM/RX2/CS0-1"/>
+<wire x1="27.94" y1="-33.02" x2="27.94" y2="63.5" width="0.1524" layer="91"/>
+<wire x1="27.94" y1="63.5" x2="30.48" y2="63.5" width="0.1524" layer="91"/>
+<label x="63.5" y="-15.24" size="1.778" layer="95" rot="R90"/>
+</segment>
+</net>
+<net name="DOUT" class="0">
+<segment>
+<pinref part="JP3" gate="A" pin="4"/>
+<wire x1="66.04" y1="-20.32" x2="66.04" y2="-35.56" width="0.1524" layer="91"/>
+<wire x1="66.04" y1="-35.56" x2="20.32" y2="-35.56" width="0.1524" layer="91"/>
+<pinref part="U$1" gate="G$1" pin="13/LED/ALT-PWM/SCK0"/>
+<wire x1="20.32" y1="-35.56" x2="20.32" y2="53.34" width="0.1524" layer="91"/>
+<wire x1="20.32" y1="53.34" x2="30.48" y2="53.34" width="0.1524" layer="91"/>
+<label x="66.04" y="-15.24" size="1.778" layer="95" rot="R90"/>
+</segment>
+</net>
+<net name="LRCLK" class="0">
+<segment>
+<pinref part="JP3" gate="A" pin="5"/>
+<wire x1="68.58" y1="-20.32" x2="68.58" y2="-38.1" width="0.1524" layer="91"/>
+<wire x1="68.58" y1="-38.1" x2="17.78" y2="-38.1" width="0.1524" layer="91"/>
+<wire x1="17.78" y1="-38.1" x2="17.78" y2="27.94" width="0.1524" layer="91"/>
+<label x="68.58" y="-15.24" size="1.778" layer="95" rot="R90"/>
+<pinref part="U$1" gate="G$1" pin="23/A9/PWM/T"/>
+<wire x1="17.78" y1="27.94" x2="30.48" y2="27.94" width="0.1524" layer="91"/>
+</segment>
+</net>
+<net name="TX_OF_GSM" class="0">
+<segment>
+<pinref part="U$1" gate="G$1" pin="0/RX1/MOSI1/T"/>
+<wire x1="30.48" y1="86.36" x2="20.32" y2="86.36" width="0.1524" layer="91"/>
+<wire x1="20.32" y1="86.36" x2="20.32" y2="96.52" width="0.1524" layer="91"/>
+<label x="22.86" y="96.52" size="1.778" layer="95" rot="R90"/>
+</segment>
+</net>
+<net name="RX_OF_GSM" class="0">
+<segment>
+<pinref part="U$1" gate="G$1" pin="1/TX1/MISO1/T"/>
+<wire x1="30.48" y1="83.82" x2="17.78" y2="83.82" width="0.1524" layer="91"/>
+<wire x1="17.78" y1="83.82" x2="17.78" y2="96.52" width="0.1524" layer="91"/>
+<label x="17.78" y="96.52" size="1.778" layer="95" rot="R90"/>
+</segment>
+</net>
+<net name="RESET_GSM" class="0">
+<segment>
+<pinref part="U$1" gate="G$1" pin="20/A6/PWM/CS0-2/ALT-SCK1"/>
+<wire x1="30.48" y1="35.56" x2="-12.7" y2="35.56" width="0.1524" layer="91"/>
+<label x="-15.24" y="35.56" size="1.778" layer="95"/>
+</segment>
+</net>
+<net name="CTS_OF_GSM" class="0">
+<segment>
+<pinref part="U$1" gate="G$1" pin="33/A14/CAN1TX/TX5/ALT-SCL0"/>
+<wire x1="30.48" y1="2.54" x2="7.62" y2="2.54" width="0.1524" layer="91"/>
+<label x="5.08" y="2.54" size="1.778" layer="95"/>
+</segment>
+</net>
+<net name="RTS_OF_GSM" class="0">
+<segment>
+<pinref part="U$1" gate="G$1" pin="34/A15/CAN1RX/RX5/ALT-SDA0"/>
+<wire x1="30.48" y1="0" x2="7.62" y2="0" width="0.1524" layer="91"/>
+<label x="5.08" y="0" size="1.778" layer="95"/>
+</segment>
+</net>

Commit message: Add more connections to Teensy
Connections:
- new net N$11: LED3.A, R7.1
- new net N$12: LED2.A, R5.1
- new net N$13: R6.2, U$1.36/A17/PWM
- new net N$14: LED4.A, R8.1
- new net N$15: LED5.A, R4.1
- new net N$2: JP1.1, U$1.5V
- new net N$3: JP1.5
- new net N$4: JP1.4
- new net N$5: R4.2, U$1.35/A16/PWM
- new net N$6: R5.2, U$1.37/A18/PWM/SCL1
- new net N$7: R7.2, U$1.38/A19/PWM/SDA1
- new net N$8: R8.2, U$1.39/A20/ALT-MISO0
- new net N$9: LED1.A, R6.1
- net GND: now also JP1.2, LED1.C, LED2.C, LED3.C, LED4.C, LED5.C
Other:
- note added: "5V"
- note added: "5V Out EN"
- note added: "Adafruit 5V Boost 500mA"
- note added: "Adafruit I2S Microphone SPH0645LM4H"
- note added: "Bat"
- note added: "EN"
- note added: "GND"
- note added: "LB"
- note added: "Low Battery Indicator"
- note removed: "5V Boost 500mA"
- note removed: "Microphone In"
- moved on the sheet: JP1, LED1, LED2, LED3, LED4, LED5, R4, R5, R6, R7, R8, SW1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

Commit message: Remove extra SMA connector
Parts:
- removed X1: ANTENNA, adafruit:SMACONNECTOR
Connections:
- removed net N$1: CON1.AN, X1.ANT
Changed lines of the file:
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@@
 <?xml version="1.0" encoding="utf-8"?>
 <!DOCTYPE eagle SYSTEM "eagle.dtd">
-<eagle version="9.2.2">
+<eagle version="9.3.0">
 <drawing>
 <settings>
@@
 <part name="R6" library="adafruit" library_urn="urn:adsk.eagle:library:420" deviceset="R-US_" device="M0805" package3d_urn="urn:adsk.eagle:package:6240587/1"/>
 <part name="R7" library="adafruit" library_urn="urn:adsk.eagle:library:420" deviceset="R-US_" device="M0805" package3d_urn="urn:adsk.eagle:package:6240587/1"/>
-<part name="X1" library="adafruit" library_urn="urn:adsk.eagle:library:420" deviceset="SMACONNECTOR" device="" package3d_urn="urn:adsk.eagle:package:6240946/1" value="ANTENNA"/>
 <part name="SW1" library="adafruit" library_urn="urn:adsk.eagle:library:420" deviceset="SPST_TACT" device="-KMR2" package3d_urn="urn:adsk.eagle:package:6240885/1"/>
 <part name="SW2" library="adafruit" library_urn="urn:adsk.eagle:library:420" deviceset="SWITCH_PUSHBUTTON" device="EVQ-PE" package3d_urn="urn:adsk.eagle:package:6240957/1"/>
@@
 <attribute name="VALUE" x="-44.45" y="-31.242" size="1.778" layer="96"/>
 </instance>
-<instance part="X1" gate="G$1" x="129.54" y="101.6" smashed="yes">
-<attribute name="NAME" x="137.16" y="104.14" size="1.27" layer="95"/>
-<attribute name="VALUE" x="137.16" y="101.6" size="1.27" layer="95"/>
-</instance>
 <instance part="SW1" gate="G$1" x="-48.26" y="96.52" smashed="yes" rot="R90">
 <attribute name="NAME" x="-45.72" y="90.17" size="1.778" layer="95" rot="R180"/>
@@
 </busses>
 <nets>
-<net name="N$1" class="0">
-<segment>
-<pinref part="CON1" gate="G$1" pin="AN"/>
-<pinref part="X1" gate="G$1" pin="ANT"/>
-<wire x1="119.38" y1="71.12" x2="119.38" y2="101.6" width="0.1524" layer="91"/>
-<wire x1="119.38" y1="101.6" x2="121.92" y2="101.6" width="0.1524" layer="91"/>
-</segment>
-</net>
 <net name="3V" class="0">
 <segment>

Commit message: Add more connections and adjust layour inlcude room for board fitting
Parts:
- removed LED1, LED2, LED3, LED4, LED5: (no value), adafruit:LEDCHIP-LED0805
- added CN1, CN2: (no value), adafruit:JST_2PIN-SMT-RA
- added ERRLED, LOWBATLED, LOWBATLED1, NETSTATLED, POWERLED, RECLED, SDLED: (no value), adafruit:LEDCHIP-LED0805
- added R9: 330R, adafruit:R-US_M0805
- added S1, S2: (no value), adafruit:31-XXSKINNY
- R1: value (none) -> 1KR
- R3, R4, R5, R6, R7, R8: value (none) -> 330R
Connections:
- removed net N$6: R5.2, U$1.37/A18/PWM/SCL1
- new net N$1: SW2.P$2, U$1.4/PWM/SDA2/CAN0RX
- new net N$10: JP1.3, R3.1
- new net N$16: LOWBATLED.A, R3.2
- new net N$17: CN1.1
- new net N$19: JP2.5, S2.S
- new net N$20: JP2.3, R9.1
- new net N$21: U$1.38/A19/PWM/SDA1
- new net N$23: LOWBATLED1.A, R9.2
- new net N$24: CN2.2, JP2.7
- new net N$25: CON1.5V, JP2.1
- new net N$3: CN1.2, JP1.6
- net CTS_OF_GSM: now also CON1.CS, R1.2
- net GND: now also CN2.1, CON1.GND1, CON1.GND2, ERRLED.C, JP2.2, JP2.4, LOWBATLED.C, LOWBATLED1.C, NETSTATLED.C, POWERLED.C, R1.1, RECLED.C, S1.S, S2.P, SDLED.C, SW2.P$1; no longer LED1.C, LED2.C, LED3.C, LED4.C, LED5.C
- net N$11: now also NETSTATLED.A; no longer LED3.A
- net N$12: now also SDLED.A; no longer LED2.A
- net N$14: now also ERRLED.A; no longer LED4.A
- net N$15: now also POWERLED.A; no longer LED5.A
- net N$4: now also S1.P
- net N$7: no longer U$1.38/A19/PWM/SDA1
- net N$8: no longer U$1.39/A20/ALT-MISO0
- net N$9: now also RECLED.A; no longer LED1.A
- net RESET_GSM: now also CON1.RST
- net RTS_OF_GSM: now also CON1.INT
- net RX_OF_GSM: now also CON1.RX
- net TX_OF_GSM: now also CON1.TX
Other:
- note added: "VBAT"
- note added: "VS"
- note added: "VUSB"
- moved on the sheet: R1, R2, R3, SW1, SW2

Commit message: Tidy up and complete schematics for review
Parts:
- removed LED6: RGBLED5050, adafruit:RGBLED5050
- removed R2: (no value), adafruit:R-US_M0805
- removed SW1: SPST_TACT-KMR2, adafruit:SPST_TACT-KMR2
- S1: value (none) -> Microcontroller and Mic power
- S2: value (none) -> GSM power
- SW2: value (none) -> Push_Button
- renumbered LOWBATLED to REC_LOW_BAT_LED, LOWBATLED1 to GSM_LOW_BAT_LED
Connections:
- net N$11: now also ERRLED.A, R8.2; no longer NETSTATLED.A, R7.1
- net N$12: now also U$1.39/A20/ALT-MISO0; no longer SDLED.A
- net N$14: now also U$1.37/A18/PWM/SCL1; no longer ERRLED.A
- net N$21: now also R7.1
- net N$7: now also NETSTATLED.A
- net N$8: now also R5.2, SDLED.A; no longer R8.2
Other:
- note added: "5V Out EN - Recorder On/Off"
- note added: "5V Out EN - Transmitter On/Off"
- note removed: "5V Out EN"
- moved on the sheet: ERRLED, NETSTATLED, R5, R7, R8, SDLED

Commit message: Fix/Swap RTS and CTS connections
Connections:
- net CTS_OF_GSM: now also CON1.INT; no longer CON1.CS, R1.2
- net RTS_OF_GSM: now also CON1.CS, R1.2; no longer CON1.INT
Changed lines of the file:
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@@
 <net name="CTS_OF_GSM" class="0">
 <segment>
+<wire x1="162.56" y1="-15.24" x2="162.56" y2="66.04" width="0.1524" layer="91"/>
+<pinref part="CON1" gate="G$1" pin="INT"/>
+<wire x1="162.56" y1="66.04" x2="157.48" y2="66.04" width="0.1524" layer="91"/>
 <pinref part="U$1" gate="G$1" pin="33/A14/CAN1TX/TX5/ALT-SCL0"/>
 <wire x1="30.48" y1="2.54" x2="-2.54" y2="2.54" width="0.1524" layer="91"/>
 <label x="0" y="2.54" size="1.778" layer="95"/>
 <wire x1="-2.54" y1="2.54" x2="-2.54" y2="-15.24" width="0.1524" layer="91"/>
-<wire x1="-2.54" y1="-15.24" x2="106.68" y2="-15.24" width="0.1524" layer="91"/>
-<pinref part="CON1" gate="G$1" pin="CS"/>
-<wire x1="119.38" y1="60.96" x2="111.76" y2="60.96" width="0.1524" layer="91"/>
-<wire x1="111.76" y1="60.96" x2="106.68" y2="60.96" width="0.1524" layer="91"/>
-<wire x1="106.68" y1="60.96" x2="106.68" y2="-15.24" width="0.1524" layer="91"/>
-<pinref part="R1" gate="G$1" pin="2"/>
-<wire x1="111.76" y1="55.88" x2="111.76" y2="60.96" width="0.1524" layer="91"/>
-<junction x="111.76" y="60.96"/>
+<wire x1="-2.54" y1="-15.24" x2="162.56" y2="-15.24" width="0.1524" layer="91"/>
 </segment>
 </net>
 <net name="RTS_OF_GSM" class="0">
 <segment>
+<label x="0" y="0" size="1.778" layer="95"/>
+</segment>
+<segment>
 <pinref part="U$1" gate="G$1" pin="34/A15/CAN1RX/RX5/ALT-SDA0"/>
 <wire x1="30.48" y1="0" x2="0" y2="0" width="0.1524" layer="91"/>
+<wire x1="0" y1="0" x2="0" y2="-12.7" width="0.1524" layer="91"/>
+<wire x1="0" y1="-12.7" x2="106.68" y2="-12.7" width="0.1524" layer="91"/>
+<pinref part="CON1" gate="G$1" pin="CS"/>
+<wire x1="119.38" y1="60.96" x2="111.76" y2="60.96" width="0.1524" layer="91"/>
+<wire x1="111.76" y1="60.96" x2="106.68" y2="60.96" width="0.1524" layer="91"/>
+<junction x="111.76" y="60.96"/>
+<pinref part="R1" gate="G$1" pin="2"/>
+<wire x1="111.76" y1="55.88" x2="111.76" y2="60.96" width="0.1524" layer="91"/>
+<wire x1="106.68" y1="-12.7" x2="106.68" y2="60.96" width="0.1524" layer="91"/>
 <label x="0" y="0" size="1.778" layer="95"/>
-<wire x1="0" y1="0" x2="0" y2="-12.7" width="0.1524" layer="91"/>
-<wire x1="0" y1="-12.7" x2="162.56" y2="-12.7" width="0.1524" layer="91"/>
-<wire x1="162.56" y1="-12.7" x2="162.56" y2="66.04" width="0.1524" layer="91"/>
-<pinref part="CON1" gate="G$1" pin="INT"/>
-<wire x1="162.56" y1="66.04" x2="157.48" y2="66.04" width="0.1524" layer="91"/>
 </segment>
 </net>
@@
 </segment>
 </net>
-<net name="N$22" class="0">
-<segment>
-<wire x1="101.6" y1="-12.7" x2="121.92" y2="-12.7" width="0.1524" layer="91"/>
-</segment>
-</net>
