File: Teensy36_I2S_Proto/wildly_teensy_proto.sch (EAGLE design)
At the start: 25 parts, among them CON1 MIKROE_BUS_CONN, SW2 Push_Button

Commit message: Clean schematics after review with Hari on 25/2/2019, BOM to be prepared
Parts:
- removed CN1, CN2: (no value), adafruit:JST_2PIN-SMT-RA
- removed CON1: MIKROE_BUS_CONN, mikrobus_lib:MIKROE_BUS_CONN
- added GSM_POWER, REC_POWER: (no value), adafruit:JST_2PIN-SMT-RA
- added MIKROELECTRONIKA_SARA_CLICK: MIKROE_BUS_CONN, mikrobus_lib:MIKROE_BUS_CONN
- R3, R4, R5, R6, R7, R8, R9: value 330R -> 1KR
Connections:
- net 3V renamed MIC_3V
- net BCLK renamed MIC_BCLK
- net DOUT renamed MIC_DOUT
- net LRCLK renamed MIC_LRCLK
- net N$10 renamed REC_LB
- net N$2 renamed REC_5V
- net N$20 renamed GSM_LB
- net N$21 renamed NETSTATLED
- removed net N$12: R5.1, U$1.39/A20/ALT-MISO0
- removed net N$13: R6.2, U$1.36/A17/PWM
- removed net N$14: R8.1, U$1.37/A18/PWM/SCL1
- removed net N$15: POWERLED.A, R4.1
- removed net N$17: CN1.1
- removed net N$18: JP1.5
- removed net N$19: JP2.5, S2.S
- removed net N$24: CN2.2, JP2.7
- removed net N$25: CON1.5V, JP2.1
- removed net N$4: JP1.4, S1.P
- removed net N$5: R4.2, U$1.35/A16/PWM
- new net ERRLED: R8.1, U$1.39/A20/ALT-MISO0
- new net GSM_5V: JP2.1, MIKROELECTRONIKA_SARA_CLICK.5V
- new net GSM_5V_EN: JP2.5, S2.P
- new net GSM_BAT: GSM_POWER.2, JP2.7
- new net GSM_BAT_RETURN: GSM_POWER.1, JP2.4
- new net N$6: JP2.6
- new net POWERLED: R4.1, U$1.35/A16/PWM
- new net RECLED: R6.1, U$1.36/A17/PWM
- new net REC_5V_EN: JP1.4, S1.S
- new net REC_BAT: JP1.6, REC_POWER.2
- new net REC_BAT_RETURN: JP1.5, REC_POWER.1
- new net SDLED: R5.1, U$1.37/A18/PWM/SCL1
- net CTS_OF_GSM: now also MIKROELECTRONIKA_SARA_CLICK.INT; no longer CON1.INT
- net GND: now also MIKROELECTRONIKA_SARA_CLICK.GND1, MIKROELECTRONIKA_SARA_CLICK.GND2, S1.P, S2.S; no longer CN2.1, CON1.GND1, CON1.GND2, JP2.4, S1.S, S2.P
- net N$3: now also POWERLED.A, R4.2; no longer CN1.2, JP1.6
- net N$9: now also R6.2; no longer R6.1
- net RESET_GSM: now also MIKROELECTRONIKA_SARA_CLICK.RST; no longer CON1.RST
- net RTS_OF_GSM: now also MIKROELECTRONIKA_SARA_CLICK.CS; no longer CON1.CS
- net RX_OF_GSM: now also MIKROELECTRONIKA_SARA_CLICK.RX; no longer CON1.RX
- net TX_OF_GSM: now also MIKROELECTRONIKA_SARA_CLICK.TX; no longer CON1.TX
Other:
- note added: "GSM Low Battery Indicator"
- note added: "Recroder Low Battery Indicator"
- note removed: "Low Battery Indicator"
- moved on the sheet: JP1, JP2, JP3, POWERLED, R1, R3, R4, R6, RECLED, REC_LOW_BAT_LED, S1, S2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

Commit message: Add Jumper to unify power supply for both recorder and GSM when needed, add LEDS for power switches, add caps for supply input
Parts:
- added C1, C3: 10uF, adafruit:C-USC0805
- added C2, C4: 100nF, adafruit:C-USC0805
- added GSM_POWER_JUMPER: (no value), jumper:JP1Q
- added GSM_PW_LED, REC_PW_LED: (no value), adafruit:LEDCHIP-LED0805
- added R10, R2: 1KR, adafruit:R-US_M0805
Connections:
- new net N$10: R2.1, REC_PW_LED.A
- new net N$12: R2.2
- new net N$4: GSM_PW_LED.A, R10.2
- new net N$5: GSM_PW_LED.C, S2.P
- net GND: now also C1.2, C2.2, C3.2, C4.2
- net GSM_5V: now also C3.1, C4.1, GSM_POWER_JUMPER.1
- net GSM_5V_EN: now also R10.1; no longer S2.P
- net REC_5V: now also C1.1, C2.1, GSM_POWER_JUMPER.2
- net REC_5V_EN: now also REC_PW_LED.C
Changed lines of the file:
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@@
 <part name="S2" library="adafruit" library_urn="urn:adsk.eagle:library:420" deviceset="31-XX" device="SKINNY" package3d_urn="urn:adsk.eagle:package:6240899/1" value="GSM power"/>
 <part name="GND1" library="supply1" library_urn="urn:adsk.eagle:library:371" deviceset="GND" device=""/>
+<part name="C1" library="adafruit" library_urn="urn:adsk.eagle:library:420" deviceset="C-US" device="C0805" package3d_urn="urn:adsk.eagle:package:6240337/1" value="10uF"/>
+<part name="C2" library="adafruit" library_urn="urn:adsk.eagle:library:420" deviceset="C-US" device="C0805" package3d_urn="urn:adsk.eagle:package:6240337/1" value="100nF"/>
+<part name="GND2" library="supply1" library_urn="urn:adsk.eagle:library:371" deviceset="GND" device=""/>
+<part name="C3" library="adafruit" library_urn="urn:adsk.eagle:library:420" deviceset="C-US" device="C0805" package3d_urn="urn:adsk.eagle:package:6240337/1" value="10uF"/>
+<part name="C4" library="adafruit" library_urn="urn:adsk.eagle:library:420" deviceset="C-US" device="C0805" package3d_urn="urn:adsk.eagle:package:6240337/1" value="100nF"/>
+<part name="GND8" library="supply1" library_urn="urn:adsk.eagle:library:371" deviceset="GND" device=""/>
+<part name="GSM_POWER_JUMPER" library="jumper" library_urn="urn:adsk.eagle:library:252" deviceset="JP1Q" device="" package3d_urn="urn:adsk.eagle:package:15455/1"/>
+<part name="GSM_PW_LED" library="adafruit" library_urn="urn:adsk.eagle:library:420" deviceset="LED" device="CHIP-LED0805" package3d_urn="urn:adsk.eagle:package:6240557/1"/>
+<part name="R2" library="adafruit" library_urn="urn:adsk.eagle:library:420" deviceset="R-US_" device="M0805" package3d_urn="urn:adsk.eagle:package:6240587/1" value="1KR"/>
+<part name="REC_PW_LED" library="adafruit" library_urn="urn:adsk.eagle:library:420" deviceset="LED" device="CHIP-LED0805" package3d_urn="urn:adsk.eagle:package:6240557/1"/>
+<part name="R10" library="adafruit" library_urn="urn:adsk.eagle:library:420" deviceset="R-US_" device="M0805" package3d_urn="urn:adsk.eagle:package:6240587/1" value="1KR"/>
 </parts>
 <sheets>
@@
 <attribute name="VALUE" x="177.8" y="114.3" size="1.778" layer="96"/>
 </instance>
+<instance part="C1" gate="G$1" x="116.84" y="86.36" smashed="yes">
+<attribute name="NAME" x="117.856" y="86.995" size="1.778" layer="95"/>
+<attribute name="VALUE" x="117.856" y="82.169" size="1.778" layer="96"/>
+</instance>
+<instance part="C2" gate="G$1" x="106.68" y="86.36" smashed="yes">
+<attribute name="NAME" x="107.696" y="86.995" size="1.778" layer="95"/>
+<attribute name="VALUE" x="107.696" y="82.169" size="1.778" layer="96"/>
+</instance>
+<instance part="GND2" gate="1" x="111.76" y="71.12" smashed="yes">
+<attribute name="VALUE" x="109.22" y="68.58" size="1.778" layer="96"/>
+</instance>
+<instance part="C3" gate="G$1" x="213.36" y="53.34" smashed="yes">
+<attribute name="NAME" x="214.376" y="53.975" size="1.778" layer="95"/>
+<attribute name="VALUE" x="214.376" y="49.149" size="1.778" layer="96"/>
+</instance>
+<instance part="C4" gate="G$1" x="203.2" y="53.34" smashed="yes">
+<attribute name="NAME" x="204.216" y="53.975" size="1.778" layer="95"/>
+<attribute name="VALUE" x="204.216" y="49.149" size="1.778" layer="96"/>
+</instance>
+<instance part="GND8" gate="1" x="208.28" y="38.1" smashed="yes">
+<attribute name="VALUE" x="205.74" y="35.56" size="1.778" layer="96"/>
+</instance>
+<instance part="GSM_POWER_JUMPER" gate="A" x="-60.96" y="119.38" smashed="yes" rot="R90">
+<attribute name="NAME" x="-48.26" y="116.84" size="1.778" layer="95" rot="R180"/>
+<attribute name="VALUE" x="-55.88" y="123.825" size="1.778" layer="96" rot="R180"/>
+</instance>
+<instance part="GSM_PW_LED" gate="G$1" x="149.86" y="127" smashed="yes" rot="R90">
+<attribute name="NAME" x="159.512" y="130.556" size="1.778" layer="95" rot="R180"/>
+<attribute name="VALUE" x="154.432" y="132.715" size="1.778" layer="96" rot="R180"/>
+</instance>
+<instance part="R2" gate="G$1" x="68.58" y="116.84" smashed="yes">
+<attribute name="NAME" x="64.77" y="118.3386" size="1.778" layer="95"/>
+<attribute name="VALUE" x="64.77" y="113.538" size="1.778" layer="96"/>
+</instance>
+<instance part="REC_PW_LED" gate="G$1" x="53.34" y="116.84" smashed="yes" rot="R270">
+<attribute name="NAME" x="43.688" y="113.284" size="1.778" layer="95"/>
+<attribute name="VALUE" x="48.768" y="111.125" size="1.778" layer="96"/>
+</instance>
+<instance part="R10" gate="G$1" x="134.62" y="127" smashed="yes">
+<attribute name="NAME" x="130.81" y="128.4986" size="1.778" layer="95"/>
+<attribute name="VALUE" x="130.81" y="123.698" size="1.778" layer="96"/>
+</instance>
 </instances>
 <busses>
@@
 <wire x1="7.62" y1="116.84" x2="7.62" y2="111.76" width="0.1524" layer="91"/>
 </segment>
+<segment>
+<pinref part="C2" gate="G$1" pin="2"/>
+<wire x1="106.68" y1="81.28" x2="106.68" y2="76.2" width="0.1524" layer="91"/>
+<wire x1="106.68" y1="76.2" x2="111.76" y2="76.2" width="0.1524" layer="91"/>
+<pinref part="C1" gate="G$1" pin="2"/>
+<wire x1="111.76" y1="76.2" x2="116.84" y2="76.2" width="0.1524" layer="91"/>
+<wire x1="116.84" y1="76.2" x2="116.84" y2="81.28" width="0.1524" layer="91"/>
+<pinref part="GND2" gate="1" pin="GND"/>
+<wire x1="111.76" y1="76.2" x2="111.76" y2="73.66" width="0.1524" layer="91"/>
+<junction x="111.76" y="76.2"/>
+</segment>
+<segment>
+<pinref part="C4" gate="G$1" pin="2"/>
+<wire x1="203.2" y1="48.26" x2="203.2" y2="43.18" width="0.1524" layer="91"/>
+<wire x1="203.2" y1="43.18" x2="208.28" y2="43.18" width="0.1524" layer="91"/>
+<pinref part="C3" gate="G$1" pin="2"/>
+<wire x1="208.28" y1="43.18" x2="213.36" y2="43.18" width="0.1524" layer="91"/>
+<wire x1="213.36" y1="43.18" x2="213.36" y2="48.26" width="0.1524" layer="91"/>
+<pinref part="GND8" gate="1" pin="GND"/>
+<wire x1="208.28" y1="43.18" x2="208.28" y2="40.64" width="0.1524" layer="91"/>
+<junction x="208.28" y="43.18"/>
+</segment>
 </net>
 <net name="TX_OF_GSM" class="0">
@@
 <segment>
 <pinref part="S1" gate="1" pin="S"/>
-<wire x1="22.86" y1="116.84" x2="45.72" y2="116.84" width="0.1524" layer="91"/>
-<label x="40.64" y="114.3" size="1.778" layer="95"/>
+<wire x1="22.86" y1="116.84" x2="48.26" y2="116.84" width="0.1524" layer="91"/>
+<label x="78.74" y="116.84" size="1.778" layer="95"/>
+<pinref part="REC_PW_LED" gate="G$1" pin="C"/>
 </segment>
 </net>
@@
 <segment>
 <pinref part="U$1" gate="G$1" pin="5V"/>
+<label x="106.68" y="91.44" size="1.778" layer="95"/>
 <wire x1="99.06" y1="91.44" x2="106.68" y2="91.44" width="0.1524" layer="91"/>
-<label x="106.68" y="91.44" size="1.778" layer="95"/>
+<pinref part="C1" gate="G$1" pin="1"/>
+<wire x1="106.68" y1="91.44" x2="116.84" y2="91.44" width="0.1524" layer="91"/>
+<wire x1="116.84" y1="91.44" x2="116.84" y2="88.9" width="0.1524" layer="91"/>
+<pinref part="C2" gate="G$1" pin="1"/>
+<wire x1="106.68" y1="91.44" x2="106.68" y2="88.9" width="0.1524" layer="91"/>
+<junction x="106.68" y="91.44"/>
+</segment>
+<segment>
+<pinref part="GSM_POWER_JUMPER" gate="A" pin="2"/>
+<wire x1="-68.58" y1="119.38" x2="-78.74" y2="119.38" width="0.1524" layer="91"/>
+<label x="-81.28" y="119.38" size="1.778" layer="95"/>
 </segment>
 </net>
@@
 <pinref part="JP2" gate="G$1" pin="6"/>
 <wire x1="-58.42" y1="43.18" x2="-45.72" y2="43.18" width="0.1524" layer="91"/>
-<label x="-45.72" y="43.18" size="1.778" layer="95"/>
 </segment>
 </net>
@@
 </segment>
 <segment>
-<pinref part="S2" gate="1" pin="P"/>
-<wire x1="162.56" y1="127" x2="104.14" y2="127" width="0.1524" layer="91"/>
-<label x="101.6" y="127" size="1.778" layer="95"/>
+<pinref part="R10" gate="G$1" pin="1"/>
+<wire x1="129.54" y1="127" x2="116.84" y2="127" width="0.1524" layer="91"/>
+<label x="106.68" y="127" size="1.778" layer="95"/>
 </segment>
 </net>
@@
 <segment>
 <pinref part="MIKROELECTRONIKA_SARA_CLICK" gate="G$1" pin="5V"/>
+<label x="198.12" y="60.96" size="1.778" layer="95"/>
 <wire x1="193.04" y1="60.96" x2="203.2" y2="60.96" width="0.1524" layer="91"/>
-<label x="198.12" y="60.96" size="1.778" layer="95"/>
+<pinref part="C3" gate="G$1" pin="1"/>
+<pinref part="C4" gate="G$1" pin="1"/>
+<wire x1="203.2" y1="60.96" x2="213.36" y2="60.96" width="0.1524" layer="91"/>
+<wire x1="213.36" y1="60.96" x2="213.36" y2="55.88" width="0.1524" layer="91"/>
+<wire x1="203.2" y1="55.88" x2="203.2" y2="60.96" width="0.1524" layer="91"/>
+<junction x="203.2" y="60.96"/>
+</segment>
+<segment>
+<pinref part="GSM_POWER_JUMPER" gate="A" pin="1"/>
+<wire x1="-53.34" y1="119.38" x2="-43.18" y2="119.38" width="0.1524" layer="91"/>
+<label x="-45.72" y="119.38" size="1.778" layer="95"/>
 </segment>
 </net>
@@
 </segment>
 </net>
+<net name="N$4" class="0">
+<segment>
+<pinref part="R10" gate="G$1" pin="2"/>
+<pinref part="GSM_PW_LED" gate="G$1" pin="A"/>
+<wire x1="139.7" y1="127" x2="147.32" y2="127" width="0.1524" layer="91"/>
+</segment>
+</net>
+<net name="N$5" class="0">
+<segment>
+<pinref part="GSM_PW_LED" gate="G$1" pin="C"/>
+<pinref part="S2" gate="1" pin="P"/>
+<wire x1="154.94" y1="127" x2="162.56" y2="127" width="0.1524" layer="91"/>
+</segment>
+</net>
+<net name="N$10" class="0">
+<segment>
+<pinref part="REC_PW_LED" gate="G$1" pin="A"/>
+<pinref part="R2" gate="G$1" pin="1"/>
+<wire x1="55.88" y1="116.84" x2="63.5" y2="116.84" width="0.1524" layer="91"/>
+</segment>
+</net>
+<net name="N$12" class="0">
+<segment>
+<pinref part="R2" gate="G$1" pin="2"/>
+<wire x1="73.66" y1="116.84" x2="83.82" y2="116.84" width="0.1524" layer="91"/>
+</segment>
+</net>

Commit message: Remove LEDs for Power Enables, Remove LEDs for Low Bat indicators, Add NPN Transistors as LED drivers - TBD: Calculate R values, Remove Power LED and change pinout to power control for resetting system power- TBD: add connection, Provide 3.3V to GSM modem
Parts:
- removed GSM_LOW_BAT_LED, GSM_PW_LED, POWERLED, REC_LOW_BAT_LED, REC_PW_LED: (no value), adafruit:LEDCHIP-LED0805
- removed R4, R5, R6, R7, R8: 1KR, adafruit:R-US_M0805
- added R11, R12, R13, R14: 1KR, adafruit:R-US_M0805
- added T1, T2, T3, T4: 2N2222, adafruit:2N2222
Connections:
- removed net N$12: R2.2
- removed net N$23: GSM_LOW_BAT_LED.A, R9.2
- removed net POWERLED: R4.1, U$1.35/A16/PWM
- new net 3V3: MIKROELECTRONIKA_SARA_CLICK.3V3, R10.2, R11.2, R12.2, R14.2
- new net N$14: R10.1, RECLED.A
- new net N$15: ERRLED.A, R11.1
- new net N$16: NETSTATLED.A, R12.1
- new net POWER_CONTRL: U$1.35/A16/PWM
- net ERRLED: now also R3.1; no longer R8.1
- net GND: now also T1.E, T2.E, T3.E, T4.E; no longer ERRLED.C, GSM_LOW_BAT_LED.C, NETSTATLED.C, POWERLED.C, RECLED.C, REC_LOW_BAT_LED.C, SDLED.C
- net GSM_5V_EN: now also S2.P; no longer R10.1
- net GSM_LB: no longer R9.1
- net N$10: now also SDLED.C, T4.C; no longer R2.1, REC_PW_LED.A
- net N$11: now also R13.2, T4.B; no longer ERRLED.A, R8.2
- net N$2: now also RECLED.C, T2.C; no longer R3.2, REC_LOW_BAT_LED.A
- net N$3: now also R2.2, T2.B; no longer POWERLED.A, R4.2
- net N$4: now also ERRLED.C, T1.C; no longer GSM_PW_LED.A, R10.2
- net N$5: now also NETSTATLED.C, T3.C; no longer GSM_PW_LED.C, S2.P
- net N$7: now also R9.2, T3.B; no longer NETSTATLED.A, R7.2
- net N$8: now also R3.2, T1.B; no longer R5.2, SDLED.A
- net N$9: now also R14.1, SDLED.A; no longer R6.2, RECLED.A
- net NETSTATLED: now also R9.1; no longer R7.1
- net RECLED: now also R2.1; no longer R6.1
- net REC_5V_EN: no longer REC_PW_LED.C
- net REC_LB: no longer R3.1
- net SDLED: now also R13.1; no longer R5.1
Other:
- note removed: "GSM Low Battery Indicator"
- note removed: "Recroder Low Battery Indicator"
- moved on the sheet: ERRLED, NETSTATLED, R10, R2, R3, R9, RECLED, S2, SDLED

Commit message: Add resistor values for LED driver, remove previous board file due to inconsistency and create a fresh layout from schematics
Parts:
- R10, R11, R12: value 1KR -> 82R
- R13, R2, R3, R9: value 1KR -> 1.65KR
Changed lines of the file:
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@@
 <part name="ERRLED" library="adafruit" library_urn="urn:adsk.eagle:library:420" deviceset="LED" device="CHIP-LED0805" package3d_urn="urn:adsk.eagle:package:6240557/1"/>
 <part name="RECLED" library="adafruit" library_urn="urn:adsk.eagle:library:420" deviceset="LED" device="CHIP-LED0805" package3d_urn="urn:adsk.eagle:package:6240557/1"/>
-<part name="R2" library="adafruit" library_urn="urn:adsk.eagle:library:420" deviceset="R-US_" device="M0805" package3d_urn="urn:adsk.eagle:package:6240587/1" value="1KR"/>
-<part name="R3" library="adafruit" library_urn="urn:adsk.eagle:library:420" deviceset="R-US_" device="M0805" package3d_urn="urn:adsk.eagle:package:6240587/1" value="1KR"/>
-<part name="R9" library="adafruit" library_urn="urn:adsk.eagle:library:420" deviceset="R-US_" device="M0805" package3d_urn="urn:adsk.eagle:package:6240587/1" value="1KR"/>
-<part name="R10" library="adafruit" library_urn="urn:adsk.eagle:library:420" deviceset="R-US_" device="M0805" package3d_urn="urn:adsk.eagle:package:6240587/1" value="1KR"/>
-<part name="R11" library="adafruit" library_urn="urn:adsk.eagle:library:420" deviceset="R-US_" device="M0805" package3d_urn="urn:adsk.eagle:package:6240587/1" value="1KR"/>
-<part name="R12" library="adafruit" library_urn="urn:adsk.eagle:library:420" deviceset="R-US_" device="M0805" package3d_urn="urn:adsk.eagle:package:6240587/1" value="1KR"/>
+<part name="R2" library="adafruit" library_urn="urn:adsk.eagle:library:420" deviceset="R-US_" device="M0805" package3d_urn="urn:adsk.eagle:package:6240587/1" value="1.65KR"/>
+<part name="R3" library="adafruit" library_urn="urn:adsk.eagle:library:420" deviceset="R-US_" device="M0805" package3d_urn="urn:adsk.eagle:package:6240587/1" value="1.65KR"/>
+<part name="R9" library="adafruit" library_urn="urn:adsk.eagle:library:420" deviceset="R-US_" device="M0805" package3d_urn="urn:adsk.eagle:package:6240587/1" value="1.65KR"/>
+<part name="R10" library="adafruit" library_urn="urn:adsk.eagle:library:420" deviceset="R-US_" device="M0805" package3d_urn="urn:adsk.eagle:package:6240587/1" value="82R"/>
+<part name="R11" library="adafruit" library_urn="urn:adsk.eagle:library:420" deviceset="R-US_" device="M0805" package3d_urn="urn:adsk.eagle:package:6240587/1" value="82R"/>
+<part name="R12" library="adafruit" library_urn="urn:adsk.eagle:library:420" deviceset="R-US_" device="M0805" package3d_urn="urn:adsk.eagle:package:6240587/1" value="82R"/>
 <part name="T1" library="adafruit" library_urn="urn:adsk.eagle:library:420" deviceset="2N2222" device="" package3d_urn="urn:adsk.eagle:package:6240647/1"/>
 <part name="T2" library="adafruit" library_urn="urn:adsk.eagle:library:420" deviceset="2N2222" device="" package3d_urn="urn:adsk.eagle:package:6240647/1"/>
 <part name="T3" library="adafruit" library_urn="urn:adsk.eagle:library:420" deviceset="2N2222" device="" package3d_urn="urn:adsk.eagle:package:6240647/1"/>
 <part name="SDLED" library="adafruit" library_urn="urn:adsk.eagle:library:420" deviceset="LED" device="CHIP-LED0805" package3d_urn="urn:adsk.eagle:package:6240557/1"/>
-<part name="R13" library="adafruit" library_urn="urn:adsk.eagle:library:420" deviceset="R-US_" device="M0805" package3d_urn="urn:adsk.eagle:package:6240587/1" value="1KR"/>
+<part name="R13" library="adafruit" library_urn="urn:adsk.eagle:library:420" deviceset="R-US_" device="M0805" package3d_urn="urn:adsk.eagle:package:6240587/1" value="1.65KR"/>
 <part name="R14" library="adafruit" library_urn="urn:adsk.eagle:library:420" deviceset="R-US_" device="M0805" package3d_urn="urn:adsk.eagle:package:6240587/1" value="1KR"/>
 <part name="T4" library="adafruit" library_urn="urn:adsk.eagle:library:420" deviceset="2N2222" device="" package3d_urn="urn:adsk.eagle:package:6240647/1"/>

Commit message: Add BOM file, fix R value for LED driver, start component placement in layout
Parts:
- R14: value 1KR -> 82R
Changed lines of the file:
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@@
 <part name="SDLED" library="adafruit" library_urn="urn:adsk.eagle:library:420" deviceset="LED" device="CHIP-LED0805" package3d_urn="urn:adsk.eagle:package:6240557/1"/>
 <part name="R13" library="adafruit" library_urn="urn:adsk.eagle:library:420" deviceset="R-US_" device="M0805" package3d_urn="urn:adsk.eagle:package:6240587/1" value="1.65KR"/>
-<part name="R14" library="adafruit" library_urn="urn:adsk.eagle:library:420" deviceset="R-US_" device="M0805" package3d_urn="urn:adsk.eagle:package:6240587/1" value="1KR"/>
+<part name="R14" library="adafruit" library_urn="urn:adsk.eagle:library:420" deviceset="R-US_" device="M0805" package3d_urn="urn:adsk.eagle:package:6240587/1" value="82R"/>
 <part name="T4" library="adafruit" library_urn="urn:adsk.eagle:library:420" deviceset="2N2222" device="" package3d_urn="urn:adsk.eagle:package:6240647/1"/>
 </parts>

Commit message: Fix power line, change layout according to review with Hari on 11/3/2019. TBD: BOM finalization and final footprint alignment
Parts:
- renumbered JP1 to WILDLY_5V_0.5A_BOOST, JP2 to WILDLY_5V_1A_BOOST, JP3 to WILDLY_I2S_MIC, S1 to REC_ON_OFF_SW, S2 to GSM_ON_OFF_SW, SW2 to REC_SW
Connections:
- removed net MIC_3V: U$1.3V3, WILDLY_I2S_MIC.1
- new net NET_STAT: MIKROELECTRONIKA_SARA_CLICK.AN, U$1.24
- net 3V3: now also U$1.3V3, WILDLY_I2S_MIC.1
- net REC_5V: now also U$1.VIN; no longer U$1.5V
Other:
- moved on the sheet: C1, C2, ERRLED, NETSTATLED, R10, R11, R12, R13, R14, R2, R3, R9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
