File: Teensy36_I2S_Proto/wildly_teensy_proto.sch (EAGLE design)
At the start: 32 parts, among them T1 2N2222, T2 2N2222, T3 2N2222, T4 2N2222

Commit message: Add latest files from Aakash Nasa with updatest to schamtic and layout to include: Pinouts for unused pins from Teensy, changes to BOM according to component availabilityetc
Parts:
- added J1, J2: 61300311121, 61300311121:61300311121
- added J3: 61300211121, 61300211121:61300211121
- added TEENSY_PINS_1-6, TEENSY_PINS_13-18, TEENSY_PINS_19-24, TEENSY_PINS_25-30, TEENSY_PINS_31-36, TEENSY_PINS_37-42, TEENSY_PINS_43-48, TEENSY_PINS_7-12: (no value), adafruit:PINHD-1X6
- GSM_ON_OFF_SW: value GSM power -> GSM Power; device adafruit:31-XXSKINNY -> 1101M2S3CQE2:1101M2S3CQE2
- REC_ON_OFF_SW: value Microcontroller and Mic power -> Microcontroller and Mic Power; device adafruit:31-XXSKINNY -> 1101M2S3CQE2:1101M2S3CQE2
- REC_SW: device adafruit:SWITCH_PUSHBUTTONEVQ-PE -> 800AWSP9M2QE:800AWSP9M2QE
- T1, T2, T3, T4: value 2N2222 -> 2N2222A; device adafruit:2N2222 -> 2N2222A:2N2222A
Connections:
- removed net N$1: REC_SW.P$2, U$1.4/PWM/SDA2/CAN0RX
- new net 25: TEENSY_PINS_13-18.5, U$1.25
- new net A0: TEENSY_PINS_37-42.1, U$1.14/A0/PWM/ALT-SCK0
- new net A1: TEENSY_PINS_31-36.6, U$1.15/A1/CS0-4/T
- new net A2: TEENSY_PINS_31-36.5, U$1.16/A2/PWM/T/ALT-SCL0
- new net A3: TEENSY_PINS_31-36.4, U$1.17/A3/PWM/T/ALT-SDA0
- new net A4: J1.1, TEENSY_PINS_31-36.3, U$1.18/A4/PWM/T/SDA0
- new net A5: J1.2, TEENSY_PINS_31-36.2, U$1.19/A5/PWM/T/SCL0
- new net AGND: TEENSY_PINS_25-30.2, U$1.AGND
- new net ALT-MOSI: TEENSY_PINS_19-24.2, U$1.28/ALT-MOSI0
- new net ALT-PWM: TEENSY_PINS_13-18.6, U$1.26/ALT-PWM/ALT-TX1/ALT-SCL2
- new net ALT-RX1: TEENSY_PINS_19-24.1, U$1.27/ALT-RX1/ALT-SCK0
- new net DAC0: TEENSY_PINS_37-42.5, U$1.DAC0
- new net DAC1: TEENSY_PINS_37-42.4, U$1.DAC1
- new net MISO: TEENSY_PINS_13-18.2, U$1.12/MISO0
- new net MOSI: TEENSY_PINS_13-18.1, U$1.11/MOSI0
- new net N$13: J1.3
- new net PWM1: TEENSY_PINS_1-6.4, U$1.2/PWM
- new net PWM10: TEENSY_PINS_19-24.4, U$1.30/PWM/T/ALT-CAN0RX
- new net PWM11: TEENSY_PINS_19-24.5, U$1.31/A12/PWM/RX4/CS1-0
- new net PWM12: TEENSY_PINS_19-24.6, U$1.32/A13/PWM/TX4/SCK1
- new net PWM13: TEENSY_PINS_25-30.6, U$1.21/A7/PWM/CS0-3/ALT-MOSI1/ALT-RX1
- new net PWM14: TEENSY_PINS_25-30.5, U$1.22/A8/PWM/T
- new net PWM2: TEENSY_PINS_1-6.5, U$1.3/PWM/SCL2/CAN0TX
- new net PWM3: REC_SW.NO_2, TEENSY_PINS_1-6.6, U$1.4/PWM/SDA2/CAN0RX
- new net PWM4: TEENSY_PINS_7-12.1, U$1.5/PWM/ALT-TX1/ALT-MISO1
- new net PWM5: TEENSY_PINS_7-12.2, U$1.6/PWM
- new net PWM6: TEENSY_PINS_7-12.3, U$1.7/PWM/RX3/ALT-SCL0/ALT-MOSI0
- new net PWM7: TEENSY_PINS_7-12.4, U$1.8/PWM/TX3/ALT-SDA0/ALT-MISO0
- new net PWM8: TEENSY_PINS_7-12.6, U$1.10/PWM/TX2/CS0-0
- new net PWM9: TEENSY_PINS_19-24.3, U$1.29/PWM/T/ALT-CAN0TX
- net 3V3: now also TEENSY_PINS_13-18.3, TEENSY_PINS_25-30.3
- net CTS_OF_GSM: now also TEENSY_PINS_43-48.6
- net ERRLED: now also TEENSY_PINS_37-42.6
- net GND: now also GSM_ON_OFF_SW.1, J3.1, REC_ON_OFF_SW.2, REC_SW.NO_1, TEENSY_PINS_1-6.1, TEENSY_PINS_37-42.3; no longer GSM_ON_OFF_SW.S, REC_ON_OFF_SW.P, REC_SW.P$1
- net GSM_5V_EN: now also GSM_ON_OFF_SW.2; no longer GSM_ON_OFF_SW.P
- net MIC_BCLK: now also TEENSY_PINS_7-12.5
- net MIC_DOUT: now also TEENSY_PINS_37-42.2
- net MIC_LRCLK: now also TEENSY_PINS_25-30.4
- net NETSTATLED: now also TEENSY_PINS_43-48.1
- net NET_STAT: now also TEENSY_PINS_13-18.4
- net POWER_CONTRL: now also TEENSY_PINS_43-48.4
- net RECLED: now also TEENSY_PINS_43-48.3
- net REC_5V: now also J3.2, TEENSY_PINS_25-30.1
- net REC_5V_EN: now also REC_ON_OFF_SW.1; no longer REC_ON_OFF_SW.S
- net RESET_GSM: now also TEENSY_PINS_31-36.1
- net RTS_OF_GSM: now also TEENSY_PINS_43-48.5
- net RX_OF_GSM: now also TEENSY_PINS_1-6.3
- net SDLED: now also TEENSY_PINS_43-48.2
- net TX_OF_GSM: now also TEENSY_PINS_1-6.2
Other:
- note added: "LIPO - FUEL GAUGE"

Commit message: Teensy Proto schematic and Layout File updated
Parts:
- removed GSM_POWER: (no value), adafruit:JST_2PIN-SMT-RA
- added SOLAR_CHARGER: 61300211121, 61300211121:61300211121
- renumbered J3 to FUEL_GAUGE, TEENSY_PINS_1-6 to TEENSY_1, TEENSY_PINS_13-18 to TEENSY_3, TEENSY_PINS_19-24 to TEENSY_4, TEENSY_PINS_25-30 to TEENSY_5, TEENSY_PINS_31-36 to TEENSY_6, TEENSY_PINS_37-42 to TEENSY_7, TEENSY_PINS_43-48 to TEENSY_8, TEENSY_PINS_7-12 to TEENSY_2
Connections:
- net GND: no longer FUEL_GAUGE.1
- net GSM_BAT: now also FUEL_GAUGE.2, SOLAR_CHARGER.1; no longer GSM_POWER.2
- net GSM_BAT_RETURN: now also FUEL_GAUGE.1, SOLAR_CHARGER.2; no longer GSM_POWER.1
- net REC_5V: no longer FUEL_GAUGE.2
Other:
- note added: "Solar Charger"
- moved on the sheet: ERRLED, NETSTATLED, R10, R11, R12, R13, R14, R2, R3, R9, RECLED, SDLED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
