File: Teensy36_I2S_Proto/wildly_teensy_proto.sch (EAGLE design)
At the start: 43 parts, among them J1 61300311121, J2 61300311121, T1 2N2222A, T2 2N2222A, T3 2N2222A, T4 2N2222A

Commit message: Added different switch footprints
Parts:
- removed GSM_ON_OFF_SW: GSM Power, 1101M2S3CQE2:1101M2S3CQE2
- removed REC_SW: Push_Button, 800AWSP9M2QE:800AWSP9M2QE
- added GSM_ON_OFF_SW1: GSM Power, EG1218:EG1218
- added REC_SW1: Push_Button, 1-1825910-4:1-1825910-4
- REC_ON_OFF_SW: device 1101M2S3CQE2:1101M2S3CQE2 -> EG1218:EG1218
Connections:
- net GND: now also GSM_ON_OFF_SW1.COM, REC_ON_OFF_SW.COM, REC_SW1.1, REC_SW1.2; no longer GSM_ON_OFF_SW.1, REC_ON_OFF_SW.2, REC_SW.NO_1
- net GSM_5V_EN: now also GSM_ON_OFF_SW1.1; no longer GSM_ON_OFF_SW.2
- net PWM3: now also REC_SW1.3, REC_SW1.4; no longer REC_SW.NO_2
Changed lines of the file:
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@@
 <part name="GND11" library="supply1" library_urn="urn:adsk.eagle:library:371" deviceset="GND" device=""/>
 <part name="GND12" library="supply1" library_urn="urn:adsk.eagle:library:371" deviceset="GND" device=""/>
-<part name="REC_ON_OFF_SW" library="1101M2S3CQE2" deviceset="1101M2S3CQE2" device="" value="Microcontroller and Mic Power"/>
-<part name="GSM_ON_OFF_SW" library="1101M2S3CQE2" deviceset="1101M2S3CQE2" device="" value="GSM Power"/>
-<part name="REC_SW" library="800AWSP9M2QE" deviceset="800AWSP9M2QE" device="" value="Push_Button"/>
 <part name="T4" library="2N2222A" deviceset="2N2222A" device=""/>
 <part name="T3" library="2N2222A" deviceset="2N2222A" device=""/>
@@
 <part name="FUEL_GAUGE" library="61300211121" deviceset="61300211121" device=""/>
 <part name="SOLAR_CHARGER" library="61300211121" deviceset="61300211121" device=""/>
+<part name="REC_ON_OFF_SW" library="EG1218" deviceset="EG1218" device="" value="Microcontroller and Mic Power"/>
+<part name="GSM_ON_OFF_SW1" library="EG1218" deviceset="EG1218" device="" value="GSM Power"/>
+<part name="REC_SW1" library="1-1825910-4" deviceset="1-1825910-4" device="" value="Push_Button"/>
 </parts>
 <sheets>
@@
 <text x="-67.564" y="71.628" size="1.778" layer="91" rot="R180">5V</text>
 <text x="-67.31" y="79.756" size="1.778" layer="91" rot="R180">EN</text>
-<text x="5.08" y="127" size="1.778" layer="91">5V Out EN - Recorder On/Off</text>
+<text x="22.86" y="137.16" size="1.778" layer="91">5V Out EN - Recorder On/Off</text>
 <text x="-65.024" y="46.482" size="1.778" layer="91" rot="R180">VBAT</text>
 <text x="-65.532" y="38.354" size="1.778" layer="91" rot="R180">GND</text>
@@
 <text x="-64.516" y="49.276" size="1.778" layer="91" rot="R180">VUSB</text>
 <text x="-66.294" y="43.688" size="1.778" layer="91" rot="R180">VS</text>
-<text x="93.98" y="127" size="1.778" layer="91">5V Out EN - Transmitter On/Off</text>
+<text x="93.98" y="137.16" size="1.778" layer="91">5V Out EN - Transmitter On/Off</text>
 <text x="147.32" y="132.08" size="1.778" layer="91">LIPO - FUEL GAUGE</text>
 <text x="190.5" y="132.08" size="1.778" layer="91">Solar Charger</text>
@@
 <attribute name="VALUE" x="-54.61" y="12.7" size="1.778" layer="96" rot="R180"/>
 </instance>
-<instance part="GND3" gate="1" x="7.62" y="109.22" smashed="yes">
-<attribute name="VALUE" x="5.08" y="106.68" size="1.778" layer="96"/>
+<instance part="GND3" gate="1" x="20.32" y="111.76" smashed="yes">
+<attribute name="VALUE" x="17.78" y="109.22" size="1.778" layer="96"/>
 </instance>
 <instance part="REC_POWER" gate="G$1" x="-63.5" y="104.14" smashed="yes" rot="R180">
@@
 <attribute name="VALUE" x="144.78" y="40.64" size="1.778" layer="96"/>
 </instance>
-<instance part="GND1" gate="1" x="119.38" y="109.22" smashed="yes">
-<attribute name="VALUE" x="116.84" y="106.68" size="1.778" layer="96"/>
+<instance part="GND1" gate="1" x="96.52" y="111.76" smashed="yes">
+<attribute name="VALUE" x="93.98" y="109.22" size="1.778" layer="96"/>
 </instance>
 <instance part="C1" gate="G$1" x="121.92" y="73.66" smashed="yes">
@@
 <instance part="GND12" gate="1" x="162.56" y="-83.82" smashed="yes">
 <attribute name="VALUE" x="160.02" y="-86.36" size="1.778" layer="96"/>
-</instance>
-<instance part="REC_ON_OFF_SW" gate="G$1" x="15.24" y="116.84" smashed="yes">
-<attribute name="NAME" x="15.240940625" y="124.46188125" size="1.27046875" layer="95"/>
-<attribute name="VALUE" x="15.24053125" y="121.91893125" size="1.27026875" layer="96"/>
-</instance>
-<instance part="GSM_ON_OFF_SW" gate="G$1" x="106.68" y="116.84" smashed="yes">
-<attribute name="NAME" x="106.680940625" y="124.46188125" size="1.27046875" layer="95"/>
-<attribute name="VALUE" x="106.68053125" y="121.91893125" size="1.27026875" layer="96"/>
-</instance>
-<instance part="REC_SW" gate="G$1" x="-20.32" y="71.12" smashed="yes">
-<attribute name="NAME" x="-13.97" y="76.2" size="1.778" layer="95" align="center-left"/>
-<attribute name="VALUE" x="-13.97" y="66.04" size="1.778" layer="96" align="center-left"/>
 </instance>
 <instance part="T4" gate="G$1" x="-30.48" y="-71.12" smashed="yes">
@@
 <instance part="SOLAR_CHARGER" gate="G$1" x="198.12" y="121.92" smashed="yes">
 <attribute name="NAME" x="189.23" y="126.238" size="1.778" layer="95"/>
+</instance>
+<instance part="REC_ON_OFF_SW" gate="G$1" x="25.4" y="121.92" smashed="yes">
+<attribute name="NAME" x="29.21" y="132.08" size="1.778" layer="95" align="center-left"/>
+<attribute name="VALUE" x="24.13" y="127" size="1.778" layer="96" align="center-left"/>
+</instance>
+<instance part="GSM_ON_OFF_SW1" gate="G$1" x="101.6" y="121.92" smashed="yes">
+<attribute name="NAME" x="100.33" y="132.08" size="1.778" layer="95" align="center-left"/>
+<attribute name="VALUE" x="105.41" y="127" size="1.778" layer="96" align="center-left"/>
+</instance>
+<instance part="REC_SW1" gate="G$1" x="-10.16" y="71.12" smashed="yes">
+<attribute name="NAME" x="-15.241909375" y="76.20381875" size="1.801359375" layer="95"/>
+<attribute name="VALUE" x="-15.241809375" y="66.036390625" size="1.80128125" layer="96"/>
 </instance>
 </instances>
@@
 </segment>
 <segment>
-<wire x1="-20.32" y1="71.12" x2="-22.86" y2="71.12" width="0.1524" layer="91"/>
 <pinref part="GND4" gate="1" pin="GND"/>
 <wire x1="-22.86" y1="71.12" x2="-22.86" y2="66.04" width="0.1524" layer="91"/>
-<pinref part="REC_SW" gate="G$1" pin="NO_1"/>
+<pinref part="REC_SW1" gate="G$1" pin="1"/>
+<pinref part="REC_SW1" gate="G$1" pin="2"/>
+<wire x1="-15.24" y1="73.66" x2="-15.24" y2="71.12" width="0.1524" layer="91"/>
+<wire x1="-15.24" y1="71.12" x2="-15.24" y2="68.58" width="0.1524" layer="91"/>
+<wire x1="-22.86" y1="71.12" x2="-15.24" y2="71.12" width="0.1524" layer="91"/>
+<junction x="-15.24" y="71.12"/>
 </segment>
 <segment>
@@
 </segment>
 <segment>
-<wire x1="111.76" y1="119.38" x2="119.38" y2="119.38" width="0.1524" layer="91"/>
 <pinref part="GND1" gate="1" pin="GND"/>
-<wire x1="119.38" y1="119.38" x2="119.38" y2="111.76" width="0.1524" layer="91"/>
-<pinref part="GSM_ON_OFF_SW" gate="G$1" pin="1"/>
-</segment>
-<segment>
-<wire x1="12.7" y1="116.84" x2="7.62" y2="116.84" width="0.1524" layer="91"/>
+<wire x1="96.52" y1="119.38" x2="96.52" y2="114.3" width="0.1524" layer="91"/>
+<pinref part="GSM_ON_OFF_SW1" gate="G$1" pin="COM"/>
+<wire x1="96.52" y1="119.38" x2="101.6" y2="119.38" width="0.1524" layer="91"/>
+</segment>
+<segment>
+<wire x1="25.4" y1="119.38" x2="20.32" y2="119.38" width="0.1524" layer="91"/>
 <pinref part="GND3" gate="1" pin="GND"/>
-<wire x1="7.62" y1="116.84" x2="7.62" y2="111.76" width="0.1524" layer="91"/>
-<pinref part="REC_ON_OFF_SW" gate="G$1" pin="2"/>
+<wire x1="20.32" y1="119.38" x2="20.32" y2="114.3" width="0.1524" layer="91"/>
+<pinref part="REC_ON_OFF_SW" gate="G$1" pin="COM"/>
 </segment>
 <segment>
@@
 <pinref part="U$1" gate="G$1" pin="4/PWM/SDA2/CAN0RX"/>
 <wire x1="30.48" y1="76.2" x2="10.16" y2="76.2" width="0.1524" layer="91"/>
-<wire x1="7.62" y1="71.12" x2="10.16" y2="71.12" width="0.1524" layer="91"/>
 <wire x1="10.16" y1="71.12" x2="10.16" y2="76.2" width="0.1524" layer="91"/>
-<pinref part="REC_SW" gate="G$1" pin="NO_2"/>
 <label x="10.16" y="76.2" size="1.778" layer="95"/>
+<pinref part="REC_SW1" gate="G$1" pin="4"/>
+<pinref part="REC_SW1" gate="G$1" pin="3"/>
+<wire x1="-2.54" y1="73.66" x2="-2.54" y2="71.12" width="0.1524" layer="91"/>
+<wire x1="-2.54" y1="71.12" x2="-2.54" y2="68.58" width="0.1524" layer="91"/>
+<wire x1="-2.54" y1="71.12" x2="10.16" y2="71.12" width="0.1524" layer="91"/>
+<junction x="-2.54" y="71.12"/>
 </segment>
 <segment>
@@
 </segment>
 <segment>
-<wire x1="20.32" y1="119.38" x2="45.72" y2="119.38" width="0.1524" layer="91"/>
-<label x="35.56" y="119.38" size="1.778" layer="95"/>
+<wire x1="0" y1="121.92" x2="25.4" y2="121.92" width="0.1524" layer="91"/>
+<label x="0" y="121.92" size="1.778" layer="95"/>
 <pinref part="REC_ON_OFF_SW" gate="G$1" pin="1"/>
 </segment>
@@
 </segment>
 <segment>
-<wire x1="96.52" y1="116.84" x2="104.14" y2="116.84" width="0.1524" layer="91"/>
-<label x="86.36" y="116.84" size="1.778" layer="95"/>
-<pinref part="GSM_ON_OFF_SW" gate="G$1" pin="2"/>
+<label x="81.28" y="121.92" size="1.778" layer="95"/>
+<pinref part="GSM_ON_OFF_SW1" gate="G$1" pin="1"/>
+<wire x1="83.82" y1="121.92" x2="101.6" y2="121.92" width="0.1524" layer="91"/>
 </segment>
 </net>
@@
 <label x="-66.802" y="0.508" size="1.778" layer="95" rot="R180"/>
 <wire x1="30.48" y1="63.5" x2="12.7" y2="63.5" width="0.1524" layer="91"/>
-<label x="2.54" y="63.5" size="1.778" layer="95"/>
+<label x="12.7" y="63.5" size="1.778" layer="95"/>
 </segment>
 <segment>
@@
 <pinref part="U$1" gate="G$1" pin="13/LED/ALT-PWM/SCK0"/>
 <label x="-66.294" y="3.048" size="1.778" layer="95" rot="R180"/>
-<label x="2.54" y="53.34" size="1.778" layer="95"/>
-<wire x1="30.48" y1="53.34" x2="10.16" y2="53.34" width="0.1524" layer="91"/>
-</segment>
-<segment>
+<label x="12.7" y="53.34" size="1.778" layer="95"/>
+<wire x1="30.48" y1="53.34" x2="12.7" y2="53.34" width="0.1524" layer="91"/>
+</segment>
+<segment>

Commit message: Power section shifted to one side along with LED's shifted downand track width increased
Parts:
- removed GSM_ON_OFF_SW1: GSM Power, EG1218:EG1218
- removed GSM_POWER_JUMPER: (no value), jumper:JP1Q
- removed REC_ON_OFF_SW: Microcontroller and Mic Power, EG1218:EG1218
- removed REC_POWER: (no value), adafruit:JST_2PIN-SMT-RA
- removed TEENSY_2, TEENSY_3, TEENSY_4, TEENSY_6, TEENSY_7, TEENSY_8, WILDLY_5V_0.5A_BOOST: (no value), adafruit:PINHD-1X6
- added 5V_INPUT: 61300211121, 61300211121:61300211121
- added BATT: (no value), adafruit:JST_2PIN-SMT-RA
- added JP1: (no value), jumper:JP1Q
- added ON_OFF_SW: GSM Power, EG1218:EG1218
- added TEENSY_PIN_2, TEENSY_PIN_3, TEENSY_PIN_4, TEENSY_PIN_6, TEENSY_PIN_7, TEENSY_PIN_8: (no value), adafruit:PINHD-1X6
- renumbered TEENSY_1 to TEENSY_PIN_1, TEENSY_5 to TEENSY_PIN_5
Connections:
- net GSM_LB renamed LB
- removed net A4: J1.1, TEENSY_6.3, U$1.18/A4/PWM/T/SDA0
- removed net A5: J1.2, TEENSY_6.2, U$1.19/A5/PWM/T/SCL0
- removed net GSM_5V: C3.1, C4.1, GSM_POWER_JUMPER.1, MIKROELECTRONIKA_SARA_CLICK.5V, WILDLY_5V_1A_BOOST.1
- removed net GSM_5V_EN: GSM_ON_OFF_SW1.1, WILDLY_5V_1A_BOOST.5
- removed net GSM_BAT: FUEL_GAUGE.2, SOLAR_CHARGER.1, WILDLY_5V_1A_BOOST.7
- removed net GSM_BAT_RETURN: FUEL_GAUGE.1, SOLAR_CHARGER.2, WILDLY_5V_1A_BOOST.4
- removed net REC_5V: C1.1, C2.1, GSM_POWER_JUMPER.2, TEENSY_PIN_5.1, U$1.VIN, WILDLY_5V_0.5A_BOOST.1
- removed net REC_5V_EN: REC_ON_OFF_SW.1, WILDLY_5V_0.5A_BOOST.4
- removed net REC_BAT: REC_POWER.2, WILDLY_5V_0.5A_BOOST.6
- removed net REC_BAT_RETURN: REC_POWER.1, WILDLY_5V_0.5A_BOOST.5
- removed net REC_LB: WILDLY_5V_0.5A_BOOST.3
- new net 5V_EN: ON_OFF_SW.1, WILDLY_5V_1A_BOOST.5
- new net 5V_SUPPLY: 5V_INPUT.1, C1.1, C2.1, C3.1, C4.1, MIKROELECTRONIKA_SARA_CLICK.5V, TEENSY_PIN_5.1, U$1.VIN, WILDLY_5V_1A_BOOST.1
- new net FUEL_GAUGE_SCL: J1.2, TEENSY_PIN_6.2, U$1.19/A5/PWM/T/SCL0
- new net FUEL_GAUGE_SDA: J1.1, TEENSY_PIN_6.3, U$1.18/A4/PWM/T/SDA0
- new net VCC: BATT.2, FUEL_GAUGE.2, SOLAR_CHARGER.1, WILDLY_5V_1A_BOOST.7
- net 25: now also TEENSY_PIN_3.5; no longer TEENSY_3.5
- net 3V3: now also JP1.1, JP1.2, TEENSY_PIN_3.3; no longer TEENSY_3.3
- net A0: now also TEENSY_PIN_7.1; no longer TEENSY_7.1
- net A1: now also TEENSY_PIN_6.6; no longer TEENSY_6.6
- net A2: now also TEENSY_PIN_6.5; no longer TEENSY_6.5
- net A3: now also TEENSY_PIN_6.4; no longer TEENSY_6.4
- net ALT-MOSI: now also TEENSY_PIN_4.2; no longer TEENSY_4.2
- net ALT-PWM: now also TEENSY_PIN_3.6; no longer TEENSY_3.6
- net ALT-RX1: now also TEENSY_PIN_4.1; no longer TEENSY_4.1
- net CTS_OF_GSM: now also TEENSY_PIN_8.6; no longer TEENSY_8.6
- net DAC0: now also TEENSY_PIN_7.5; no longer TEENSY_7.5
- net DAC1: now also TEENSY_PIN_7.4; no longer TEENSY_7.4
- net ERRLED: now also TEENSY_PIN_7.6; no longer TEENSY_7.6
- net GND: now also 5V_INPUT.2, BATT.1, FUEL_GAUGE.1, ON_OFF_SW.COM, SOLAR_CHARGER.2, TEENSY_PIN_7.3, WILDLY_5V_1A_BOOST.4; no longer GSM_ON_OFF_SW1.COM, REC_ON_OFF_SW.COM, TEENSY_7.3, WILDLY_5V_0.5A_BOOST.2
- net MIC_BCLK: now also TEENSY_PIN_2.5; no longer TEENSY_2.5
- net MIC_DOUT: now also TEENSY_PIN_7.2; no longer TEENSY_7.2
- net MISO: now also TEENSY_PIN_3.2; no longer TEENSY_3.2
- net MOSI: now also TEENSY_PIN_3.1; no longer TEENSY_3.1
- net NETSTATLED: now also TEENSY_PIN_8.1; no longer TEENSY_8.1
- net NET_STAT: now also TEENSY_PIN_3.4; no longer TEENSY_3.4
- net POWER_CONTRL: now also TEENSY_PIN_8.4; no longer TEENSY_8.4
- net PWM10: now also TEENSY_PIN_4.4; no longer TEENSY_4.4
- net PWM11: now also TEENSY_PIN_4.5; no longer TEENSY_4.5
- net PWM12: now also TEENSY_PIN_4.6; no longer TEENSY_4.6
- net PWM4: now also TEENSY_PIN_2.1; no longer TEENSY_2.1
- net PWM5: now also TEENSY_PIN_2.2; no longer TEENSY_2.2
- net PWM6: now also TEENSY_PIN_2.3; no longer TEENSY_2.3
- net PWM7: now also TEENSY_PIN_2.4; no longer TEENSY_2.4
- net PWM8: now also TEENSY_PIN_2.6; no longer TEENSY_2.6
- net PWM9: now also TEENSY_PIN_4.3; no longer TEENSY_4.3
- net RECLED: now also TEENSY_PIN_8.3; no longer TEENSY_8.3
- net RESET_GSM: now also TEENSY_PIN_6.1; no longer TEENSY_6.1
- net RTS_OF_GSM: now also TEENSY_PIN_8.5; no longer TEENSY_8.5
- net SDLED: now also TEENSY_PIN_8.2; no longer TEENSY_8.2
Other:
- note added: "5V - SUPPLY"
- note added: "LiPo Battery Connector"
- note removed: "5V Out EN - Recorder On/Off"
- note removed: "Adafruit 5V Boost 500mA"
- note removed: "Bat"
- moved on the sheet: FUEL_GAUGE, SOLAR_CHARGER, WILDLY_5V_1A_BOOST, WILDLY_I2S_MIC

Commit message: Added new transistor BC847 along with some 0R reistors
Parts:
- added R4, R5, R6: 0R, adafruit:R-US_M0805
- T1, T2, T3, T4: value 2N2222A -> BC847BLT1G; device 2N2222A:2N2222A -> BC847BLT1G:BC847BLT1G
Connections:
- net 5V_SUPPLY: now also R4.1, R4.2
- net RX_OF_GSM: now also R5.1, R5.2
- net TX_OF_GSM: now also R6.1, R6.2
Other:
- note added: "Note - When powering the board from boost R4 = 0 ohm should be mounted"
- moved on the sheet: JP1, R13, R2, R3, R9

Commit message: Changed all the power symbols to +5V and 3V3 accordingly
Connections:
- new net +3V3: JP1.1, R10.2, R11.2, R12.2, R14.2
- new net +5V: 5V_INPUT.1, C1.1, C2.1, C3.1, C4.1, MIKROELECTRONIKA_SARA_CLICK.5V, R4.1, TEENSY_PIN_5.1, U$1.VIN
- net 3V3: no longer JP1.1, R10.2, R11.2, R12.2, R14.2
- net 5V_SUPPLY: no longer 5V_INPUT.1, C1.1, C2.1, C3.1, C4.1, MIKROELECTRONIKA_SARA_CLICK.5V, R4.1, TEENSY_PIN_5.1, U$1.VIN

Commit message: Positioning of filter capacitors along with connections corrected
Parts:
- BATT: value (none) -> B2B-PH-SM4-TB(LF)(SN); device adafruit:JST_2PIN-SMT-RA -> B2B-PH-SM4-TB_LF__SN_:B2B-PH-SM4-TB(LF)(SN)
Connections:
- removed net A3: TEENSY_PIN_6.4, U$1.17/A3/PWM/T/ALT-SDA0
- new net PWM_SARA: MIKROELECTRONIKA_SARA_CLICK.PWM, TEENSY_PIN_6.4, U$1.17/A3/PWM/T/ALT-SDA0
Other:
- moved on the sheet: BATT
Changed lines of the file:
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@@
 <part name="WILDLY_5V_1A_BOOST" library="adafruit" library_urn="urn:adsk.eagle:library:420" deviceset="PINHD-1X8" device="BIG" package3d_urn="urn:adsk.eagle:package:6240707/1"/>
 <part name="WILDLY_I2S_MIC" library="adafruit" library_urn="urn:adsk.eagle:library:420" deviceset="PINHD-1X6" device="" package3d_urn="urn:adsk.eagle:package:6240711/1"/>
-<part name="BATT" library="adafruit" library_urn="urn:adsk.eagle:library:420" deviceset="JST_2PIN" device="-SMT-RA" package3d_urn="urn:adsk.eagle:package:6240692/1"/>
 <part name="GND4" library="supply1" library_urn="urn:adsk.eagle:library:371" deviceset="GND" device=""/>
 <part name="GND5" library="supply1" library_urn="urn:adsk.eagle:library:371" deviceset="GND" device=""/>
@@
 <part name="+3V8" library="supply1" library_urn="urn:adsk.eagle:library:371" deviceset="+3V3" device=""/>
 <part name="+3V9" library="supply1" library_urn="urn:adsk.eagle:library:371" deviceset="+3V3" device=""/>
+<part name="GND17" library="supply1" library_urn="urn:adsk.eagle:library:371" deviceset="GND" device=""/>
+<part name="BATT" library="B2B-PH-SM4-TB_LF__SN_" deviceset="B2B-PH-SM4-TB(LF)(SN)" device=""/>
 </parts>
 <sheets>
@@
 <attribute name="VALUE" x="-69.85" y="20.32" size="1.778" layer="96" rot="R180"/>
 </instance>
-<instance part="BATT" gate="G$1" x="-78.74" y="134.62" smashed="yes" rot="R180">
-<attribute name="NAME" x="-67.31" y="128.905" size="1.778" layer="95" rot="R180"/>
-<attribute name="VALUE" x="-72.39" y="139.7" size="1.778" layer="96" rot="R180"/>
-</instance>
 <instance part="GND4" gate="1" x="-22.86" y="63.5" smashed="yes">
 <attribute name="VALUE" x="-25.4" y="60.96" size="1.778" layer="96"/>
@@
 <instance part="+3V9" gate="G$1" x="162.56" y="-30.48" smashed="yes">
 <attribute name="VALUE" x="160.02" y="-35.56" size="1.778" layer="96" rot="R90"/>
+</instance>
+<instance part="GND17" gate="1" x="-38.1" y="-2.54" smashed="yes">
+<attribute name="VALUE" x="-40.64" y="-5.08" size="1.778" layer="96"/>
+</instance>
+<instance part="BATT" gate="G$1" x="-78.74" y="132.08" smashed="yes" rot="R180">
+<attribute name="NAME" x="-76.19638125" y="129.027659375" size="1.271809375" layer="95" rot="R180"/>
 </instance>
 </instances>
@@
 <segment>
 <pinref part="WILDLY_I2S_MIC" gate="A" pin="2"/>
-<wire x1="-73.66" y1="5.08" x2="-58.42" y2="5.08" width="0.1524" layer="91"/>
-<label x="-58.42" y="5.08" size="1.778" layer="95"/>
+<wire x1="-73.66" y1="5.08" x2="-38.1" y2="5.08" width="0.1524" layer="91"/>
+<pinref part="GND17" gate="1" pin="GND"/>
+<wire x1="-38.1" y1="5.08" x2="-38.1" y2="0" width="0.1524" layer="91"/>
 </segment>
 <segment>
@@
 </segment>
 <segment>
-<pinref part="BATT" gate="G$1" pin="1"/>
-<wire x1="-76.2" y1="132.08" x2="-63.5" y2="132.08" width="0.1524" layer="91"/>
+<wire x1="-73.66" y1="132.08" x2="-63.5" y2="132.08" width="0.1524" layer="91"/>
 <wire x1="-63.5" y1="132.08" x2="-63.5" y2="121.92" width="0.1524" layer="91"/>
 <pinref part="GND3" gate="1" pin="GND"/>
+<pinref part="BATT" gate="G$1" pin="1"/>
 </segment>
 <segment>
@@
 <segment>
 <pinref part="U$1" gate="G$1" pin="33/A14/CAN1TX/TX5/ALT-SCL0"/>
-<wire x1="30.48" y1="2.54" x2="-2.54" y2="2.54" width="0.1524" layer="91"/>
+<wire x1="30.48" y1="2.54" x2="0" y2="2.54" width="0.1524" layer="91"/>
 <label x="0" y="2.54" size="1.778" layer="95"/>
 </segment>
@@
 <segment>
 <pinref part="U$1" gate="G$1" pin="39/A20/ALT-MISO0"/>
-<wire x1="99.06" y1="0" x2="121.92" y2="0" width="0.1524" layer="91"/>
+<wire x1="99.06" y1="0" x2="119.38" y2="0" width="0.1524" layer="91"/>
 <label x="101.6" y="0" size="1.778" layer="95"/>
 </segment>
@@
 </segment>
 </net>
-<net name="A3" class="0">
-<segment>
-<pinref part="U$1" gate="G$1" pin="17/A3/PWM/T/ALT-SDA0"/>
-<wire x1="30.48" y1="43.18" x2="12.7" y2="43.18" width="0.1524" layer="91"/>
-<label x="12.7" y="43.18" size="1.778" layer="95"/>
-</segment>
-<segment>
-<pinref part="TEENSY_PIN_6" gate="A" pin="4"/>
-<wire x1="182.88" y1="-15.24" x2="167.64" y2="-15.24" width="0.1524" layer="91"/>
-<label x="167.64" y="-15.24" size="1.778" layer="95"/>
-</segment>
-</net>
 <net name="PWM13" class="0">
 <segment>
@@
 <net name="VCC" class="0">
 <segment>
-<pinref part="BATT" gate="G$1" pin="2"/>
-<wire x1="-76.2" y1="134.62" x2="-45.72" y2="134.62" width="0.1524" layer="91"/>
+<wire x1="-73.66" y1="134.62" x2="-45.72" y2="134.62" width="0.1524" layer="91"/>
 <pinref part="P+1" gate="VCC" pin="VCC"/>
 <wire x1="-45.72" y1="134.62" x2="-45.72" y2="139.7" width="0.1524" layer="91"/>
+<pinref part="BATT" gate="G$1" pin="2"/>
 </segment>
 <segment>
@@
 </segment>
 </net>
+<net name="PWM_SARA" class="0">
+<segment>
+<pinref part="U$1" gate="G$1" pin="17/A3/PWM/T/ALT-SDA0"/>
+<wire x1="30.48" y1="43.18" x2="12.7" y2="43.18" width="0.1524" layer="91"/>
+<label x="2.54" y="43.18" size="1.778" layer="95"/>
+</segment>
+<segment>
+<pinref part="TEENSY_PIN_6" gate="A" pin="4"/>
+<wire x1="182.88" y1="-15.24" x2="167.64" y2="-15.24" width="0.1524" layer="91"/>
+<label x="167.64" y="-15.24" size="1.778" layer="95"/>
+</segment>
+<segment>
+<pinref part="MIKROELECTRONIKA_SARA_CLICK" gate="G$1" pin="PWM"/>
+<wire x1="193.04" y1="91.44" x2="205.74" y2="91.44" width="0.1524" layer="91"/>
+<label x="198.12" y="91.44" size="1.778" layer="95"/>
+</segment>
+</net>

Commit message: Move capacitors and resistors in layout according to flow of signal as in schematics, rename net names, increase mount hole diameters
Connections:
- new net N$10: MIKROELECTRONIKA_SARA_CLICK.RX, R5.2
- new net N$12: MIKROELECTRONIKA_SARA_CLICK.TX, R6.2
- net RX_OF_GSM: no longer MIKROELECTRONIKA_SARA_CLICK.RX, R5.2
- net TX_OF_GSM: no longer MIKROELECTRONIKA_SARA_CLICK.TX, R6.2
Changed lines of the file:
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@@
-</segment>
-<segment>
-<pinref part="MIKROELECTRONIKA_SARA_CLICK" gate="G$1" pin="TX"/>
-<wire x1="193.04" y1="76.2" x2="203.2" y2="76.2" width="0.1524" layer="91"/>
-<pinref part="R6" gate="G$1" pin="2"/>
 </segment>
 <segment>
@@
 <segment>
 <pinref part="R6" gate="G$1" pin="1"/>
-<wire x1="213.36" y1="76.2" x2="228.6" y2="76.2" width="0.1524" layer="91"/>
+<wire x1="213.36" y1="76.2" x2="220.98" y2="76.2" width="0.1524" layer="91"/>
 <label x="215.9" y="76.2" size="1.778" layer="95"/>
 </segment>
@@
 </segment>
 <segment>
-<pinref part="MIKROELECTRONIKA_SARA_CLICK" gate="G$1" pin="RX"/>
-<wire x1="193.04" y1="81.28" x2="203.2" y2="81.28" width="0.1524" layer="91"/>
-<pinref part="R5" gate="G$1" pin="2"/>
-</segment>
-<segment>
 <pinref part="TEENSY_PIN_1" gate="A" pin="3"/>
 <wire x1="147.32" y1="17.78" x2="132.08" y2="17.78" width="0.1524" layer="91"/>
@@
 <segment>
 <pinref part="R5" gate="G$1" pin="1"/>
-<wire x1="213.36" y1="81.28" x2="228.6" y2="81.28" width="0.1524" layer="91"/>
+<wire x1="213.36" y1="81.28" x2="220.98" y2="81.28" width="0.1524" layer="91"/>
 <label x="215.9" y="81.28" size="1.778" layer="95"/>
 </segment>
@@
 </segment>
 </net>
+<net name="N$10" class="0">
+<segment>
+<pinref part="MIKROELECTRONIKA_SARA_CLICK" gate="G$1" pin="RX"/>
+<pinref part="R5" gate="G$1" pin="2"/>
+<wire x1="193.04" y1="81.28" x2="203.2" y2="81.28" width="0.1524" layer="91"/>
+</segment>
+</net>
+<net name="N$12" class="0">
+<segment>
+<pinref part="MIKROELECTRONIKA_SARA_CLICK" gate="G$1" pin="TX"/>
+<pinref part="R6" gate="G$1" pin="2"/>
+<wire x1="193.04" y1="76.2" x2="203.2" y2="76.2" width="0.1524" layer="91"/>
+</segment>
+</net>
