File: Teensy36_I2S_Proto/wildly_teensy_proto.sch (EAGLE design)
At the start: 45 parts, among them J1 61300311121, J2 61300311121, T1 BC847BLT1G, T2 BC847BLT1G, T3 BC847BLT1G, T4 BC847BLT1G

Commit message: Rx and Tx connections interchanged and positioning of fuel gauge adjusted
Connections:
- net RX_OF_GSM: now also R6.1; no longer R5.1
- net TX_OF_GSM: now also R5.1; no longer R6.1
Other:
- moved on the sheet: R5, R6
Changed lines of the file:
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@@
 <part name="T2" library="BC847BLT1G" deviceset="BC847BLT1G" device=""/>
 <part name="R4" library="adafruit" library_urn="urn:adsk.eagle:library:420" deviceset="R-US_" device="M0805" package3d_urn="urn:adsk.eagle:package:6240587/1" value="0R"/>
-<part name="R5" library="adafruit" library_urn="urn:adsk.eagle:library:420" deviceset="R-US_" device="M0805" package3d_urn="urn:adsk.eagle:package:6240587/1" value="0R"/>
-<part name="R6" library="adafruit" library_urn="urn:adsk.eagle:library:420" deviceset="R-US_" device="M0805" package3d_urn="urn:adsk.eagle:package:6240587/1" value="0R"/>
 <part name="GND16" library="supply1" library_urn="urn:adsk.eagle:library:371" deviceset="GND" device=""/>
 <part name="P+5" library="supply1" library_urn="urn:adsk.eagle:library:371" deviceset="+5V" device=""/>
@@
 <part name="GND17" library="supply1" library_urn="urn:adsk.eagle:library:371" deviceset="GND" device=""/>
 <part name="BATT" library="B2B-PH-SM4-TB_LF__SN_" deviceset="B2B-PH-SM4-TB(LF)(SN)" device=""/>
+<part name="R5" library="adafruit" library_urn="urn:adsk.eagle:library:420" deviceset="R-US_" device="M0805" package3d_urn="urn:adsk.eagle:package:6240587/1" value="0R"/>
+<part name="R6" library="adafruit" library_urn="urn:adsk.eagle:library:420" deviceset="R-US_" device="M0805" package3d_urn="urn:adsk.eagle:package:6240587/1" value="0R"/>
 </parts>
 <sheets>
@@
 <attribute name="VALUE" x="-49.53" y="56.642" size="1.778" layer="96" rot="R180"/>
 </instance>
-<instance part="R5" gate="G$1" x="208.28" y="81.28" smashed="yes" rot="R180">
-<attribute name="NAME" x="204.47" y="79.7814" size="1.778" layer="95" rot="R180"/>
-<attribute name="VALUE" x="214.63" y="79.502" size="1.778" layer="96" rot="R180"/>
-</instance>
-<instance part="R6" gate="G$1" x="208.28" y="76.2" smashed="yes" rot="R180">
-<attribute name="NAME" x="204.47" y="74.7014" size="1.778" layer="95" rot="R180"/>
-<attribute name="VALUE" x="214.63" y="74.422" size="1.778" layer="96" rot="R180"/>
-</instance>
 <instance part="GND16" gate="1" x="114.3" y="10.16" smashed="yes">
 <attribute name="VALUE" x="111.76" y="7.62" size="1.778" layer="96"/>
@@
 <instance part="BATT" gate="G$1" x="-78.74" y="132.08" smashed="yes" rot="R180">
 <attribute name="NAME" x="-76.19638125" y="129.027659375" size="1.271809375" layer="95" rot="R180"/>
+</instance>
+<instance part="R5" gate="G$1" x="207.518" y="81.28" smashed="yes" rot="R180">
+<attribute name="NAME" x="204.47" y="79.7814" size="1.778" layer="95" rot="R180"/>
+<attribute name="VALUE" x="211.836" y="79.756" size="1.778" layer="96" rot="R180"/>
+</instance>
+<instance part="R6" gate="G$1" x="207.772" y="76.2" smashed="yes" rot="R180">
+<attribute name="NAME" x="204.724" y="74.7014" size="1.778" layer="95" rot="R180"/>
+<attribute name="VALUE" x="212.09" y="74.676" size="1.778" layer="96" rot="R180"/>
 </instance>
 </instances>
@@
 </segment>
 <segment>
-<pinref part="R6" gate="G$1" pin="1"/>
-<wire x1="213.36" y1="76.2" x2="220.98" y2="76.2" width="0.1524" layer="91"/>
-<label x="215.9" y="76.2" size="1.778" layer="95"/>
+<pinref part="R5" gate="G$1" pin="1"/>
+<wire x1="212.598" y1="81.28" x2="223.52" y2="81.28" width="0.1524" layer="91"/>
+<label x="215.9" y="81.28" size="1.778" layer="95"/>
 </segment>
 </net>
@@
 </segment>
 <segment>
-<pinref part="R5" gate="G$1" pin="1"/>
-<wire x1="213.36" y1="81.28" x2="220.98" y2="81.28" width="0.1524" layer="91"/>
-<label x="215.9" y="81.28" size="1.778" layer="95"/>
+<pinref part="R6" gate="G$1" pin="1"/>
+<wire x1="212.852" y1="76.2" x2="223.52" y2="76.2" width="0.1524" layer="91"/>
+<label x="215.9" y="76.2" size="1.778" layer="95"/>
 </segment>
 </net>
@@
 <pinref part="MIKROELECTRONIKA_SARA_CLICK" gate="G$1" pin="RX"/>
 <pinref part="R5" gate="G$1" pin="2"/>
-<wire x1="193.04" y1="81.28" x2="203.2" y2="81.28" width="0.1524" layer="91"/>
-</segment>
-</net>
-<net name="N$12" class="0">
+<wire x1="193.04" y1="81.28" x2="202.438" y2="81.28" width="0.1524" layer="91"/>
+</segment>
+</net>
+<net name="N$17" class="0">
 <segment>
 <pinref part="MIKROELECTRONIKA_SARA_CLICK" gate="G$1" pin="TX"/>
 <pinref part="R6" gate="G$1" pin="2"/>
-<wire x1="193.04" y1="76.2" x2="203.2" y2="76.2" width="0.1524" layer="91"/>
-</segment>
-</net>
+<wire x1="193.04" y1="76.2" x2="202.692" y2="76.2" width="0.1524" layer="91"/>
+</segment>
+</net>

Commit message: Added the fuel Gauge circuit on board and rearranged the Transistors for grouping and short routing to the LEDs
Parts:
- removed FUEL_GAUGE: 61300211121, 61300211121:61300211121
- removed J1, J2: 61300311121, 61300311121:61300311121
- added C5: 1uF, rcl:C-EUC0805
- added C6: 10nF, rcl:C-EUC0805
- added IC1: MAX17043G+T, MAX17043G+T:MAX17043G+T
- added R15, R16: 4.7K, adafruit:R-US_M0805
- added R17, R18: 0R, adafruit:R-US_M0805
- added R7: 1K, adafruit:R-US_M0805
- added R8: 180R, adafruit:R-US_M0805
- R10, R11, R12, R14: value 82R -> 870R
- renumbered ON_OFF_SW to SWITCH
Connections:
- removed net N$13: J1.3
- new net FUEL_GAUGE_ALT: IC1.!ALRT
- new net FUEL_GAUGE_QST: IC1.QSTRT
- new net N$12: C5.1, IC1.CELL, R7.1
- new net N$18: C6.1, IC1.VDD, R8.2
- new net SCL: IC1.SCL, R16.2, R18.1
- new net SDA: IC1.SDA, R15.2, R17.1
- net FUEL_GAUGE_SCL: now also R18.2; no longer J1.2
- net FUEL_GAUGE_SDA: now also R17.2; no longer J1.1
- net GND: now also BATT.2, C5.2, C6.2, IC1.CTG, IC1.EP, IC1.GND; no longer BATT.1, FUEL_GAUGE.1
- net VCC: now also BATT.1, R15.1, R16.1, R7.2, R8.1; no longer BATT.2, FUEL_GAUGE.2
Other:
- note added: "Fuel Gauge"
- note removed: "LIPO - FUEL GAUGE"
- moved on the sheet: SOLAR_CHARGER
