File: Teensy36_I2S_Proto/wildly_teensy_proto.brd (EAGLE design)
At the start: 100 x 85.1 mm, 22 parts, among them CON1 MIKROE_BUS_CONN, SW1 SPST_TACT-KMR2, X1 ANTENNA

Commit message: Remove extra SMA connector
Parts:
- removed X1: ANTENNA, adafruit:SMA90_DIP
- moved CON1 18.2 mm to (12.7, 7.62), turned to 90 degrees
Connections:
- removed net GND1: X1.GND1
- removed net GND2: X1.GND2
- removed net GND3: X1.GND3
- removed net GND4: X1.GND4
- removed net N$1: CON1.P$1, X1.ANTENNA
Routing:
- net N$2: track 0.00 -> 24.4 mm
Changed lines of the file:
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@@
 <?xml version="1.0" encoding="utf-8"?>
 <!DOCTYPE eagle SYSTEM "eagle.dtd">
-<eagle version="9.2.2">
+<eagle version="9.3.0">
 <drawing>
 <settings>
@@
 </autorouter>
 <elements>
-<element name="CON1" library="mikrobus_lib" package="MIKROBUS_HOST_CONN" value="MIKROE_BUS_CONN" x="5.08" y="24.13" smashed="yes"/>
+<element name="CON1" library="mikrobus_lib" package="MIKROBUS_HOST_CONN" value="MIKROE_BUS_CONN" x="12.7" y="7.62" smashed="yes" rot="R90"/>
 <element name="JP1" library="adafruit" library_urn="urn:adsk.eagle:library:420" package="1X06" package3d_urn="urn:adsk.eagle:package:6240711/1" value="" x="11.43" y="50.8" smashed="yes" rot="R90">
 <attribute name="NAME" x="9.6012" y="43.1038" size="1.27" layer="25" ratio="10" rot="R90"/>
@@
 </element>
 <element name="U$1" library="Teensy_3_6" package="T36" value="TEENSY3_6--ALLPINS" x="46.99" y="46.99" smashed="yes"/>
-<element name="X1" library="adafruit" library_urn="urn:adsk.eagle:library:420" package="SMA90_DIP" package3d_urn="urn:adsk.eagle:package:6240946/1" value="ANTENNA" x="8.89" y="74.93" smashed="yes">
-<attribute name="NAME" x="6.858" y="79.756" size="0.8128" layer="25" ratio="18"/>
-<attribute name="VALUE" x="6.858" y="78.994" size="0.4064" layer="27" ratio="10"/>
-</element>
 </elements>
 <signals>
-<signal name="GND1">
-<contactref element="X1" pad="GND1"/>
-</signal>
-<signal name="GND2">
-<contactref element="X1" pad="GND2"/>
-</signal>
-<signal name="GND3">
-<contactref element="X1" pad="GND3"/>
-</signal>
-<signal name="GND4">
-<contactref element="X1" pad="GND4"/>
-</signal>
-<signal name="N$1">
-<contactref element="CON1" pad="P$1"/>
-<contactref element="X1" pad="ANTENNA"/>
-<wire x1="5.08" y1="24.13" x2="8.89" y2="74.93" width="0" layer="19" extent="1-1"/>
-</signal>
 <signal name="3V">
 <contactref element="JP3" pad="1"/>
@@
 <contactref element="U$1" pad="5V"/>
 <contactref element="JP1" pad="1"/>
-<wire x1="35.56" y1="45.085" x2="11.43" y2="44.45" width="0" layer="19" extent="1-1"/>
+<wire x1="11.43" y1="44.45" x2="34.925" y2="44.45" width="0.1524" layer="1"/>
+<wire x1="34.925" y1="44.45" x2="35.56" y2="45.085" width="0.1524" layer="1"/>
 </signal>
 <signal name="N$3">

Commit message: Add more connections and adjust layour inlcude room for board fitting
Parts:
- added CN1, CN2: (no value), adafruit:JST-PH-2-SMT-RA
- added LOWBATLED, LOWBATLED1: (no value), adafruit:CHIP-LED0805
- added R9: 330R, adafruit:M0805
- added S1, S2: (no value), adafruit:B3F-31XX-SKINNIER
- R1: value (none) -> 1KR
- R3, R4, R5, R6, R7, R8: value (none) -> 330R
- moved CON1 48.3 mm to (61.0, 5.08)
- moved JP2 47.3 mm to (7.62, 11.4), turned to 90 degrees
- moved JP1 5.39 mm to (7.62, 54.6)
- moved U$1 4.02 mm to (45.7, 50.8)
- renumbered LED1 to RECLED, LED2 to SDLED, LED3 to NETSTATLED, LED4 to ERRLED, LED5 to POWERLED
Connections:
- removed net N$6: R5.2, U$1.37
- new net N$1: SW2.P$2, U$1.4
- new net N$10: JP1.3, R3.1
- new net N$16: LOWBATLED.A, R3.2
- new net N$17: CN1.2
- new net N$19: JP2.5, S2.2
- new net N$20: JP2.3, R9.1
- new net N$21: U$1.38
- new net N$23: LOWBATLED1.A, R9.2
- new net N$24: CN2.1, JP2.7
- new net N$25: CON1.P$10, JP2.1
- new net N$3: CN1.1, JP1.6
- net CTS_OF_GSM: now also CON1.P$3, R1.2
- net GND: now also CN2.2, CON1.P$8, CON1.P$9, JP2.2, JP2.4, LOWBATLED.C, LOWBATLED1.C, R1.1, S1.2, S2.1, SW2.P$1
- net N$4: now also S1.1
- net N$7: no longer U$1.38
- net N$8: no longer U$1.39
- net RESET_GSM: now also CON1.P$2
- net RTS_OF_GSM: now also CON1.P$15
- net RX_OF_GSM: now also CON1.P$14
- net TX_OF_GSM: now also CON1.P$13
Routing:
- net N$2: track 24.4 -> 26.9 mm
Other:
- board text added: "Adafruit 5V Boost 1A"
- board text added: "Battery Connector"
- board text added: "Teensy 3.6"

Commit message: Tidy up and complete schematics for review
Parts:
- removed LED6: RGBLED5050, adafruit:RGBLED5050
- removed R2: (no value), adafruit:M0805
- removed SW1: SPST_TACT-KMR2, adafruit:KMR2
- S1: value (none) -> Microcontroller and Mic power
- S2: value (none) -> GSM power
- SW2: value (none) -> Push_Button
- renumbered LOWBATLED to REC_LOW_BAT_LED, LOWBATLED1 to GSM_LOW_BAT_LED
Connections:
- net N$11: now also ERRLED.A, R8.2; no longer NETSTATLED.A, R7.1
- net N$12: now also U$1.39; no longer SDLED.A
- net N$14: now also U$1.37; no longer ERRLED.A
- net N$21: now also R7.1
- net N$7: now also NETSTATLED.A
- net N$8: now also R5.2, SDLED.A; no longer R8.2
Changed lines of the file:
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@@
 <?xml version="1.0" encoding="utf-8"?>
 <!DOCTYPE eagle SYSTEM "eagle.dtd">
-<eagle version="9.2.2">
+<eagle version="9.3.0">
 <drawing>
 <settings>
@@
 <attribute name="VALUE" x="-54.61" y="60.96" size="1.27" layer="27" rot="R90"/>
 </element>
-<element name="LED6" library="adafruit" library_urn="urn:adsk.eagle:library:420" package="RGBLED5050" package3d_urn="urn:adsk.eagle:package:6240865/1" value="RGBLED5050" x="-31.75" y="63.5" smashed="yes">
-<attribute name="NAME" x="-33.45" y="66.4" size="1.27" layer="25" font="vector"/>
-<attribute name="VALUE" x="-33.75" y="59.4" size="1.27" layer="27" font="vector"/>
-</element>
 <element name="R1" library="adafruit" library_urn="urn:adsk.eagle:library:420" package="M0805" package3d_urn="urn:adsk.eagle:package:6240587/1" value="1KR" x="-15.24" y="80.01" smashed="yes">
 <attribute name="NAME" x="-16.256" y="81.026" size="1.27" layer="25"/>
 <attribute name="VALUE" x="-16.256" y="77.724" size="1.27" layer="27"/>
 </element>
-<element name="R2" library="adafruit" library_urn="urn:adsk.eagle:library:420" package="M0805" package3d_urn="urn:adsk.eagle:package:6240587/1" value="" x="-20.32" y="80.01" smashed="yes">
-<attribute name="NAME" x="-21.336" y="81.026" size="1.27" layer="25"/>
-<attribute name="VALUE" x="-21.336" y="77.724" size="1.27" layer="27"/>
-</element>
 <element name="R3" library="adafruit" library_urn="urn:adsk.eagle:library:420" package="M0805" package3d_urn="urn:adsk.eagle:package:6240587/1" value="330R" x="-25.4" y="80.01" smashed="yes">
 <attribute name="NAME" x="-26.416" y="81.026" size="1.27" layer="25"/>
@@
 <attribute name="VALUE" x="-51.816" y="77.724" size="1.27" layer="27"/>
 </element>
-<element name="SW1" library="adafruit" library_urn="urn:adsk.eagle:library:420" package="KMR2" package3d_urn="urn:adsk.eagle:package:6240885/1" value="SPST_TACT-KMR2" x="-55.88" y="81.28" smashed="yes"/>
-<element name="SW2" library="adafruit" library_urn="urn:adsk.eagle:library:420" package="TACT_PANA-EVQ" package3d_urn="urn:adsk.eagle:package:6240957/1" value="" x="-66.04" y="60.96" smashed="yes">
+<element name="SW2" library="adafruit" library_urn="urn:adsk.eagle:library:420" package="TACT_PANA-EVQ" package3d_urn="urn:adsk.eagle:package:6240957/1" value="Push_Button" x="-66.04" y="60.96" smashed="yes">
 <attribute name="NAME" x="-69.083" y="63.13" size="0.8128" layer="25" ratio="18"/>
 <attribute name="VALUE" x="-69.056" y="58.509" size="0.4064" layer="27" ratio="10"/>
 </element>
 <element name="U$1" library="Teensy_3_6" package="T36" value="TEENSY3_6--ALLPINS" x="45.72" y="50.8" smashed="yes"/>
-<element name="LOWBATLED" library="adafruit" library_urn="urn:adsk.eagle:library:420" package="CHIP-LED0805" package3d_urn="urn:adsk.eagle:package:6240557/1" value="" x="-67.31" y="-16.51" smashed="yes">
+<element name="REC_LOW_BAT_LED" library="adafruit" library_urn="urn:adsk.eagle:library:420" package="CHIP-LED0805" package3d_urn="urn:adsk.eagle:package:6240557/1" value="" x="-67.31" y="-16.51" smashed="yes">
 <attribute name="NAME" x="-68.58" y="-17.78" size="1.27" layer="25" rot="R90"/>
 <attribute name="VALUE" x="-64.77" y="-17.78" size="1.27" layer="27" rot="R90"/>
 </element>
-<element name="S1" library="adafruit" library_urn="urn:adsk.eagle:library:420" package="B3F-31XX-SKINNIER" package3d_urn="urn:adsk.eagle:package:6240899/1" value="" x="15.24" y="73.66" smashed="yes" rot="R180">
+<element name="S1" library="adafruit" library_urn="urn:adsk.eagle:library:420" package="B3F-31XX-SKINNIER" package3d_urn="urn:adsk.eagle:package:6240899/1" value="Microcontroller and Mic power" x="15.24" y="73.66" smashed="yes" rot="R180">
 <attribute name="NAME" x="17.78" y="71.12" size="1.27" layer="25" ratio="10" rot="R180"/>
 <attribute name="VALUE" x="18.923" y="79.629" size="1.27" layer="27" ratio="10" rot="R180"/>
@@
 <attribute name="VALUE" x="-69.596" y="-53.086" size="1.27" layer="27"/>
 </element>
-<element name="LOWBATLED1" library="adafruit" library_urn="urn:adsk.eagle:library:420" package="CHIP-LED0805" package3d_urn="urn:adsk.eagle:package:6240557/1" value="" x="-67.31" y="-44.45" smashed="yes">
+<element name="GSM_LOW_BAT_LED" library="adafruit" library_urn="urn:adsk.eagle:library:420" package="CHIP-LED0805" package3d_urn="urn:adsk.eagle:package:6240557/1" value="" x="-67.31" y="-44.45" smashed="yes">
 <attribute name="NAME" x="-68.58" y="-45.72" size="1.27" layer="25" rot="R90"/>
 <attribute name="VALUE" x="-64.77" y="-45.72" size="1.27" layer="27" rot="R90"/>
 </element>
-<element name="S2" library="adafruit" library_urn="urn:adsk.eagle:library:420" package="B3F-31XX-SKINNIER" package3d_urn="urn:adsk.eagle:package:6240899/1" value="" x="-64.77" y="-58.42" smashed="yes">
+<element name="S2" library="adafruit" library_urn="urn:adsk.eagle:library:420" package="B3F-31XX-SKINNIER" package3d_urn="urn:adsk.eagle:package:6240899/1" value="GSM power" x="-64.77" y="-58.42" smashed="yes">
 <attribute name="NAME" x="-67.31" y="-55.88" size="1.27" layer="25" ratio="10"/>
 <attribute name="VALUE" x="-68.453" y="-64.389" size="1.27" layer="27" ratio="10"/>
@@
 <contactref element="JP1" pad="2"/>
 <contactref element="RECLED" pad="C"/>
-<contactref element="SDLED" pad="C"/>
-<contactref element="NETSTATLED" pad="C"/>
-<contactref element="ERRLED" pad="C"/>
 <contactref element="POWERLED" pad="C"/>
-<contactref element="LOWBATLED" pad="C"/>
+<contactref element="REC_LOW_BAT_LED" pad="C"/>
 <contactref element="S1" pad="2"/>
 <contactref element="SW2" pad="P$1"/>
@@
 <contactref element="R1" pad="1"/>
 <contactref element="CON1" pad="P$8"/>
-<contactref element="LOWBATLED1" pad="C"/>
+<contactref element="GSM_LOW_BAT_LED" pad="C"/>
 <contactref element="JP2" pad="2"/>
 <contactref element="JP2" pad="4"/>
 <contactref element="CN2" pad="2"/>
 <contactref element="S2" pad="1"/>
+<contactref element="SDLED" pad="C"/>
+<contactref element="ERRLED" pad="C"/>
+<contactref element="NETSTATLED" pad="C"/>
 <wire x1="73.66" y1="53.34" x2="86.36" y2="53.34" width="0" layer="19" extent="1-1"/>
 <wire x1="63.5" y1="60.96" x2="73.66" y2="53.34" width="0" layer="19" extent="1-1"/>
@@
 <wire x1="7.62" y1="55.88" x2="17.5006" y2="74.9046" width="0" layer="19" extent="1-1"/>
 </signal>
-<signal name="N$7">
-<contactref element="R7" pad="2"/>
-</signal>
-<signal name="N$8">
-<contactref element="R8" pad="2"/>
-</signal>
 <signal name="N$9">
 <contactref element="RECLED" pad="A"/>
@@
 <wire x1="-39.69" y1="80.01" x2="78.74" y2="60.96" width="0" layer="19" extent="1-1"/>
 </signal>
-<signal name="N$14">
-<contactref element="ERRLED" pad="A"/>
-<contactref element="R8" pad="1"/>
-<wire x1="-52.07" y1="61.18" x2="-51.75" y2="80.01" width="0" layer="19" extent="1-1"/>
-</signal>
-<signal name="N$11">
-<contactref element="NETSTATLED" pad="A"/>
-<contactref element="R7" pad="1"/>
-<wire x1="-46.99" y1="61.18" x2="-46.67" y2="80.01" width="0" layer="19" extent="1-1"/>
-</signal>
-<signal name="N$12">
-<contactref element="SDLED" pad="A"/>
-<contactref element="R5" pad="1"/>
-<wire x1="-41.91" y1="61.18" x2="-36.51" y2="80.01" width="0" layer="19" extent="1-1"/>
-</signal>
 <signal name="N$15">
 <contactref element="POWERLED" pad="A"/>
@@
 <signal name="N$16">
 <contactref element="R3" pad="2"/>
-<contactref element="LOWBATLED" pad="A"/>
+<contactref element="REC_LOW_BAT_LED" pad="A"/>
 <wire x1="-24.45" y1="80.01" x2="-67.31" y2="-17.56" width="0" layer="19" extent="1-1"/>
 </signal>
@@
 <signal name="N$21">
 <contactref element="U$1" pad="38"/>
+<contactref element="R7" pad="1"/>
+<wire x1="-46.67" y1="80.01" x2="73.66" y2="60.96" width="0" layer="19" extent="1-1"/>
 </signal>
 <signal name="N$22">
@@
 <signal name="N$23">
 <contactref element="R9" pad="2"/>
-<contactref element="LOWBATLED1" pad="A"/>
+<contactref element="GSM_LOW_BAT_LED" pad="A"/>
 <wire x1="-67.31" y1="-45.5" x2="-67.63" y2="-50.8" width="0" layer="19" extent="1-1"/>
 </signal>
@@
 <wire x1="7.62" y1="12.7" x2="-62.5094" y2="-59.6646" width="0" layer="19" extent="1-1"/>
 </signal>
+<signal name="N$8">
+<contactref element="R5" pad="2"/>
+<contactref element="SDLED" pad="A"/>
+<wire x1="-41.91" y1="61.18" x2="-34.61" y2="80.01" width="0" layer="19" extent="1-1"/>
+</signal>
+<signal name="N$11">
+<contactref element="R8" pad="2"/>
+<contactref element="ERRLED" pad="A"/>
+<wire x1="-52.07" y1="61.18" x2="-49.85" y2="80.01" width="0" layer="19" extent="1-1"/>
+</signal>
+<signal name="N$12">
+<contactref element="U$1" pad="39"/>
+<contactref element="R5" pad="1"/>
+<wire x1="-36.51" y1="80.01" x2="71.12" y2="60.96" width="0" layer="19" extent="1-1"/>
+</signal>
+<signal name="N$14">
+<contactref element="U$1" pad="37"/>
+<contactref element="R8" pad="1"/>
+<wire x1="-51.75" y1="80.01" x2="76.2" y2="60.96" width="0" layer="19" extent="1-1"/>
+</signal>
+<signal name="N$7">
+<contactref element="NETSTATLED" pad="A"/>
+<contactref element="R7" pad="2"/>
+<wire x1="-46.99" y1="61.18" x2="-44.77" y2="80.01" width="0" layer="19" extent="1-1"/>
+</signal>
 </signals>

Commit message: Fix/Swap RTS and CTS connections
Connections:
- net CTS_OF_GSM: now also CON1.P$15; no longer CON1.P$3, R1.2
- net RTS_OF_GSM: now also CON1.P$3, R1.2; no longer CON1.P$15
Changed lines of the file:
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@@
 <wire x1="63.5" y1="5.08" x2="43.18" y2="60.96" width="0" layer="19" extent="1-1"/>
-</signal>
-<signal name="CTS_OF_GSM">
-<contactref element="U$1" pad="33"/>
-<contactref element="CON1" pad="P$3"/>
-<contactref element="R1" pad="2"/>
-<wire x1="66.04" y1="5.08" x2="86.36" y2="60.96" width="0" layer="19" extent="1-1"/>
-<wire x1="-14.29" y1="80.01" x2="86.36" y2="60.96" width="0" layer="19" extent="1-1"/>
-</signal>
-<signal name="RTS_OF_GSM">
-<contactref element="U$1" pad="34"/>
-<contactref element="CON1" pad="P$15"/>
-<wire x1="63.5" y1="27.94" x2="83.82" y2="60.96" width="0" layer="19" extent="1-1"/>
 </signal>
 <signal name="N$2">
@@
 <wire x1="-46.67" y1="80.01" x2="73.66" y2="60.96" width="0" layer="19" extent="1-1"/>
 </signal>
-<signal name="N$22">
-</signal>
 <signal name="N$23">
 <contactref element="R9" pad="2"/>
@@
 <wire x1="-46.99" y1="61.18" x2="-44.77" y2="80.01" width="0" layer="19" extent="1-1"/>
 </signal>
+<signal name="RTS_OF_GSM">
+<contactref element="U$1" pad="34"/>
+<contactref element="CON1" pad="P$3"/>
+<contactref element="R1" pad="2"/>
+<wire x1="66.04" y1="5.08" x2="83.82" y2="60.96" width="0" layer="19" extent="1-1"/>
+<wire x1="-14.29" y1="80.01" x2="83.82" y2="60.96" width="0" layer="19" extent="1-1"/>
+</signal>
+<signal name="CTS_OF_GSM">
+<contactref element="CON1" pad="P$15"/>
+<contactref element="U$1" pad="33"/>
+<wire x1="63.5" y1="27.94" x2="86.36" y2="60.96" width="0" layer="19" extent="1-1"/>
+</signal>
 </signals>

Commit message: Compoenent placement, Ground plane, drill holes etc on the layout
Parts:
- moved R9 174.4 mm to (95.2, 8.89), turned to 90 degrees
- moved GSM_LOW_BAT_LED 172.7 mm to (95.2, 14.0)
- moved CN2 170.5 mm to (92.7, 36.8), turned to 270 degrees
- moved R8 120.1 mm to (62.2, 39.4)
- moved ERRLED 117.4 mm to (62.2, 35.6), turned to 90 degrees
- moved POWERLED 111.2 mm to (50.8, 35.6), turned to 90 degrees
- moved R7 110.5 mm to (34.3, 3.81)
- moved NETSTATLED 102.4 mm to (34.3, 0.00), turned to 90 degrees
- moved S2 98.8 mm to (14.0, 1.27)
- moved REC_LOW_BAT_LED 95.5 mm to (10.2, 39.4), turned to 90 degrees
- moved R4 90.9 mm to (50.8, 39.4)
- moved R6 90.9 mm to (40.6, 39.4)
- moved SW2 82.7 mm to (16.5, 55.9)
- moved RECLED 81.9 mm to (40.6, 35.6), turned to 90 degrees
- moved R5 76.5 mm to (29.2, 39.4)
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Routing:
- added copper zone on layer 1, net GND
Other:
- board size 100 x 85.1 mm -> 96.2 x 82.5 mm

Commit message: Clean schematics after review with Hari on 25/2/2019, BOM to be prepared
Parts:
- R3, R4, R5, R6, R7, R8, R9: value 330R -> 1KR
- renumbered CN1 to REC_POWER, CN2 to GSM_POWER, CON1 to MIKROELECTRONIKA_SARA_CLICK
Connections:
- net 3V renamed MIC_3V
- net BCLK renamed MIC_BCLK
- net DOUT renamed MIC_DOUT
- net LRCLK renamed MIC_LRCLK
- net N$10 renamed REC_LB
- net N$2 renamed REC_5V
- net N$20 renamed GSM_LB
- net N$21 renamed NETSTATLED
- net N$24 renamed GSM_BAT
- net N$25 renamed GSM_5V
- net N$3 renamed REC_BAT
- removed net N$12: R5.1, U$1.39
- removed net N$13: R6.2, U$1.36
- removed net N$14: R8.1, U$1.37
- removed net N$15: POWERLED.A, R4.1
- removed net N$17: REC_POWER.2
- removed net N$18: JP1.5
- removed net N$19: JP2.5, S2.2
- removed net N$4: JP1.4, S1.1
- removed net N$5: R4.2, U$1.35
- new net ERRLED: R8.1, U$1.39
- new net GSM_5V_EN: JP2.5, S2.1
- new net GSM_BAT_RETURN: GSM_POWER.2, JP2.4
- new net N$3: POWERLED.A, R4.2
- new net N$6: JP2.6
- new net POWERLED: R4.1, U$1.35
- new net RECLED: R6.1, U$1.36
- new net REC_5V_EN: JP1.4, S1.2
- new net REC_BAT_RETURN: JP1.5, REC_POWER.2
- new net SDLED: R5.1, U$1.37
- net GND: now also S1.1, S2.2; no longer GSM_POWER.2, JP2.4, S1.2, S2.1
- net N$9: now also R6.2; no longer R6.1
Routing:
- net REC_5V: track 26.9 -> 0.90 mm
