File: Teensy36_I2S_Proto/wildly_teensy_proto.brd (EAGLE design)
At the start: 96.2 x 82.5 mm, 25 parts, among them SW2 Push_Button

Commit message: Add Jumper to unify power supply for both recorder and GSM when needed, add LEDS for power switches, add caps for supply input
Parts:
- added C1, C3: 10uF, adafruit:C0805
- added C2, C4: 100nF, adafruit:C0805
- added GSM_POWER_JUMPER: (no value), jumper:JP1
- added GSM_PW_LED, REC_PW_LED: (no value), adafruit:CHIP-LED0805
- added R10, R2: 1KR, adafruit:M0805
Connections:
- new net N$10: R2.1, REC_PW_LED.A
- new net N$12: R2.2
- new net N$4: GSM_PW_LED.A, R10.2
- new net N$5: GSM_PW_LED.C, S2.1
- net GND: now also C1.2, C2.2, C3.2, C4.2
- net GSM_5V: now also C3.1, C4.1, GSM_POWER_JUMPER.1
- net GSM_5V_EN: now also R10.1; no longer S2.1
- net REC_5V: now also C1.1, C2.1, GSM_POWER_JUMPER.2
- net REC_5V_EN: now also REC_PW_LED.C
Changed lines of the file:
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@@
 <attribute name="VALUE" x="10.287" y="4.191" size="1.27" layer="27" ratio="10"/>
+</element>
+<element name="C1" library="adafruit" library_urn="urn:adsk.eagle:library:420" package="C0805" package3d_urn="urn:adsk.eagle:package:6240337/1" value="10uF" x="-3.81" y="-8.89" smashed="yes">
+<attribute name="NAME" x="-4.699" y="-7.874" size="1.27" layer="25"/>
+<attribute name="VALUE" x="-4.699" y="-11.176" size="1.27" layer="27"/>
+</element>
+<element name="C2" library="adafruit" library_urn="urn:adsk.eagle:library:420" package="C0805" package3d_urn="urn:adsk.eagle:package:6240337/1" value="100nF" x="-3.81" y="-13.97" smashed="yes">
+<attribute name="NAME" x="-4.699" y="-12.954" size="1.27" layer="25"/>
+<attribute name="VALUE" x="-4.699" y="-16.256" size="1.27" layer="27"/>
+</element>
+<element name="C3" library="adafruit" library_urn="urn:adsk.eagle:library:420" package="C0805" package3d_urn="urn:adsk.eagle:package:6240337/1" value="10uF" x="-3.81" y="-26.67" smashed="yes">
+<attribute name="NAME" x="-4.699" y="-25.654" size="1.27" layer="25"/>
+<attribute name="VALUE" x="-4.699" y="-28.956" size="1.27" layer="27"/>
+</element>
+<element name="C4" library="adafruit" library_urn="urn:adsk.eagle:library:420" package="C0805" package3d_urn="urn:adsk.eagle:package:6240337/1" value="100nF" x="-3.81" y="-20.32" smashed="yes">
+<attribute name="NAME" x="-4.699" y="-19.304" size="1.27" layer="25"/>
+<attribute name="VALUE" x="-4.699" y="-22.606" size="1.27" layer="27"/>
+</element>
+<element name="GSM_POWER_JUMPER" library="jumper" library_urn="urn:adsk.eagle:library:252" package="JP1" package3d_urn="urn:adsk.eagle:package:15455/1" value="" x="-19.05" y="-30.48" smashed="yes">
+<attribute name="NAME" x="-20.701" y="-33.02" size="1.27" layer="25" ratio="10" rot="R90"/>
+<attribute name="VALUE" x="-16.129" y="-33.02" size="1.27" layer="27" ratio="10" rot="R90"/>
+</element>
+<element name="GSM_PW_LED" library="adafruit" library_urn="urn:adsk.eagle:library:420" package="CHIP-LED0805" package3d_urn="urn:adsk.eagle:package:6240557/1" value="" x="-19.05" y="-40.64" smashed="yes">
+<attribute name="NAME" x="-20.32" y="-41.91" size="1.27" layer="25" rot="R90"/>
+<attribute name="VALUE" x="-16.51" y="-41.91" size="1.27" layer="27" rot="R90"/>
+</element>
+<element name="R2" library="adafruit" library_urn="urn:adsk.eagle:library:420" package="M0805" package3d_urn="urn:adsk.eagle:package:6240587/1" value="1KR" x="-20.32" y="-46.99" smashed="yes">
+<attribute name="NAME" x="-21.336" y="-45.974" size="1.27" layer="25"/>
+<attribute name="VALUE" x="-21.336" y="-49.276" size="1.27" layer="27"/>
+</element>
+<element name="REC_PW_LED" library="adafruit" library_urn="urn:adsk.eagle:library:420" package="CHIP-LED0805" package3d_urn="urn:adsk.eagle:package:6240557/1" value="" x="-19.05" y="-57.15" smashed="yes">
+<attribute name="NAME" x="-20.32" y="-58.42" size="1.27" layer="25" rot="R90"/>
+<attribute name="VALUE" x="-16.51" y="-58.42" size="1.27" layer="27" rot="R90"/>
+</element>
+<element name="R10" library="adafruit" library_urn="urn:adsk.eagle:library:420" package="M0805" package3d_urn="urn:adsk.eagle:package:6240587/1" value="1KR" x="-20.32" y="-63.5" smashed="yes">
+<attribute name="NAME" x="-21.336" y="-62.484" size="1.27" layer="25"/>
+<attribute name="VALUE" x="-21.336" y="-65.786" size="1.27" layer="27"/>
 </element>
 </elements>
@@
 <contactref element="S2" pad="2"/>
 <contactref element="S1" pad="1"/>
+<contactref element="C2" pad="2"/>
+<contactref element="C1" pad="2"/>
+<contactref element="C4" pad="2"/>
+<contactref element="C3" pad="2"/>
 <wire x1="73.66" y1="53.34" x2="86.36" y2="53.34" width="0" layer="19" extent="1-1"/>
 <wire x1="63.5" y1="60.96" x2="73.66" y2="53.34" width="0" layer="19" extent="1-1"/>
@@
 <wire x1="16.2306" y1="0.0254" x2="7.62" y2="5.08" width="0" layer="19" extent="1-1"/>
 <wire x1="33.24" y1="0" x2="16.2306" y2="0.0254" width="0" layer="19" extent="1-1"/>
+<wire x1="-2.96" y1="-8.89" x2="7.62" y2="5.08" width="0" layer="19" extent="1-1"/>
+<wire x1="-2.96" y1="-13.97" x2="-2.96" y2="-8.89" width="0" layer="19" extent="1-1"/>
+<wire x1="-2.96" y1="-20.32" x2="-2.96" y2="-13.97" width="0" layer="19" extent="1-1"/>
+<wire x1="-2.96" y1="-26.67" x2="-2.96" y2="-20.32" width="0" layer="19" extent="1-1"/>
 </signal>
 <signal name="TX_OF_GSM">
@@
 <contactref element="JP1" pad="4"/>
 <contactref element="S1" pad="2"/>
+<contactref element="REC_PW_LED" pad="C"/>
 <wire x1="7.62" y1="55.88" x2="12.9794" y2="74.9046" width="0" layer="19" extent="1-1"/>
+<wire x1="-19.05" y1="-56.1" x2="7.62" y2="55.88" width="0" layer="19" extent="1-1"/>
 </signal>
 <signal name="REC_LB">
@@
 <contactref element="U$1" pad="5V"/>
 <wire x1="34.29" y1="48.895" x2="33.655" y2="48.26" width="0.1524" layer="1"/>
+<contactref element="C1" pad="1"/>
+<contactref element="C2" pad="1"/>
+<contactref element="GSM_POWER_JUMPER" pad="2"/>
 <wire x1="7.62" y1="48.26" x2="33.655" y2="48.26" width="0" layer="19" extent="1-1"/>
+<wire x1="-4.66" y1="-8.89" x2="7.62" y2="48.26" width="0" layer="19" extent="1-1"/>
+<wire x1="-4.66" y1="-13.97" x2="-4.66" y2="-8.89" width="0" layer="19" extent="1-1"/>
+<wire x1="-19.05" y1="-29.21" x2="-4.66" y2="-13.97" width="0" layer="19" extent="1-1"/>
 </signal>
 <signal name="GSM_BAT">
@@
 <signal name="GSM_5V_EN">
 <contactref element="JP2" pad="5"/>
-<contactref element="S2" pad="1"/>
-<wire x1="11.7094" y1="0.0254" x2="7.62" y2="12.7" width="0" layer="19" extent="1-1"/>
+<contactref element="R10" pad="1"/>
+<wire x1="7.62" y1="12.7" x2="-21.27" y2="-63.5" width="0" layer="19" extent="1-1"/>
 </signal>
 <signal name="GSM_LB">
@@
 <contactref element="JP2" pad="1"/>
 <contactref element="MIKROELECTRONIKA_SARA_CLICK" pad="P$10"/>
+<contactref element="C3" pad="1"/>
+<contactref element="C4" pad="1"/>
+<contactref element="GSM_POWER_JUMPER" pad="1"/>
 <wire x1="7.62" y1="2.54" x2="76.2" y2="27.94" width="0" layer="19" extent="1-1"/>
+<wire x1="-4.66" y1="-20.32" x2="7.62" y2="2.54" width="0" layer="19" extent="1-1"/>
+<wire x1="-4.66" y1="-26.67" x2="-4.66" y2="-20.32" width="0" layer="19" extent="1-1"/>
+<wire x1="-19.05" y1="-31.75" x2="-4.66" y2="-26.67" width="0" layer="19" extent="1-1"/>
 </signal>
 <signal name="N$2">
@@
 <wire x1="49.85" y1="39.37" x2="81.28" y2="60.96" width="0" layer="19" extent="1-1"/>
 </signal>
+<signal name="N$4">
+<contactref element="R10" pad="2"/>
+<contactref element="GSM_PW_LED" pad="A"/>
+<wire x1="-19.05" y1="-41.69" x2="-19.37" y2="-63.5" width="0" layer="19" extent="1-1"/>
+</signal>
+<signal name="N$5">
+<contactref element="GSM_PW_LED" pad="C"/>
+<contactref element="S2" pad="1"/>
+<wire x1="11.7094" y1="0.0254" x2="-19.05" y2="-39.59" width="0" layer="19" extent="1-1"/>
+</signal>
+<signal name="N$10">
+<contactref element="REC_PW_LED" pad="A"/>
+<contactref element="R2" pad="1"/>
+<wire x1="-21.27" y1="-46.99" x2="-19.05" y2="-58.2" width="0" layer="19" extent="1-1"/>
+</signal>
+<signal name="N$12">
+<contactref element="R2" pad="2"/>
+</signal>
 </signals>

Commit message: Remove LEDs for Power Enables, Remove LEDs for Low Bat indicators, Add NPN Transistors as LED drivers - TBD: Calculate R values, Remove Power LED and change pinout to power control for resetting system power- TBD: add connection, Provide 3.3V to GSM modem
Parts:
- removed C1, C3: 10uF, adafruit:C0805
- removed C2, C4: 100nF, adafruit:C0805
- removed GSM_POWER_JUMPER: (no value), jumper:JP1
- removed GSM_PW_LED, REC_PW_LED: (no value), adafruit:CHIP-LED0805
- removed R10, R2: 1KR, adafruit:M0805
- R3, R4, R5, R6, R7, R8, R9: value 1KR -> 330R
- renumbered GSM_POWER to CN2, MIKROELECTRONIKA_SARA_CLICK to CON1, REC_POWER to CN1
Connections:
- net GSM_BAT renamed N$24
- net GSM_LB renamed N$20
- net MIC_3V renamed 3V
- net MIC_BCLK renamed BCLK
- net MIC_DOUT renamed DOUT
- net MIC_LRCLK renamed LRCLK
- net NETSTATLED renamed N$21
- net REC_BAT renamed N$3
- net REC_LB renamed N$10
- removed net ERRLED: R8.1, U$1.39
- removed net GSM_5V: C3.1, C4.1, CON1.P$10, GSM_POWER_JUMPER.1, JP2.1
- removed net GSM_5V_EN: JP2.5, R10.1
- removed net GSM_BAT_RETURN: CN2.2, JP2.4
- removed net N$10 (its old number): R2.1, REC_PW_LED.A
- removed net N$3 (its old number): POWERLED.A, R4.2
- removed net N$6: JP2.6
- removed net POWERLED: R4.1, U$1.35
- removed net RECLED: R6.1, U$1.36
- removed net REC_5V: C1.1, C2.1, GSM_POWER_JUMPER.2, JP1.1, U$1.5V
- removed net REC_5V_EN: JP1.4, REC_PW_LED.C, S1.2
- removed net REC_BAT_RETURN: CN1.2, JP1.5
- removed net SDLED: R5.1, U$1.37
- new net N$13: R6.2, U$1.36
- new net N$14: R8.1, U$1.37
- new net N$15: POWERLED.A, R4.1
- new net N$17: CN1.2
- new net N$18: JP1.5
- new net N$19: JP2.5, S2.2
- new net N$2: JP1.1, U$1.5V
- new net N$25: CON1.P$10, JP2.1
- net GND: now also CN2.2, JP2.4, S1.2, S2.1; no longer C1.2, C2.2, C3.2, C4.2, S1.1, S2.2
- net N$12: now also R5.1, U$1.39; no longer R2.2
- net N$4: now also JP1.4, S1.1; no longer GSM_PW_LED.A, R10.2
- net N$5: now also R4.2, U$1.35; no longer GSM_PW_LED.C, S2.1
- net N$9: now also R6.1; no longer R6.2
Routing:
- net N$2: track 0.00 -> 26.9 mm
- net REC_5V: track 0.90 -> 0.00 mm
