File: Teensy36_I2S_Proto/wildly_teensy_proto.brd (EAGLE design)
At the start: 96.2 x 82.5 mm, 25 parts, among them CON1 MIKROE_BUS_CONN, SW2 Push_Button

Commit message: Add resistor values for LED driver, remove previous board file due to inconsistency and create a fresh layout from schematics
Parts:
- removed CN1, CN2: (no value), adafruit:JST-PH-2-SMT-RA
- removed CON1: MIKROE_BUS_CONN, mikrobus_lib:MIKROBUS_HOST_CONN
- removed GSM_LOW_BAT_LED, POWERLED, REC_LOW_BAT_LED: (no value), adafruit:CHIP-LED0805
- removed R4, R5, R6, R7, R8: 330R, adafruit:M0805
- added C1, C3: 10uF, adafruit:C0805
- added C2, C4: 100nF, adafruit:C0805
- added GSM_POWER, REC_POWER: (no value), adafruit:JST-PH-2-SMT-RA
- added GSM_POWER_JUMPER: (no value), jumper:JP1
- added MIKROELECTRONIKA_SARA_CLICK: MIKROE_BUS_CONN, mikrobus_lib:MIKROBUS_HOST_CONN
- added R10, R11, R12: 82R, adafruit:M0805
- added R13, R2: 1.65KR, adafruit:M0805
- added R14: 1KR, adafruit:M0805
- added T1, T2, T3, T4: 2N2222, adafruit:TO92-EBC-OVAL
- R3, R9: value 330R -> 1.65KR
- moved R9 155.7 mm to (-34.3, 95.2), turned to 0 degrees
- moved JP2 119.6 mm to (-72.4, 100.3), turned to 0 degrees
- moved R1 112.4 mm to (-74.9, 95.2)
- moved SDLED 107.9 mm to (-67.3, 83.8), turned to 0 degrees
- moved U$1 105.8 mm to (-59.7, 41.9)
- moved JP3 105.0 mm to (-53.3, 100.3)
- moved ERRLED 101.2 mm to (-26.7, 83.8), turned to 0 degrees
- moved SW2 96.8 mm to (-76.2, 83.8)
- moved S2 92.9 mm to (-20.3, 87.6)
- moved RECLED 87.0 mm to (-31.8, 83.8), turned to 0 degrees
- moved S1 85.6 mm to (-69.8, 64.8), turned to 0 degrees
- moved NETSTATLED 82.8 mm to (-20.3, 62.2), turned to 0 degrees
- moved JP1 63.8 mm to (-36.8, 100.3), turned to 0 degrees
- moved R3 63.7 mm to (-26.7, 95.2), turned to 0 degrees
Connections:
- net 3V renamed MIC_3V
- net BCLK renamed MIC_BCLK
- net DOUT renamed MIC_DOUT
- net LRCLK renamed MIC_LRCLK
- removed net N$12: R5.1, U$1.39
- removed net N$13: R6.2, U$1.36
- removed net N$17: CN1.2
- removed net N$18: JP1.5
- removed net N$19: JP2.5, S2.2
- removed net N$20: JP2.3, R9.1
- removed net N$21: R7.1, U$1.38
- removed net N$23: GSM_LOW_BAT_LED.A, R9.2
- removed net N$24: CN2.1, JP2.7
- removed net N$25: CON1.P$10, JP2.1
- new net 3V3: MIKROELECTRONIKA_SARA_CLICK.P$7, R10.2, R11.2, R12.2, R14.2
- new net ERRLED: R3.1, U$1.39
- new net GSM_5V: C3.1, C4.1, GSM_POWER_JUMPER.1, JP2.1, MIKROELECTRONIKA_SARA_CLICK.P$10
- new net GSM_5V_EN: JP2.5, S2.1
- new net GSM_BAT: GSM_POWER.1, JP2.7
- new net GSM_BAT_RETURN: GSM_POWER.2, JP2.4
- new net GSM_LB: JP2.3
- new net N$6: JP2.6
- new net NETSTATLED: R9.1, U$1.38
- new net POWER_CONTRL: U$1.35
- new net RECLED: R2.1, U$1.36
- new net REC_5V: C1.1, C2.1, GSM_POWER_JUMPER.2, JP1.1, U$1.5V
- new net REC_5V_EN: JP1.4, S1.2
- new net REC_BAT: JP1.6, REC_POWER.1
- new net REC_BAT_RETURN: JP1.5, REC_POWER.2
- new net REC_LB: JP1.3
- new net SDLED: R13.1, U$1.37
- net CTS_OF_GSM: now also MIKROELECTRONIKA_SARA_CLICK.P$15; no longer CON1.P$15
- net GND: now also C1.2, C2.2, C3.2, C4.2, MIKROELECTRONIKA_SARA_CLICK.P$8, MIKROELECTRONIKA_SARA_CLICK.P$9, S1.1, S2.2, T1.E, T2.E, T3.E, T4.E; no longer CN2.2, CON1.P$8, CON1.P$9, ERRLED.C, GSM_LOW_BAT_LED.C, JP2.4, NETSTATLED.C, POWERLED.C, RECLED.C, REC_LOW_BAT_LED.C, S1.2, S2.1, SDLED.C
- net N$10: now also SDLED.C, T4.C; no longer JP1.3, R3.1
- net N$11: now also R13.2, T4.B; no longer ERRLED.A, R8.2
- net N$14: now also R10.1, RECLED.A; no longer R8.1, U$1.37
- net N$15: now also ERRLED.A, R11.1; no longer POWERLED.A, R4.1
- net N$16: now also NETSTATLED.A, R12.1; no longer R3.2, REC_LOW_BAT_LED.A
- net N$2: now also RECLED.C, T2.C; no longer JP1.1, U$1.5V
- net N$3: now also R2.2, T2.B; no longer CN1.1, JP1.6
- net N$4: now also ERRLED.C, T1.C; no longer JP1.4, S1.1
- net N$5: now also NETSTATLED.C, T3.C; no longer R4.2, U$1.35
- net N$7: now also R9.2, T3.B; no longer NETSTATLED.A, R7.2
- net N$8: now also R3.2, T1.B; no longer R5.2, SDLED.A
- net N$9: now also R14.1, SDLED.A; no longer R6.1, RECLED.A
- net RESET_GSM: now also MIKROELECTRONIKA_SARA_CLICK.P$2; no longer CON1.P$2
- net RTS_OF_GSM: now also MIKROELECTRONIKA_SARA_CLICK.P$3; no longer CON1.P$3
- net RX_OF_GSM: now also MIKROELECTRONIKA_SARA_CLICK.P$14; no longer CON1.P$14
- net TX_OF_GSM: now also MIKROELECTRONIKA_SARA_CLICK.P$13; no longer CON1.P$13
Routing:
- net N$2: track 26.9 -> 0.00 mm
- removed copper zone on layer 1, net GND
Other:
- board size 96.2 x 82.5 mm -> 100 x 80 mm
- board text removed: "Adafruit 5V Boost"
- board text removed: "Adafruit 5V Boost 1A"
- board text removed: "Adafruit I2S Mic SPH0645LM4H"
- board text removed: "Battery Connector"
- board text removed: "Mikroelectronika Click SARA 3G"
- board text removed: "Teensy 3.6"

Commit message: Add BOM file, fix R value for LED driver, start component placement in layout
Parts:
- R14: value 1KR -> 82R
- moved R1 185.7 mm to (91.4, 12.7), turned to 90 degrees
- moved C3 182.1 mm to (87.6, 3.81)
- moved R14 181.5 mm to (91.4, 35.6), turned to 90 degrees
- moved JP3 175.6 mm to (96.5, 8.89), turned to 90 degrees
- moved SW2 173.8 mm to (77.5, 2.54)
- moved SDLED 171.7 mm to (97.8, 36.8)
- moved C1 153.6 mm to (88.9, 76.2)
- moved C2 144.0 mm to (91.4, 66.0), turned to 90 degrees
- moved R12 142.0 mm to (91.4, 22.9), turned to 90 degrees
- moved C4 138.5 mm to (80.0, 76.2)
- moved JP1 136.5 mm to (96.5, 71.1), turned to 90 degrees
- moved RECLED 135.0 mm to (97.8, 45.7)
- moved U$1 135.0 mm to (74.9, 52.1), turned to 270 degrees
- moved T4 132.5 mm to (53.3, 21.6)
- moved S1 131.3 mm to (61.0, 76.2)
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
Commit message: Add routing, clear DRC with sparkfun design rules
Parts:
- moved GSM_POWER 68.7 mm to (41.9, 72.4)
- moved R12 43.8 mm to (48.3, 15.2), turned to 180 degrees
- moved R14 43.5 mm to (48.3, 30.5), turned to 180 degrees
- moved R10 43.2 mm to (48.3, 44.5), turned to 180 degrees
- moved R11 43.2 mm to (48.3, 54.6), turned to 180 degrees
- moved NETSTATLED 37.6 mm to (61.0, 15.2), turned to 90 degrees
- moved SDLED 37.4 mm to (61.0, 30.5), turned to 90 degrees
- moved ERRLED 36.9 mm to (61.0, 54.6), turned to 90 degrees
- moved RECLED 36.9 mm to (61.0, 44.5), turned to 90 degrees
- moved C1 33.9 mm to (96.5, 43.2), turned to 90 degrees
- moved S1 30.5 mm to (91.4, 76.2)
- moved C4 19.7 mm to (61.0, 71.1)
- moved C2 16.1 mm to (96.5, 50.8)
- moved R1 15.2 mm to (91.4, 27.9)
- moved JP1 7.62 mm to (96.5, 63.5)
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Routing:
- net GND: track 0.00 -> 443.6 mm, vias 0 -> 7
- net RESET_GSM: track 0.00 -> 198.1 mm, vias 0 -> 1
- net GSM_5V: track 0.00 -> 179.9 mm, vias 0 -> 1
- net ERRLED: track 0.00 -> 179.2 mm, vias 0 -> 1
- net RTS_OF_GSM: track 0.00 -> 152.3 mm
- net 3V3: track 0.00 -> 141.0 mm, vias 0 -> 3
- net MIC_3V: track 0.00 -> 138.8 mm, vias 0 -> 1
- net REC_5V: track 0.00 -> 133.5 mm, vias 0 -> 6
- net CTS_OF_GSM: track 0.00 -> 104.4 mm
- net MIC_BCLK: track 0.00 -> 93.6 mm, vias 0 -> 3
- net RECLED: track 0.00 -> 93.0 mm, vias 0 -> 5
- net REC_BAT_RETURN: track 0.00 -> 88.5 mm
- net REC_BAT: track 0.00 -> 87.3 mm
- net GSM_5V_EN: track 0.00 -> 77.0 mm
- net MIC_LRCLK: track 0.00 -> 71.5 mm
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Other:
- board size 100 x 80 mm -> 96.2 x 80 mm

Commit message: Fix power line, change layout according to review with Hari on 11/3/2019. TBD: BOM finalization and final footprint alignment
Parts:
- removed JP1, JP3: (no value), adafruit:1X06
- removed JP2: (no value), adafruit:1X08-BIG
- removed S1: Microcontroller and Mic power, adafruit:B3F-31XX-SKINNIER
- removed S2: GSM power, adafruit:B3F-31XX-SKINNIER
- removed SW2: Push_Button, adafruit:TACT_PANA-EVQ
- added GSM_ON_OFF_SW: GSM power, adafruit:B3F-31XX-SKINNIER
- added REC_ON_OFF_SW: Microcontroller and Mic power, adafruit:B3F-31XX-SKINNIER
- added REC_SW: Push_Button, adafruit:TACT_PANA-EVQ
- added WILDLY_5V_0.5A_BOOST, WILDLY_I2S_MIC: (no value), adafruit:1X06
- added WILDLY_5V_1A_BOOST: (no value), adafruit:1X08-BIG
- moved C3 87.1 mm to (25.4, 64.8), turned to 180 degrees
- moved R1 71.7 mm to (20.3, 19.1), turned to 180 degrees
- moved GSM_POWER_JUMPER 67.4 mm to (49.5, 71.1)
- moved REC_POWER 67.1 mm to (94.0, 63.5), turned to 270 degrees
- moved C1 42.3 mm to (61.0, 66.0), turned to 0 degrees
- moved C4 35.7 mm to (25.4, 68.6), turned to 180 degrees
- moved GSM_POWER 33.6 mm to (8.89, 66.0), turned to 90 degrees
- moved R3 26.9 mm to (61.0, 45.7)
- moved SDLED 25.7 mm to (52.1, 6.35)
- moved R14 25.6 mm to (59.7, 7.62)
- moved C2 21.7 mm to (88.9, 71.1), turned to 180 degrees
- moved R2 20.5 mm to (61.0, 38.1)
- moved R9 19.7 mm to (59.7, 22.9)
- moved R10 18.0 mm to (45.7, 26.7)
- moved T1 17.8 mm to (52.1, 47.0)
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Connections:
- removed net MIC_3V: JP3.1, U$1.3V3(1), U$1.3V3(2), U$1.3V3(3), U$1.3V3(4)
- new net NET_STAT: MIKROELECTRONIKA_SARA_CLICK.P$1, U$1.24
- net 3V3: now also U$1.3V3(1), U$1.3V3(2), U$1.3V3(3), U$1.3V3(4), WILDLY_I2S_MIC.1
- net GND: now also GSM_ON_OFF_SW.2, REC_ON_OFF_SW.1, REC_SW.P$1, WILDLY_5V_0.5A_BOOST.2, WILDLY_5V_1A_BOOST.2, WILDLY_I2S_MIC.2; no longer JP1.2, JP2.2, JP3.2, S1.1, S2.2, SW2.P$1
- net GSM_5V: now also WILDLY_5V_1A_BOOST.1; no longer JP2.1
- net GSM_5V_EN: now also GSM_ON_OFF_SW.1, WILDLY_5V_1A_BOOST.5; no longer JP2.5, S2.1
- net GSM_BAT: now also WILDLY_5V_1A_BOOST.7; no longer JP2.7
- net GSM_BAT_RETURN: now also WILDLY_5V_1A_BOOST.4; no longer JP2.4
- net GSM_LB: now also WILDLY_5V_1A_BOOST.3; no longer JP2.3
- net MIC_BCLK: now also WILDLY_I2S_MIC.3; no longer JP3.3
- net MIC_DOUT: now also WILDLY_I2S_MIC.4; no longer JP3.4
- net MIC_LRCLK: now also WILDLY_I2S_MIC.5; no longer JP3.5
- net N$1: now also REC_SW.P$2; no longer SW2.P$2
- net N$6: now also WILDLY_5V_1A_BOOST.6; no longer JP2.6
- net REC_5V: now also U$1.VIN, WILDLY_5V_0.5A_BOOST.1; no longer JP1.1, U$1.5V
- net REC_5V_EN: now also REC_ON_OFF_SW.2, WILDLY_5V_0.5A_BOOST.4; no longer JP1.4, S1.2
- net REC_BAT: now also WILDLY_5V_0.5A_BOOST.6; no longer JP1.6
- net REC_BAT_RETURN: now also WILDLY_5V_0.5A_BOOST.5; no longer JP1.5
- net REC_LB: now also WILDLY_5V_0.5A_BOOST.3; no longer JP1.3
Routing:
- net MIC_3V: track 138.8 -> 0.00 mm, vias 1 -> 0
- net ERRLED: track 179.2 -> 44.7 mm, vias 1 -> 2
- net RESET_GSM: track 198.1 -> 95.3 mm, vias 1 -> 2
- net 3V3: track 141.0 -> 224.6 mm, vias 3 -> 1
- net REC_5V: track 133.5 -> 54.5 mm, vias 6 -> 0
- net GSM_5V: track 179.9 -> 102.6 mm, vias 1 -> 0
- net REC_BAT: track 87.3 -> 21.4 mm, vias 0 -> 2
- net NET_STAT: track 0.00 -> 62.1 mm, vias 0 -> 2
- net RTS_OF_GSM: track 152.3 -> 91.5 mm, vias 0 -> 2
- net MIC_BCLK: track 93.6 -> 33.3 mm, vias 3 -> 2
- net REC_BAT_RETURN: track 88.5 -> 34.1 mm
- net MIC_LRCLK: track 71.5 -> 17.3 mm
- net GND: track 443.6 -> 390.7 mm, vias 7 -> 20
- net GSM_5V_EN: track 77.0 -> 24.9 mm
- net N$1: track 69.6 -> 19.5 mm, vias 3 -> 2
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- added copper zone on layer 1, net GND

Commit message: Add copper pours, resize board, adjust routing for sufficient spacing etc
Routing:
- net GND: track 390.7 -> 394.5 mm, vias 20 -> 24
- net REC_5V: track 54.5 -> 57.1 mm
- net REC_BAT: track 21.4 -> 19.6 mm, vias 2 -> 1
- net N$4: track 8.45 -> 9.94 mm
- net REC_5V_EN: track 27.9 -> 29.1 mm
- net N$3: track 14.7 -> 15.8 mm
- net N$9: track 10.3 -> 11.2 mm
- net RTS_OF_GSM: track 91.5 -> 92.3 mm
- net N$2: track 7.36 -> 8.11 mm
- net N$10: track 7.18 -> 7.93 mm
- net N$15: track 7.42 -> 8.16 mm
- added copper zone on layer 16, net GND
Other:
- board outline removed
- board text added: "Wildly_Listen_Proto_v1"

Commit message: Add latest files from Aakash Nasa with updatest to schamtic and layout to include: Pinouts for unused pins from Teensy, changes to BOM according to component availabilityetc
Parts:
- added J1, J2: 61300311121, 61300311121:61300311121
- added J3: 61300211121, 61300211121:61300211121
- added TEENSY_PINS_1-6, TEENSY_PINS_13-18, TEENSY_PINS_19-24, TEENSY_PINS_25-30, TEENSY_PINS_31-36, TEENSY_PINS_37-42, TEENSY_PINS_43-48, TEENSY_PINS_7-12: (no value), adafruit:1X06
- GSM_ON_OFF_SW: value GSM power -> GSM Power; device adafruit:B3F-31XX-SKINNIER -> 1101M2S3CQE2:SW_1101M2S3CQE2
- REC_ON_OFF_SW: value Microcontroller and Mic power -> Microcontroller and Mic Power; device adafruit:B3F-31XX-SKINNIER -> 1101M2S3CQE2:SW_1101M2S3CQE2
- REC_SW: device adafruit:TACT_PANA-EVQ -> 800AWSP9M2QE:800AWSP9M2QE
- T1, T2, T3, T4: value 2N2222 -> 2N2222A; device adafruit:TO92-EBC-OVAL -> 2N2222A:TO127P584H533-3
- moved C2 44.7 mm to (44.5, 66.0), turned to 0 degrees
- moved WILDLY_I2S_MIC 22.2 mm to (83.8, 27.9)
- moved ERRLED 18.2 mm to (34.3, 43.2), turned to 270 degrees
- moved RECLED 18.0 mm to (34.3, 31.8), turned to 270 degrees
- moved SDLED 18.0 mm to (34.3, 8.89), turned to 270 degrees
- moved NETSTATLED 17.8 mm to (34.3, 20.3), turned to 270 degrees
- moved GSM_POWER_JUMPER 17.3 mm to (33.0, 66.0)
- moved C1 16.7 mm to (44.5, 63.5)
- moved R2 16.6 mm to (44.5, 39.4)
- moved R13 16.1 mm to (44.5, 16.5), turned to 180 degrees
- moved R9 15.7 mm to (44.5, 26.7), turned to 180 degrees
- moved R14 15.5 mm to (44.5, 5.08), turned to 0 degrees
- moved R3 15.3 mm to (45.7, 47.0), turned to 180 degrees
- moved REC_SW 14.5 mm to (34.3, 58.4)
- moved REC_ON_OFF_SW 14.0 mm to (48.3, 74.9), turned to 90 degrees
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Connections:
- removed net N$1: REC_SW.P$2, U$1.4
- new net 25: TEENSY_PINS_13-18.5, U$1.25
- new net A0: TEENSY_PINS_37-42.1, U$1.14
- new net A1: TEENSY_PINS_31-36.6, U$1.15
- new net A2: TEENSY_PINS_31-36.5, U$1.16
- new net A3: TEENSY_PINS_31-36.4, U$1.17
- new net A4: J1.1, TEENSY_PINS_31-36.3, U$1.18
- new net A5: J1.2, TEENSY_PINS_31-36.2, U$1.19
- new net AGND: TEENSY_PINS_25-30.2, U$1.AGND
- new net ALT-MOSI: TEENSY_PINS_19-24.2, U$1.28
- new net ALT-PWM: TEENSY_PINS_13-18.6, U$1.26
- new net ALT-RX1: TEENSY_PINS_19-24.1, U$1.27
- new net DAC0: TEENSY_PINS_37-42.5, U$1.DAC0
- new net DAC1: TEENSY_PINS_37-42.4, U$1.DAC1
- new net MISO: TEENSY_PINS_13-18.2, U$1.12
- new net MOSI: TEENSY_PINS_13-18.1, U$1.11
- new net N$13: J1.3
- new net PWM1: TEENSY_PINS_1-6.4, U$1.2
- new net PWM10: TEENSY_PINS_19-24.4, U$1.30
- new net PWM11: TEENSY_PINS_19-24.5, U$1.31
- new net PWM12: TEENSY_PINS_19-24.6, U$1.32
- new net PWM13: TEENSY_PINS_25-30.6, U$1.21
- new net PWM14: TEENSY_PINS_25-30.5, U$1.22
- new net PWM2: TEENSY_PINS_1-6.5, U$1.3
- new net PWM3: REC_SW.3, TEENSY_PINS_1-6.6, U$1.4
- new net PWM4: TEENSY_PINS_7-12.1, U$1.5
- new net PWM5: TEENSY_PINS_7-12.2, U$1.6
- new net PWM6: TEENSY_PINS_7-12.3, U$1.7
- new net PWM7: TEENSY_PINS_7-12.4, U$1.8
- new net PWM8: TEENSY_PINS_7-12.6, U$1.10
- new net PWM9: TEENSY_PINS_19-24.3, U$1.29
- net 3V3: now also TEENSY_PINS_13-18.3, TEENSY_PINS_25-30.3
- net CTS_OF_GSM: now also TEENSY_PINS_43-48.6
- net ERRLED: now also TEENSY_PINS_37-42.6
- net GND: now also GSM_ON_OFF_SW.1, J3.1, REC_ON_OFF_SW.2, REC_SW.1, T1.1, T2.1, T3.1, T4.1, TEENSY_PINS_1-6.1, TEENSY_PINS_37-42.3; no longer GSM_ON_OFF_SW.2, REC_ON_OFF_SW.1, REC_SW.P$1, T1.E, T2.E, T3.E, T4.E
- net GSM_5V_EN: now also GSM_ON_OFF_SW.2; no longer GSM_ON_OFF_SW.1
- net MIC_BCLK: now also TEENSY_PINS_7-12.5
- net MIC_DOUT: now also TEENSY_PINS_37-42.2
- net MIC_LRCLK: now also TEENSY_PINS_25-30.4
- net N$10: now also T4.3; no longer T4.C
- net N$11: now also T4.2; no longer T4.B
- net N$2: now also T2.3; no longer T2.C
- net N$3: now also T2.2; no longer T2.B
- net N$4: now also T1.3; no longer T1.C
- net N$5: now also T3.3; no longer T3.C
- net N$7: now also T3.2; no longer T3.B
- net N$8: now also T1.2; no longer T1.B
- net NETSTATLED: now also TEENSY_PINS_43-48.1
- net NET_STAT: now also TEENSY_PINS_13-18.4
- net POWER_CONTRL: now also TEENSY_PINS_43-48.4
- net RECLED: now also TEENSY_PINS_43-48.3
- net REC_5V: now also J3.2, TEENSY_PINS_25-30.1
- net REC_5V_EN: now also REC_ON_OFF_SW.1; no longer REC_ON_OFF_SW.2
- net RESET_GSM: now also TEENSY_PINS_31-36.1
- net RTS_OF_GSM: now also TEENSY_PINS_43-48.5
- net RX_OF_GSM: now also TEENSY_PINS_1-6.3
- net SDLED: now also TEENSY_PINS_43-48.2
- net TX_OF_GSM: now also TEENSY_PINS_1-6.2
Routing:
- net GND: track 394.5 -> 483.1 mm
- net GSM_5V: track 102.6 -> 62.8 mm, vias 0 -> 1
- net REC_5V: track 57.1 -> 83.2 mm
- net RESET_GSM: track 95.3 -> 71.1 mm, vias 2 -> 1
- net MIC_LRCLK: track 17.3 -> 41.5 mm, vias 0 -> 2
- net PWM3: track 0.00 -> 23.5 mm, vias 0 -> 2
- net CTS_OF_GSM: track 55.3 -> 77.4 mm, vias 1 -> 2
- net NET_STAT: track 62.1 -> 40.7 mm, vias 2 -> 1
- net N$1: track 19.5 -> 0.00 mm, vias 2 -> 0
- net A4: track 0.00 -> 14.3 mm
- net A5: track 0.00 -> 13.5 mm
- net RX_OF_GSM: track 82.5 -> 70.1 mm, vias 0 -> 1
- net TX_OF_GSM: track 82.5 -> 70.1 mm, vias 2 -> 1
- net MIC_BCLK: track 33.3 -> 44.5 mm
- net RTS_OF_GSM: track 92.3 -> 82.5 mm, vias 2 -> 0
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Other:
- board text added: "3V3"
- board text added: "GND"
- board text added: "GSM_5V"
- board text added: "GSM_5V_EN"
- board text added: "GSM_BAT"
- board text added: "GSM_BAT_RETURN"
- board text added: "GSM_LB"
- board text added: "MIC_BCLK"
- board text added: "MIC_DOUT"
- board text added: "MIC_LRCLK"
- board text added: "REC_5V"
- board text added: "REC_5V_EN"
- board text added: "REC_BAT"
- board text added: "REC_BAT_RETURN"
- board text added: "REC_LB"

Commit message: Teensy Proto schematic and Layout File updated
Parts:
- removed GSM_POWER: (no value), adafruit:JST-PH-2-SMT-RA
- removed J3: 61300211121, 61300211121:61300211121
- added FUEL_GAUGE, SOLAR_CHARGER: 61300211121, 61300211121:61300211121
- moved MIKROELECTRONIKA_SARA_CLICK 16.5 mm to (26.7, 35.6)
- moved R1 16.5 mm to (21.6, 40.6)
- moved REC_ON_OFF_SW 3.81 mm to (44.5, 74.9)
- moved GSM_ON_OFF_SW 2.54 mm to (30.5, 74.9)
- moved ERRLED 2.54 mm to (34.3, 45.7)
- moved J1 2.54 mm to (77.5, 53.3)
- moved J2 2.54 mm to (85.1, 53.3)
- moved REC_SW 1.27 mm to (35.6, 58.4)
- moved WILDLY_5V_1A_BOOST 1.27 mm to (12.7, 76.2)
- moved C3 1.27 mm to (21.6, 63.5)
- moved C4 1.27 mm to (21.6, 66.0)
- moved WILDLY_I2S_MIC 1.27 mm to (83.8, 29.2)
- renumbered TEENSY_PINS_1-6 to TEENSY_1, TEENSY_PINS_13-18 to TEENSY_3, TEENSY_PINS_19-24 to TEENSY_4, TEENSY_PINS_25-30 to TEENSY_5, TEENSY_PINS_31-36 to TEENSY_6, TEENSY_PINS_37-42 to TEENSY_7, TEENSY_PINS_43-48 to TEENSY_8, TEENSY_PINS_7-12 to TEENSY_2
Connections:
- net GND: no longer J3.1
- net GSM_BAT: now also FUEL_GAUGE.2, SOLAR_CHARGER.1; no longer GSM_POWER.1
- net GSM_BAT_RETURN: now also FUEL_GAUGE.1, SOLAR_CHARGER.2; no longer GSM_POWER.2
- net REC_5V: no longer J3.2
Routing:
- net GSM_BAT: track 10.2 -> 128.8 mm, vias 0 -> 2
- net GSM_BAT_RETURN: track 15.0 -> 121.7 mm, vias 0 -> 2
- net GND: track 483.1 -> 454.7 mm, vias 24 -> 21
- net REC_5V: track 83.2 -> 64.8 mm
- net RTS_OF_GSM: track 82.5 -> 99.0 mm
- net CTS_OF_GSM: track 77.4 -> 92.4 mm
- net RESET_GSM: track 71.1 -> 56.8 mm
- net GSM_5V: track 62.8 -> 49.2 mm
- net RX_OF_GSM: track 70.1 -> 61.8 mm
- net NET_STAT: track 40.7 -> 33.6 mm
- net TX_OF_GSM: track 70.1 -> 63.2 mm
- net MIC_LRCLK: track 41.5 -> 34.7 mm
- net REC_5V_EN: track 37.1 -> 40.9 mm
- net A4: track 14.3 -> 11.0 mm
- net N$15: track 4.03 -> 7.18 mm
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
Commit message: Added different switch footprints
Parts:
- removed GSM_ON_OFF_SW: GSM Power, 1101M2S3CQE2:SW_1101M2S3CQE2
- removed REC_SW: Push_Button, 800AWSP9M2QE:800AWSP9M2QE
- added GSM_ON_OFF_SW1: GSM Power, EG1218:3PIN_SLIDE_SWITCH
- added REC_SW1: Push_Button, 1-1825910-4:TE_1-1825910-4
- REC_ON_OFF_SW: device 1101M2S3CQE2:SW_1101M2S3CQE2 -> EG1218:3PIN_SLIDE_SWITCH
- moved REC_ON_OFF_SW 1.80 mm to (43.2, 76.2), turned to 0 degrees
Connections:
- net GND: now also GSM_ON_OFF_SW1.2, REC_SW1.1, REC_SW1.2; no longer GSM_ON_OFF_SW.1, REC_SW.1
- net GSM_5V_EN: now also GSM_ON_OFF_SW1.1; no longer GSM_ON_OFF_SW.2
- net PWM3: now also REC_SW1.3, REC_SW1.4; no longer REC_SW.3
Routing:
- net PWM3: track 21.2 -> 29.3 mm
- net GND: track 454.7 -> 459.9 mm
- net GSM_5V_EN: track 21.7 -> 19.4 mm
- net REC_5V_EN: track 40.9 -> 41.8 mm
Other:
- board outline added: 87.6 x 80 mm
