File: Teensy36_I2S_Proto/wildly_teensy_proto.brd (EAGLE design)
At the start: 87.6 x 80 mm, 43 parts, among them J1 61300311121, J2 61300311121, T1 2N2222A, T2 2N2222A, T3 2N2222A, T4 2N2222A

Commit message: Power section shifted to one side along with LED's shifted downand track width increased
Parts:
- removed GSM_ON_OFF_SW1: GSM Power, EG1218:3PIN_SLIDE_SWITCH
- removed GSM_POWER_JUMPER: (no value), jumper:JP1
- removed REC_ON_OFF_SW: Microcontroller and Mic Power, EG1218:3PIN_SLIDE_SWITCH
- removed REC_POWER: (no value), adafruit:JST-PH-2-SMT-RA
- removed WILDLY_5V_0.5A_BOOST: (no value), adafruit:1X06
- added 5V_INPUT: 61300211121, 61300211121:61300211121
- added BATT: (no value), adafruit:JST-PH-2-SMT-RA
- added JP1: (no value), jumper:JP1
- added ON_OFF_SW: GSM Power, EG1218:3PIN_SLIDE_SWITCH
- moved WILDLY_5V_1A_BOOST 72.2 mm to (83.8, 63.5), turned to 90 degrees
- moved WILDLY_I2S_MIC 63.9 mm to (38.1, 73.8), turned to 180 degrees
- moved C4 53.7 mm to (74.9, 72.4), turned to 90 degrees
- moved C3 51.6 mm to (72.4, 72.4), turned to 90 degrees
- moved ERRLED 43.7 mm to (33.3, 2.03)
- moved RECLED 29.9 mm to (38.0, 2.03), turned to 90 degrees
- moved NETSTATLED 20.7 mm to (44.1, 2.03)
- moved SDLED 16.9 mm to (49.8, 2.03)
- moved FUEL_GAUGE 13.7 mm to (81.7, 34.5)
- moved J1 13.7 mm to (77.9, 39.6)
- moved J2 13.7 mm to (85.5, 39.6)
- moved R11 13.3 mm to (27.9, 26.7), turned to 0 degrees
- moved R10 9.16 mm to (27.9, 22.9), turned to 0 degrees
- moved SOLAR_CHARGER 8.80 mm to (84.6, 6.48), turned to 270 degrees
- moved R13 7.73 mm to (36.8, 17.8)
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- renumbered TEENSY_1 to TEENSY_PIN_1, TEENSY_2 to TEENSY_PIN_2, TEENSY_3 to TEENSY_PIN_3, TEENSY_4 to TEENSY_PIN_4, TEENSY_5 to TEENSY_PIN_5, TEENSY_6 to TEENSY_PIN_6, TEENSY_7 to TEENSY_PIN_7, TEENSY_8 to TEENSY_PIN_8
Connections:
- net A4 renamed FUEL_GAUGE_SDA
- net A5 renamed FUEL_GAUGE_SCL
- net GSM_LB renamed LB
- removed net GSM_5V: C3.1, C4.1, GSM_POWER_JUMPER.1, MIKROELECTRONIKA_SARA_CLICK.P$10, WILDLY_5V_1A_BOOST.1
- removed net GSM_5V_EN: GSM_ON_OFF_SW1.1, WILDLY_5V_1A_BOOST.5
- removed net GSM_BAT: FUEL_GAUGE.2, SOLAR_CHARGER.1, WILDLY_5V_1A_BOOST.7
- removed net GSM_BAT_RETURN: FUEL_GAUGE.1, SOLAR_CHARGER.2, WILDLY_5V_1A_BOOST.4
- removed net REC_5V: C1.1, C2.1, GSM_POWER_JUMPER.2, TEENSY_PIN_5.1, U$1.VIN, WILDLY_5V_0.5A_BOOST.1
- removed net REC_5V_EN: REC_ON_OFF_SW.1, WILDLY_5V_0.5A_BOOST.4
- removed net REC_BAT: REC_POWER.1, WILDLY_5V_0.5A_BOOST.6
- removed net REC_BAT_RETURN: REC_POWER.2, WILDLY_5V_0.5A_BOOST.5
- removed net REC_LB: WILDLY_5V_0.5A_BOOST.3
- new net 5V_EN: ON_OFF_SW.1, WILDLY_5V_1A_BOOST.5
- new net 5V_SUPPLY: 5V_INPUT.1, C1.1, C2.1, C3.1, C4.1, MIKROELECTRONIKA_SARA_CLICK.P$10, TEENSY_PIN_5.1, U$1.VIN, WILDLY_5V_1A_BOOST.1
- new net VCC: BATT.1, FUEL_GAUGE.2, SOLAR_CHARGER.1, WILDLY_5V_1A_BOOST.7
- net 3V3: now also JP1.1, JP1.2
- net GND: now also 5V_INPUT.2, BATT.2, FUEL_GAUGE.1, ON_OFF_SW.2, SOLAR_CHARGER.2, WILDLY_5V_1A_BOOST.4; no longer GSM_ON_OFF_SW1.2, REC_ON_OFF_SW.2, WILDLY_5V_0.5A_BOOST.2
Routing:
- net GSM_BAT: track 128.8 -> 0.00 mm, vias 2 -> 0
- net 5V_SUPPLY: track 0.00 -> 128.1 mm, vias 0 -> 2
- net GSM_BAT_RETURN: track 121.7 -> 0.00 mm, vias 2 -> 0
- net GND: track 459.9 -> 544.4 mm, vias 21 -> 20
- net VCC: track 0.00 -> 83.7 mm
- net 5V_EN: track 0.00 -> 72.3 mm, vias 0 -> 1
- net REC_5V: track 64.8 -> 0.00 mm
- net N$4: track 13.2 -> 66.2 mm
- net MIC_DOUT: track 16.3 -> 65.8 mm, vias 0 -> 1
- net GSM_5V: track 49.2 -> 0.00 mm, vias 1 -> 0
- net REC_5V_EN: track 41.8 -> 0.00 mm
- net 3V3: track 224.8 -> 187.4 mm, vias 1 -> 2
- net N$2: track 14.3 -> 49.8 mm, vias 0 -> 2
- net N$14: track 5.16 -> 35.1 mm, vias 0 -> 2
- net N$5: track 13.0 -> 42.9 mm, vias 0 -> 1
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Other:
- board size 87.6 x 80 mm -> 87.6 x 77.5 mm
- board text added: "5V"
- board text added: "5V_EN"
- board text added: "VCC"
- board text removed: "GSM_5V"
- board text removed: "GSM_5V_EN"
- board text removed: "GSM_BAT"
- board text removed: "GSM_BAT_RETURN"
- board text removed: "GSM_LB"
- board text removed: "REC_5V"
- board text removed: "REC_5V_EN"
- board text removed: "REC_BAT"
- board text removed: "REC_BAT_RETURN"
- board text removed: "REC_LB"

Commit message: Added new transistor BC847 along with some 0R reistors
Parts:
- added R4, R5, R6: 0R, adafruit:M0805
- T1, T2, T3, T4: value 2N2222A -> BC847BLT1G; device 2N2222A:TO127P584H533-3 -> BC847BLT1G:SOT96P237X111-3N
- moved R13 6.92 mm to (43.7, 16.9)
- moved R1 2.67 mm to (18.9, 40.6)
- moved C3 2.54 mm to (69.8, 72.4)
- moved C4 2.54 mm to (72.4, 72.4)
- moved R3 2.07 mm to (43.7, 49.1)
- moved 5V_INPUT 1.66 mm to (9.27, 74.0)
- moved T2 1.08 mm to (41.4, 32.3)
- moved T1 0.76 mm to (41.4, 44.5)
- moved T4 0.72 mm to (41.4, 11.9)
- moved T3 0.72 mm to (41.4, 22.1)
- moved R2 0.64 mm to (43.8, 39.4)
- moved R9 0.51 mm to (43.7, 26.7)
- moved ON_OFF_SW 0.28 mm to (22.9, 73.7)
Connections:
- net 5V_SUPPLY: now also R4.1, R4.2
- net GND: now also T1.2, T2.2, T3.2, T4.2; no longer T1.1, T2.1, T3.1, T4.1
- net N$11: now also T4.1; no longer T4.2
- net N$3: now also T2.1; no longer T2.2
- net N$7: now also T3.1; no longer T3.2
- net N$8: now also T1.1; no longer T1.2
- net RX_OF_GSM: now also R5.1, R5.2
- net TX_OF_GSM: now also R6.1, R6.2
Routing:
- net GND: track 544.4 -> 524.5 mm
- net SDLED: track 35.7 -> 28.4 mm
- net N$11: track 12.2 -> 5.05 mm
- net 5V_SUPPLY: track 128.1 -> 132.6 mm
- net RTS_OF_GSM: track 80.2 -> 84.8 mm
- net N$5: track 42.9 -> 46.7 mm, vias 1 -> 2
- net N$8: track 8.25 -> 4.79 mm
- net NETSTATLED: track 34.0 -> 31.4 mm
- net PWM3: track 25.5 -> 28.0 mm
- net N$7: track 6.48 -> 4.67 mm
- net N$3: track 9.59 -> 8.42 mm
- net 5V_EN: track 72.3 -> 73.4 mm
- net NET_STAT: track 30.9 -> 31.9 mm
- net RX_OF_GSM: track 57.9 -> 57.2 mm
- net N$1: track 12.6 -> 13.3 mm
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
Commit message: Changed all the power symbols to +5V and 3V3 accordingly
Parts:
- moved JP1 0.54 mm to (44.1, 5.46), turned to 270 degrees
Connections:
- new net +3V3: JP1.1, R10.2, R11.2, R12.2, R14.2
- new net +5V: 5V_INPUT.1, C1.1, C2.1, C3.1, C4.1, MIKROELECTRONIKA_SARA_CLICK.P$10, R4.1, TEENSY_PIN_5.1, U$1.VIN
- net 3V3: no longer JP1.1, R10.2, R11.2, R12.2, R14.2
- net 5V_SUPPLY: no longer 5V_INPUT.1, C1.1, C2.1, C3.1, C4.1, MIKROELECTRONIKA_SARA_CLICK.P$10, R4.1, TEENSY_PIN_5.1, U$1.VIN
Routing:
- net 5V_SUPPLY: track 132.6 -> 19.3 mm, vias 2 -> 1
- net +5V: track 0.00 -> 113.3 mm, vias 0 -> 1
- net +3V3: track 0.00 -> 49.3 mm, vias 0 -> 1
- net 3V3: track 187.4 -> 146.4 mm, vias 2 -> 1
- net N$2: track 49.4 -> 47.8 mm

Commit message: Positioning of filter capacitors along with connections corrected
Parts:
- BATT: value (none) -> B2B-PH-SM4-TB(LF)(SN); device adafruit:JST-PH-2-SMT-RA -> B2B-PH-SM4-TB_LF__SN_:JST_B2B-PH-SM4-TB(LF)(SN)
- moved C4 44.8 mm to (28.4, 63.5), turned to 0 degrees
- moved C3 41.9 mm to (28.4, 66.0), turned to 0 degrees
- moved C1 28.6 mm to (71.8, 71.9), turned to 90 degrees
- moved C2 25.4 mm to (69.2, 71.9), turned to 90 degrees
- moved R1 13.2 mm to (32.0, 39.2), turned to 180 degrees
- moved BATT 5.95 mm to (82.0, 12.2)
- moved SOLAR_CHARGER 5.82 mm to (79.9, 3.05), turned to 180 degrees
- moved R11 4.36 mm to (32.3, 26.0)
- moved R6 3.45 mm to (44.1, 61.8)
- moved R5 2.55 mm to (44.2, 58.4)
- moved SDLED 2.04 mm to (47.8, 1.91)
- moved NETSTATLED 1.40 mm to (42.7, 1.91)
- moved 5V_INPUT 1.28 mm to (8.00, 74.2)
- moved JP1 0.80 mm to (43.8, 6.22)
- moved ERRLED 0.77 mm to (32.5, 1.91)
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Connections:
- removed net A3: TEENSY_PIN_6.4, U$1.17
- new net PWM_SARA: MIKROELECTRONIKA_SARA_CLICK.P$16, TEENSY_PIN_6.4, U$1.17
- net GND: now also BATT.1; no longer BATT.2
- net VCC: now also BATT.2; no longer BATT.1
Routing:
- net PWM_SARA: track 0.00 -> 78.8 mm, vias 0 -> 2
- net GND: track 524.5 -> 504.5 mm, vias 20 -> 21
- net RTS_OF_GSM: track 84.8 -> 76.5 mm
- net N$9: track 15.6 -> 11.4 mm
- net N$4: track 66.3 -> 62.1 mm
- net A3: track 3.81 -> 0.00 mm
- net N$14: track 35.1 -> 32.0 mm, vias 2 -> 0
- net VCC: track 83.7 -> 86.8 mm
- net N$15: track 32.9 -> 35.9 mm
- net +3V3: track 49.3 -> 46.5 mm
- net RESET_GSM: track 56.8 -> 54.3 mm
- net CTS_OF_GSM: track 89.5 -> 87.3 mm
- net N$16: track 13.4 -> 11.6 mm
- net +5V: track 113.3 -> 114.6 mm
- net RX_OF_GSM: track 57.2 -> 58.3 mm
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Other:
- board text added: "Wildly_Listen_Proto_V1"
- board text removed: "Wildly_Listen_Proto_v1"

Commit message: Move capacitors and resistors in layout according to flow of signal as in schematics, rename net names, increase mount hole diameters
Parts:
- moved C3 18.2 mm to (10.7, 62.2)
- moved C4 18.2 mm to (10.7, 59.7)
- moved C1 8.98 mm to (78.1, 65.5), turned to 270 degrees
- moved C2 8.98 mm to (75.6, 65.5), turned to 270 degrees
- moved WILDLY_5V_1A_BOOST 2.54 mm to (83.8, 61.0)
- moved R4 1.80 mm to (75.7, 72.1)
- turned R5 to 180 degrees
- turned R6 to 180 degrees
Connections:
- new net N$10: MIKROELECTRONIKA_SARA_CLICK.P$14, R5.2
- new net N$12: MIKROELECTRONIKA_SARA_CLICK.P$13, R6.2
- net RX_OF_GSM: no longer MIKROELECTRONIKA_SARA_CLICK.P$14, R5.2
- net TX_OF_GSM: no longer MIKROELECTRONIKA_SARA_CLICK.P$13, R6.2
Routing:
- net GND: track 504.5 -> 347.0 mm, vias 21 -> 19
- net N$10: track 0.00 -> 53.5 mm
- net N$12: track 0.00 -> 51.5 mm
- net TX_OF_GSM: track 59.9 -> 9.00 mm, vias 1 -> 0
- net RX_OF_GSM: track 58.3 -> 9.25 mm, vias 1 -> 0
- net 5V_SUPPLY: track 18.7 -> 25.4 mm
- net VCC: track 86.8 -> 80.5 mm
- net +5V: track 114.6 -> 110.1 mm, vias 1 -> 0
- net PWM3: track 27.8 -> 23.6 mm
- net 5V_EN: track 73.4 -> 76.0 mm

Commit message: Rx and Tx connections interchanged and positioning of fuel gauge adjusted
Parts:
- moved J1 4.45 mm to (77.7, 35.2)
- moved J2 4.45 mm to (85.3, 35.2)
- moved FUEL_GAUGE 4.45 mm to (81.5, 30.1)
- moved R6 2.19 mm to (44.5, 64.0)
- moved R5 1.17 mm to (44.5, 59.6)
Connections:
- net RX_OF_GSM: now also R6.1; no longer R5.1
- net TX_OF_GSM: now also R5.1; no longer R6.1
Routing:
- net GND: track 347.0 -> 339.4 mm
- net RX_OF_GSM: track 9.25 -> 14.5 mm
- net FUEL_GAUGE_SDA: track 15.0 -> 19.4 mm
- net FUEL_GAUGE_SCL: track 15.5 -> 19.9 mm
- net VCC: track 80.5 -> 77.9 mm
- net N$10: track 53.5 -> 52.5 mm
- net 5V_EN: track 76.0 -> 76.8 mm
- net 5V_SUPPLY: track 25.4 -> 24.6 mm
- net TX_OF_GSM: track 9.00 -> 9.57 mm
Other:
- board text added: "OFF"
- board text added: "ON"

Commit message: Added the fuel Gauge circuit on board and rearranged the Transistors for grouping and short routing to the LEDs
Parts:
- removed FUEL_GAUGE: 61300211121, 61300211121:61300211121
- removed J1, J2: 61300311121, 61300311121:61300311121
- added C5: 1uF, rcl:C0805
- added C6: 10nF, rcl:C0805
- added IC1: MAX17043G+T, MAX17043G+T:SON50P300X200X80-9N
- added R15, R16: 4.7K, adafruit:M0805
- added R17, R18: 0R, adafruit:M0805
- added R7: 1K, adafruit:M0805
- added R8: 180R, adafruit:M0805
- R10, R11, R12, R14: value 82R -> 870R
- moved R2 24.2 mm to (35.1, 16.8), turned to 180 degrees
- moved R3 24.2 mm to (34.8, 26.7)
- moved T1 23.2 mm to (35.1, 22.1)
- moved T2 21.0 mm to (35.2, 12.2)
- moved R11 20.7 mm to (25.0, 6.60), turned to 180 degrees
- moved R10 16.3 mm to (29.5, 6.60), turned to 180 degrees
- moved R12 3.05 mm to (34.0, 6.60)
- moved R14 2.03 mm to (38.4, 6.60)
- moved R9 1.78 mm to (41.9, 26.7)
- moved T4 1.42 mm to (42.8, 12.2)
- moved T3 1.40 mm to (42.8, 22.1)
- moved R13 1.15 mm to (42.5, 16.8)
- moved C3 1.14 mm to (10.7, 63.4)
- moved JP1 0.76 mm to (43.8, 6.99)
- moved C4 0.51 mm to (10.7, 60.2)
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- renumbered ON_OFF_SW to SWITCH
Connections:
- removed net N$13: J1.3
- new net FUEL_GAUGE_ALT: IC1.5
- new net FUEL_GAUGE_QST: IC1.6
- new net N$12: C5.1, IC1.2, R7.1
- new net N$18: C6.1, IC1.3, R8.2
- new net SCL: IC1.7, R16.2, R18.1
- new net SDA: IC1.8, R15.2, R17.1
- net FUEL_GAUGE_SCL: now also R18.2; no longer J1.2
- net FUEL_GAUGE_SDA: now also R17.2; no longer J1.1
- net GND: now also BATT.2, C5.2, C6.2, IC1.1, IC1.4, IC1.9; no longer BATT.1, FUEL_GAUGE.1
- net VCC: now also BATT.1, R15.1, R16.1, R7.2, R8.1; no longer BATT.2, FUEL_GAUGE.2
Routing:
- net N$2: track 46.8 -> 16.2 mm
- net N$15: track 35.9 -> 8.24 mm
- net N$4: track 62.1 -> 36.9 mm, vias 0 -> 2
- net N$14: track 32.0 -> 8.07 mm
- net VCC: track 77.9 -> 98.4 mm, vias 0 -> 2
- net N$18: track 0.00 -> 19.2 mm
- net +3V3: track 46.5 -> 29.6 mm, vias 1 -> 0
- net RECLED: track 54.7 -> 39.1 mm, vias 2 -> 1
- net N$5: track 47.4 -> 33.7 mm
- net N$12: track 0.00 -> 11.7 mm
- net FUEL_GAUGE_SCL: track 19.9 -> 9.23 mm
- net FUEL_GAUGE_SDA: track 19.4 -> 9.98 mm
- net SCL: track 0.00 -> 9.26 mm
- net SDA: track 0.00 -> 8.74 mm
- net ERRLED: track 46.1 -> 39.5 mm, vias 1 -> 0
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
Commit message: Finalized Proto board with 3 way and 2 way switches included for on/off GSM and for on/off/test the board
Parts:
- removed C5: 1uF, rcl:C0805
- removed C6: 10nF, rcl:C0805
- removed IC1: MAX17043G+T, MAX17043G+T:SON50P300X200X80-9N
- removed R15, R16: 4.7K, adafruit:M0805
- removed R17, R18: 0R, adafruit:M0805
- removed R7: 1K, adafruit:M0805
- removed R8: 180R, adafruit:M0805
- added J1: 61300211121, 61300211121:61300211121
- added J2, J3: 61300311121, 61300311121:61300311121
- added JP2, JP3: (no value), jumper:JP1
- added SWITCH_1: On/Off/Test Switch, OS103011MS8QP1:OS103011MS8QP1
- moved SWITCH 21.0 mm to (3.56, 65.3), turned to 90 degrees
- moved WILDLY_I2S_MIC 4.07 mm to (42.2, 74.0)
- moved SOLAR_CHARGER 4.07 mm to (75.8, 2.79)
- moved 5V_INPUT 3.06 mm to (11.0, 74.4)
Connections:
- removed net FUEL_GAUGE_ALT: IC1.5
- removed net FUEL_GAUGE_QST: IC1.6
- removed net SCL: IC1.7, R16.2, R18.1
- removed net SDA: IC1.8, R15.2, R17.1
- new net N$13: JP2.2, JP3.1, WILDLY_5V_1A_BOOST.7
- net +5V: now also SWITCH.2; no longer C3.1, C4.1, MIKROELECTRONIKA_SARA_CLICK.P$10
- net 5V_EN: now also SWITCH_1.1; no longer SWITCH.1
- net FUEL_GAUGE_SCL: now also J2.2; no longer R18.2
- net FUEL_GAUGE_SDA: now also J2.1; no longer R17.2
- net GND: now also J1.2, SWITCH_1.2, SWITCH_1.5, SWITCH_1.6; no longer C5.2, C6.2, IC1.1, IC1.4, IC1.9, SWITCH.2
- net N$12: now also J3.1, JP2.1; no longer C5.1, IC1.2, R7.1
- net N$18: now also C3.1, C4.1, MIKROELECTRONIKA_SARA_CLICK.P$10, SWITCH.1; no longer C6.1, IC1.3, R8.2
- net POWER_CONTRL: now also SWITCH_1.3
- net VCC: now also J1.1, JP3.2; no longer R15.1, R16.1, R7.2, R8.1, WILDLY_5V_1A_BOOST.7
Routing:
- net GND: track 337.9 -> 9.42 mm, vias 16 -> 1
- net POWER_CONTRL: track 3.81 -> 88.8 mm, vias 0 -> 2
- net VCC: track 98.4 -> 49.4 mm, vias 2 -> 0
- net N$13: track 0.00 -> 28.8 mm
- net +5V: track 111.6 -> 97.3 mm
- net FUEL_GAUGE_SCL: track 9.23 -> 19.3 mm
- net FUEL_GAUGE_SDA: track 9.98 -> 19.8 mm
- net SCL: track 9.26 -> 0.00 mm
- net SDA: track 8.74 -> 0.00 mm
- net 3V3: track 146.2 -> 140.5 mm
- net N$12: track 11.7 -> 6.31 mm
- net MIC_LRCLK: track 47.3 -> 43.4 mm
- net MIC_DOUT: track 66.4 -> 62.5 mm
- net MIC_BCLK: track 48.9 -> 45.0 mm
- net N$18: track 19.2 -> 21.6 mm
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Other:
- board text added: "FUEL_GAUGE"
- board text added: "TEST"
