File: Teensy_I2S_Proto/wildly_teensy_proto.sch (EAGLE design)
At the start: 25 parts, among them CON1 MIKROE_BUS_CONN, SW2 Push_Button

Commit message: Compoenent placement, Ground plane, drill holes etc on the layout
Parts:
- removed CN1, CN2: (no value), adafruit:JST_2PIN-SMT-RA
- removed ERRLED, GSM_LOW_BAT_LED, NETSTATLED, POWERLED, RECLED, REC_LOW_BAT_LED, SDLED: (no value), adafruit:LEDCHIP-LED0805
- removed R9: 330R, adafruit:R-US_M0805
- removed S1: Microcontroller and Mic power, adafruit:31-XXSKINNY
- removed S2: GSM power, adafruit:31-XXSKINNY
- added LED1, LED2, LED3, LED4, LED5: (no value), adafruit:LEDCHIP-LED0805
- added LED6: RGBLED5050, adafruit:RGBLED5050
- added R2: (no value), adafruit:R-US_M0805
- added SW1: SPST_TACT-KMR2, adafruit:SPST_TACT-KMR2
- added X1: ANTENNA, adafruit:SMACONNECTOR
- R1: value 1KR -> (none)
- R3, R4, R5, R6, R7, R8: value 330R -> (none)
- SW2: value Push_Button -> (none)
Connections:
- removed net 3V: JP3.1, U$1.3V3
- removed net BCLK: JP3.3, U$1.9/PWM/RX2/CS0-1
- removed net CTS_OF_GSM: CON1.INT, U$1.33/A14/CAN1TX/TX5/ALT-SCL0
- removed net DOUT: JP3.4, U$1.13/LED/ALT-PWM/SCK0
- removed net GND: CN2.1, CON1.GND1, CON1.GND2, ERRLED.C, GSM_LOW_BAT_LED.C, JP1.2, JP2.2, JP2.4, JP3.2, NETSTATLED.C, POWERLED.C, R1.1, RECLED.C, REC_LOW_BAT_LED.C, S1.S, S2.P, SDLED.C, SW2.P$1, U$1.GND
- removed net LRCLK: JP3.5, U$1.23/A9/PWM/T
- removed net N$10: JP1.3, R3.1
- removed net N$11: ERRLED.A, R8.2
- removed net N$12: R5.1, U$1.39/A20/ALT-MISO0
- removed net N$13: R6.2, U$1.36/A17/PWM
- removed net N$14: R8.1, U$1.37/A18/PWM/SCL1
- removed net N$15: POWERLED.A, R4.1
- removed net N$16: R3.2, REC_LOW_BAT_LED.A
- removed net N$17: CN1.1
- removed net N$18: JP1.5
- removed net N$19: JP2.5, S2.S
- removed net N$2: JP1.1, U$1.5V
- removed net N$20: JP2.3, R9.1
- removed net N$21: R7.1, U$1.38/A19/PWM/SDA1
- removed net N$23: GSM_LOW_BAT_LED.A, R9.2
- removed net N$24: CN2.2, JP2.7
- removed net N$25: CON1.5V, JP2.1
- removed net N$3: CN1.2, JP1.6
- removed net N$4: JP1.4, S1.P
- removed net N$5: R4.2, U$1.35/A16/PWM
- removed net N$7: NETSTATLED.A, R7.2
- removed net N$8: R5.2, SDLED.A
- removed net N$9: R6.1, RECLED.A
- removed net RESET_GSM: CON1.RST, U$1.20/A6/PWM/CS0-2/ALT-SCK1
- removed net RTS_OF_GSM: CON1.CS, R1.2, U$1.34/A15/CAN1RX/RX5/ALT-SDA0
- removed net RX_OF_GSM: CON1.RX, U$1.1/TX1/MISO1/T
- removed net TX_OF_GSM: CON1.TX, U$1.0/RX1/MOSI1/T
- net N$1: now also CON1.AN, X1.ANT; no longer SW2.P$2, U$1.4/PWM/SDA2/CAN0RX
Other:
- note added: "5V Boost 500mA"
- note added: "Microphone In"
- note removed: "5V"
- note removed: "5V Out EN - Recorder On/Off"
- note removed: "5V Out EN - Transmitter On/Off"
- note removed: "Adafruit 5V Boost 500mA"
- note removed: "Adafruit I2S Microphone SPH0645LM4H"
- note removed: "Bat"
- note removed: "EN"
- note removed: "GND"
- note removed: "LB"
- note removed: "Low Battery Indicator"
- note removed: "VBAT"
- note removed: "VS"
- note removed: "VUSB"
- moved on the sheet: JP1, JP3, R1, R3, R4, R5, R6, R7, R8, SW2
