File: SARA_U201_BREAKOUT_BOARD/SARA_U201.brd (EAGLE design)
At the start: 103.9 x 69.8 mm, 54 parts, among them J6 -, T1 BC847, U1 LT1764AEQ#PBF, U2 SN74AVC4T774, U3 SN74AVC4T774, X1 CCM03-3013LFT_R102

Commit message: Updated Layout with changed footprint for level shifters and SARA-U201
Parts:
- removed U$1: SARA_U201, SARA_U201:SARA_U201
- added U4: SARA-U201-03B, SARA-U201-03B:SARA-U201-03B
- C4: value 10uF -> 100nF
- R13: value 9K1 -> 6K8
- U2, U3: value SN74AVC4T774 -> SN74AVC4T774PW; device Arduino-ICs:RSV -> SN74AVC4T774PW:SOP65P640X120-16N
- moved R20 19.4 mm to (41.7, 48.3)
- moved C4 18.0 mm to (62.5, 21.1), turned to 0 degrees
- moved TP3 14.8 mm to (62.0, 49.8)
- moved TP1 6.89 mm to (64.8, 51.3)
- moved TP2 6.81 mm to (52.3, 52.8)
- moved TP4 6.12 mm to (56.1, 56.9)
- moved U2 4.13 mm to (45.2, 56.4), turned to 270 degrees
- moved C16 2.42 mm to (18.3, 55.9)
- moved U3 2.34 mm to (60.5, 56.4), turned to 270 degrees
- moved TP5 1.77 mm to (74.4, 53.3)
- moved C10 0.81 mm to (11.7, 48.8)
- moved C21 0.76 mm to (44.2, 22.5)
- moved C20 0.51 mm to (38.5, 27.0)
- moved C22 0.51 mm to (36.0, 22.5)
- moved C3 0.12 mm to (18.5, 47.8)
Connections:
- removed net GND1: U2.16, U2.5, U2.6
- removed net N$10: U$1.1, U$1.3, U$1.5
- net ANT: now also U4.56; no longer U$1.56
- net ANT_DET: now also U4.62; no longer U$1.62
- net CODEC_CLK: now also U4.19; no longer U$1.19
- net CTS: now also U3.6; no longer U3.4
- net CTS1: now also U3.11, U4.11; no longer U$1.11, U3.9
- net DCD: now also U2.6; no longer U2.4
- net DCD1: now also U2.11, U4.8; no longer U$1.8, U2.9
- net DSR: now also U2.4; no longer U2.2
- net DSR1: now also U2.13, U4.6; no longer U$1.6, U2.11
- net DTR: now also U2.3; no longer U2.1
- net DTR1: now also U2.14, U4.9; no longer U$1.9, U2.12
- net GND: now also U2.10, U2.2, U2.7, U2.8, U2.9, U3.1, U3.10, U3.9, U4.1, U4.20, U4.21, U4.22, U4.3, U4.32, U4.33, U4.43, U4.5, U4.50, U4.54, U4.55, U4.57, U4.58, U4.59, U4.60, U4.61, U4.63, U4.64, U4.65, U4.66, U4.67, U4.68, U4.69, U4.70, U4.71, U4.72, U4.73, U4.74, U4.75, U4.76, U4.77, U4.78, U4.79, U4.80, U4.81, U4.82, U4.83, U4.84, U4.85, U4.86, U4.87, U4.88, U4.89, U4.90, U4.91, U4.92, U4.93, U4.94, U4.95, U4.96; no longer U$1.20, U$1.21, U$1.22, U$1.32, U$1.33, U$1.43, U$1.50, U$1.54, U$1.55, U$1.57, U$1.58, U$1.59, U$1.60, U$1.61, U$1.63, U$1.64, U$1.65, U$1.66, U$1.67, U$1.68, U$1.69, U$1.70, U$1.71, U$1.72, U$1.73, U$1.74, U$1.75, U$1.76, U$1.77, U$1.78, U$1.79, U$1.80, U$1.81, U$1.82, U$1.83, U$1.84, U$1.85, U$1.86, U$1.87, U$1.88, U$1.89, U$1.90, U$1.91, U$1.92, U$1.93, U$1.94, U$1.95, U$1.96, U3.16, U3.6, U3.7
- net GND2: now also U4.14; no longer U$1.14, U2.7, U2.8
- net GPIO2: now also U4.23; no longer U$1.23
- net GPIO3: now also U4.24; no longer U$1.24
- net GPIO4: now also U4.25; no longer U$1.25
- net I2S_CLK: now also U4.36; no longer U$1.36
- net I2S_RXD: now also U4.37; no longer U$1.37
- net I2S_TXD: now also U4.35; no longer U$1.35
- net I2S_WA: now also U4.34; no longer U$1.34
- net NET_STAT: now also U4.16; no longer U$1.16
- net PWR_ON: now also U4.15; no longer U$1.15
- net RI: now also U2.5; no longer U2.3
- net RI1: now also U2.12, U4.7; no longer U$1.7, U2.10
- net RST: now also U4.18; no longer U$1.18
- net RTS: now also U3.5; no longer U3.3
- net RTS1: now also TP2.TP, U3.12, U4.10; no longer TP3.TP, U$1.10, U3.10
- net RXD: now also U3.3; no longer U3.2
- net RXD1: now also TP3.TP, U3.13, U4.13; no longer TP2.TP, U$1.13, U3.11
- net SCL: now also U4.27; no longer U$1.27
- net SDA: now also U4.26; no longer U$1.26
- net SIM_CLK: now also U4.38; no longer U$1.38
- net SIM_DET: now also U4.42; no longer U$1.42
- net SIM_I/O: now also U4.39; no longer U$1.39
- net SIM_RST: now also U4.40; no longer U$1.40
- net TXD: now also U3.4; no longer U3.1
- net TXD1: now also U3.14, U4.12; no longer U$1.12, U3.12
- net USB_D+: now also U4.29; no longer U$1.29
- net USB_D-: now also U4.28; no longer U$1.28
- net USB_GND: now also U4.30; no longer U$1.30
- net VCC: now also U2.1, U2.16, U3.16, U3.2, U3.7, U4.51, U4.52, U4.53; no longer U$1.51, U$1.52, U$1.53, U2.14, U2.15, U3.14, U3.15, U3.5
- net VCCINT: now also U2.15, U3.15, U4.4; no longer U$1.4, U2.13, U3.13
- net VSIM: now also U4.41; no longer U$1.41
- net VUSB_DET: now also U4.17; no longer U$1.17
- net V_BCKP: now also U4.2; no longer U$1.2
Routing:
- net GND2: track 94.1 -> 10.1 mm
- net TXD1: track 107.9 -> 26.2 mm, vias 6 -> 4
- net VUSB_DET: track 139.2 -> 199.1 mm, vias 6 -> 11
- net GND: track 971.4 -> 924.7 mm, vias 416 -> 342
- net VCC: track 175.4 -> 219.5 mm, vias 13 -> 18
- net ANT: track 5.22 -> 38.2 mm, vias 0 -> 4
- net USB_GND: track 51.1 -> 83.2 mm, vias 4 -> 6
- net GPIO3: track 71.7 -> 101.3 mm, vias 2 -> 3
- net USB_D-: track 80.1 -> 108.6 mm, vias 7 -> 11
- net V_BCKP: track 83.0 -> 54.7 mm, vias 4 -> 0
- net SCL: track 44.8 -> 73.1 mm, vias 1 -> 4
- net SDA: track 43.2 -> 71.0 mm, vias 3 -> 5
- net GPIO2: track 73.5 -> 100.3 mm
- net I2S_WA: track 31.3 -> 57.9 mm, vias 0 -> 4
- net CODEC_CLK: track 92.6 -> 118.5 mm, vias 2 -> 4
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Other:
- board text added: "C3"

Commit message: Added the USB switch and power LED
Parts:
- added IC1: TS3USB221ERSER, TS3USB221ERSER:TS3USB221ERSER
- added LED1: SML-LX0805GC-TR, SML-LX0805GC-TR:LEDC2012X120N
- added R1: 470, rcl:R0805
- moved TP4 2.59 mm to (53.6, 56.4)
- moved TP2 1.05 mm to (51.3, 52.6)
- moved TP3 0.92 mm to (61.5, 49.0)
- moved TP1 0.36 mm to (65.0, 51.6)
- moved JP2 0.28 mm to (100.2, 51.1), turned to 90 degrees
Connections:
- new net MC_USB_D+: IC1.1, JP4.3
- new net MC_USB_D-: IC1.2, JP4.2
- new net M_USB_D+: ESD3.3, IC1.3, USB.3
- new net M_USB_D-: ESD3.2, IC1.4, USB.4
- new net N$1: LED1.C, R1.2
- new net SW_EN: IC1.6, JP2.1
- new net SW_SEL: IC1.9, JP2.2
- new net USB_D+1: JP2.3
- new net USB_GND1: JP2.4
- net +5V: now also LED1.A
- net GND: now also R1.1; no longer JP2.2
- net SCL: no longer JP2.3
- net SDA: no longer JP2.4
- net USB_D+: now also IC1.8; no longer ESD3.3, JP4.3, USB.3
- net USB_D-: now also IC1.7; no longer ESD3.2, JP4.2, USB.4
- net USB_GND: now also IC1.5
- net VCC: now also IC1.10
- net VCCINT: no longer JP2.1
Routing:
- net USB_D-: track 108.6 -> 61.0 mm, vias 11 -> 8
- net SCL: track 73.1 -> 36.0 mm, vias 4 -> 3
- net M_USB_D+: track 0.00 -> 33.5 mm, vias 0 -> 4
- net M_USB_D-: track 0.00 -> 31.1 mm, vias 0 -> 3
- net USB_D+: track 90.3 -> 64.7 mm, vias 7 -> 6
- net VCCINT: track 136.7 -> 113.0 mm, vias 10 -> 8
- net SDA: track 71.0 -> 47.7 mm, vias 5 -> 4
- net MC_USB_D-: track 0.00 -> 22.4 mm, vias 0 -> 1
- net SW_EN: track 0.00 -> 22.1 mm, vias 0 -> 1
- net MC_USB_D+: track 0.00 -> 20.4 mm, vias 0 -> 1
- net SW_SEL: track 0.00 -> 18.2 mm, vias 0 -> 1
- net VCC: track 219.5 -> 236.6 mm, vias 18 -> 19
- net VUSB_DET: track 199.1 -> 185.8 mm
- net GND: track 924.7 -> 935.8 mm
- net USB_GND: track 83.2 -> 89.6 mm
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Other:
- board text added: "C4"
- board text removed: "JP2"
- board text removed: "SCL"
- board text removed: "SDA"
- board text removed: "VCCINT"

Commit message: Changed the pad for L2 and used minimum no. of vias to connect to the USB switch
Parts:
- L2: device rcl:L1812 -> 490-15685-1-ND:FB_BLM18PG121SN1D
- moved L2 2.40 mm to (30.8, 36.6), turned to 270 degrees
- moved IC1 0.25 mm to (87.9, 38.4), turned to 90 degrees
Connections:
- net GND: now also L2.1; no longer L2.2
- net N$7: now also L2.2; no longer L2.1
Routing:
- net USB_D+: track 64.7 -> 54.1 mm, vias 6 -> 4
- net MC_USB_D-: track 22.4 -> 12.5 mm, vias 1 -> 0
- net USB_GND: track 89.6 -> 99.3 mm, vias 6 -> 5
- net USB_D-: track 61.0 -> 52.1 mm, vias 8 -> 4
- net MC_USB_D+: track 20.4 -> 11.7 mm, vias 1 -> 0
- net SW_SEL: track 18.2 -> 24.7 mm
- net M_USB_D-: track 31.1 -> 37.3 mm, vias 3 -> 2
- net VCC: track 236.6 -> 242.6 mm
- net M_USB_D+: track 33.5 -> 28.0 mm, vias 4 -> 2
- net SW_EN: track 22.1 -> 16.8 mm
- net VUSB_DET: track 185.8 -> 182.9 mm, vias 11 -> 12
- net GPIO2: track 100.9 -> 103.7 mm, vias 2 -> 4
- net GND: track 935.8 -> 933.3 mm
- net GPIO3: track 101.9 -> 103.9 mm, vias 3 -> 5
- net N$5: track 73.3 -> 71.3 mm
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
Commit message: Added Teensy, MIC, Boost connectors along with some layout changes with USB switch and rerouting all the connections
Parts:
- removed C1, C2: 100nF, rcl:C0805
- removed H1, H2, H3, H4: MOUNT-HOLE3.0, holes:3,0
- removed J6: -, Arduino-connectors:U.FL-R-SMT-1(60)
- removed JP1: (no value), pinhead:1X13
- removed TP1, TP2, TP3, TP4: TPB1,27, testpad:B1,27
- removed U1: LT1764AEQ#PBF, LT1764AEQ_PBF:DDPAK-5_Q
- removed U3: SN74AVC4T774PW, SN74AVC4T774PW:SOP65P640X120-16N
- added C11, C13: (no value), rcl:C0805
- added IC2: MCP1826T-3302E_DC, MCP1826T-3302E_DC:SOT127P706X180-6N
- added J1: SMA_CONNECTOR, SMA_CONNECTOR:LPRS_SMA_CONNECTOR
- added J3, SOLAR_CHARGER: 61300211121, 61300211121:61300211121
- added J4, J5: 61300311121, 61300311121:61300311121
- added R3: 100K, rcl:R0805
- added R4, R5, R6: 0R, adafruit:M0805
- added SWITCH: GSM Power, EG1218:3PIN_SLIDE_SWITCH
- added U$1: TEENSY3_6--ALLPINS, Teensy_3_6:T36
- added WILDLY_5V_1A_BOOST: (no value), adafruit:1X08-BIG
- added WILDLY_I2S_MIC: (no value), adafruit:1X06
- C7: value 10uF -> 2.2uF
- J2: value (none) -> B2B-PH-SM4-TB(LF)(SN); device SparkFun-Connectors:JST-2-SMD -> B2B-PH-SM4-TB_LF__SN_:JST_B2B-PH-SM4-TB(LF)(SN)
- R13: value 6K8 -> 10K
- R14: value 3K9 -> 1K
- U2: value SN74AVC4T774PW -> TXB0106PWR; device SN74AVC4T774PW:SOP65P640X120-16N -> TXB0106PWR:SOP65P640X120-16N
- moved LED1 92.0 mm to (102.1, 13.4), turned to 270 degrees
- moved R1 90.8 mm to (98.8, 13.4), turned to 90 degrees
- moved ESD1 76.5 mm to (18.6, 70.0), turned to 0 degrees
- moved JP3 74.4 mm to (87.2, 77.7)
- moved X1 61.4 mm to (39.8, 70.7)
- moved C10 59.2 mm to (66.3, 25.9), turned to 90 degrees
- moved C22 56.9 mm to (57.4, 75.2), flipped to the bottom
- moved ESD2 55.1 mm to (57.8, 70.9), flipped to the bottom, turned to 180 degrees
- moved C18 54.2 mm to (18.5, 74.7), flipped to the bottom
- moved R11 54.0 mm to (18.5, 77.5), flipped to the bottom, turned to 180 degrees
- moved C21 51.9 mm to (62.9, 70.9), flipped to the bottom, turned to 270 degrees
- moved C6 46.1 mm to (60.7, 65.3), flipped to the bottom
- moved C19 45.0 mm to (18.5, 65.8), flipped to the bottom, turned to 180 degrees
- moved R14 44.5 mm to (5.82, 74.0)
- moved C20 42.8 mm to (57.7, 65.3), flipped to the bottom
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Connections:
- removed net DCD: JP1.8, U2.6
- removed net DSR: JP1.6, U2.4
- removed net DTR: JP1.5, U2.3
- new net 5V_EN: SWITCH.1, WILDLY_5V_1A_BOOST.5
- new net 5V_SUPPLY: R4.2, WILDLY_5V_1A_BOOST.1
- new net FUEL_GAUGE_SCL: J4.2, U$1.19
- new net FUEL_GAUGE_SDA: J4.1, U$1.18
- new net LB: WILDLY_5V_1A_BOOST.3
- new net MIC_BCLK: U$1.9, WILDLY_I2S_MIC.3
- new net MIC_DOUT: U$1.13, WILDLY_I2S_MIC.4
- new net MIC_LRCLK: U$1.23, WILDLY_I2S_MIC.5
- new net N$2: IC2.5, R13.2, R3.1
- new net N$4: WILDLY_5V_1A_BOOST.6
- new net STAT: U$1.24, U2.16
- new net V+: C8.1, IC2.1, IC2.2, J2.1, J3.1, SOLAR_CHARGER.1, WILDLY_5V_1A_BOOST.7
- new net VDD: C4.2, C7.1, IC2.4, R15.2, R3.2, U4.51, U4.52, U4.53
- net +5V: now also C11.1, C13.1, R4.1, U$1.VIN; no longer C8.1, J2.2, JP1.10, U1.1, U1.2
- net CTS: now also U$1.33, U2.12; no longer JP1.4, U3.6
- net CTS1: now also U2.5; no longer TP4.TP, U3.11
- net DCD1: no longer U2.11
- net DSR1: no longer U2.13
- net DTR1: no longer U2.14
- net GND: now also C11.2, C13.2, IC2.3, IC2.6, J1.2, J1.3, J1.4, J1.5, J2.2, J3.2, SOLAR_CHARGER.2, SWITCH.2, U$1.G0, U$1.G1, U$1.G2, U$1.G3, U$1.G4, U$1.G5, U$1.G6, WILDLY_5V_1A_BOOST.2, WILDLY_5V_1A_BOOST.4, WILDLY_I2S_MIC.2; no longer C1.2, C2.2, J2.1, J6.GND1, J6.GND2, JP1.9, U1.3, U1.6, U2.10, U2.2, U2.7, U2.8, U3.1, U3.10, U3.8, U3.9
- net MC_USB_D+: now also U$1.D+
- net MC_USB_D-: now also U$1.D-
- net N$3: no longer U1.5
- net N$6: now also J1.1; no longer J6.SIG
- net NET_STAT: now also U2.1
- net PWR_ON: now also U$1.35; no longer JP1.11
- net RI: now also U$1.17, U2.10; no longer JP1.7, U2.5
- net RI1: now also U2.7; no longer U2.12
- net RST: now also U$1.20; no longer JP1.12
- net RTS: now also U$1.34, U2.11; no longer JP1.3, U3.5
- net RTS1: now also U2.6; no longer TP2.TP, U3.12
- net RXD: now also R6.1, R6.2, U$1.1, U2.13; no longer JP1.2, U3.3
- net RXD1: now also U2.3; no longer TP3.TP, U3.13
- net TXD: now also R5.1, R5.2, U$1.0, U2.14; no longer JP1.1, U3.4
- net TXD1: now also U2.4; no longer TP1.TP, U3.14
- net VCC: now also U$1.3V3(1), U$1.3V3(2), U$1.3V3(3), U$1.3V3(4), U2.15, WILDLY_I2S_MIC.1; no longer C2.1, C4.2, C7.1, JP1.13, R13.2, R15.2, U1.4, U2.1, U2.16, U3.16, U3.2, U3.7, U4.51, U4.52, U4.53
- net VCCINT: now also U2.2, U2.8; no longer C1.1, U2.15, U3.15
- net VUSB_DET: now also U$1.VUSB
Routing:
- net GND: track 933.3 -> 0.00 mm, vias 342 -> 0
- net VCC: track 242.6 -> 116.6 mm, vias 19 -> 1
- net RTS1: track 104.5 -> 10.3 mm, vias 2 -> 0
- net FUEL_GAUGE_SCL: track 0.00 -> 76.0 mm
- net FUEL_GAUGE_SDA: track 0.00 -> 72.4 mm
- net N$6: track 18.5 -> 88.7 mm, vias 2 -> 3
- net V+: track 0.00 -> 64.9 mm
- net MIC_LRCLK: track 0.00 -> 62.7 mm
- net VDD: track 0.00 -> 59.5 mm
- net CODEC_CLK: track 118.7 -> 61.0 mm, vias 6 -> 2
- net GPIO3: track 103.9 -> 47.0 mm, vias 5 -> 2
- net MIC_BCLK: track 0.00 -> 56.0 mm
- net N$5: track 71.3 -> 17.2 mm, vias 2 -> 0
- net GPIO2: track 103.7 -> 50.2 mm, vias 4 -> 2
- net VUSB_DET: track 182.9 -> 131.0 mm, vias 12 -> 3
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Other:
- board size 103.9 x 69.8 mm -> 103.9 x 80 mm
- board text added: "C7"
- board text added: "OFF"
- board text added: "ON"
- board text added: "R15"
- board text removed: "+5V"
- board text removed: "ANT DET"
- board text removed: "CODEC CLK"
- board text removed: "CTS"
- board text removed: "DCD"
- board text removed: "DSR"
- board text removed: "DTR"
- board text removed: "GND"
- board text removed: "GPIO2"
- board text removed: "GPIO3"
- board text removed: "GPIO4"
- board text removed: "I2S CLK"
- board text removed: "I2S RXD"
- board text removed: "I2S TXD"
- board text removed: "I2S WA"
- board text removed: "JP1"
- board text removed: "JP3"
- board text removed: "PIN1"
- board text removed: "PWR_ON"
- board text removed: "RI"
- board text removed: "RST"
- board text removed: "RTS"
- board text removed: "RXD"
- board text removed: "TXD"
- board text removed: "USB D+"
- board text removed: "USB D-"
- board text removed: "USB GND"
- board text removed: "VBUS_DET"
- board text removed: "VCC"
- board text removed: "WILDLY HSPA/GSM MODULE"

Commit message: Removed the RST pin connection from Teensy as it requires a level shifter
Connections:
- net RST: no longer U$1.20
Routing:
- net RST: track 149.8 -> 88.9 mm, vias 4 -> 3
Changed lines of the file:
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@@
 <contactref element="ESD1" pad="4"/>
 <contactref element="U4" pad="18"/>
-<contactref element="U$1" pad="20"/>
 <wire x1="17.36140625" y1="69.09239375" x2="16.09140625" y2="67.82239375" width="0.3048" layer="16"/>
 <wire x1="16.09140625" y1="67.82239375" x2="16.09140625" y2="63.91859375" width="0.3048" layer="16"/>
@@
 <wire x1="18.796" y1="59.436" x2="18.542" y2="59.182" width="0.3048" layer="16"/>
 <wire x1="18.542" y1="59.182" x2="18.542" y2="48.514" width="0.3048" layer="16"/>
-<via x="70.358" y="33.02" extent="1-16" drill="0.508"/>
-<wire x1="70.358" y1="33.02" x2="68.326" y2="35.052" width="0.3048" layer="1"/>
-<wire x1="68.326" y1="35.052" x2="66.294" y2="35.052" width="0.3048" layer="1"/>
-<wire x1="66.294" y1="35.052" x2="62.55140625" y2="38.79459375" width="0.3048" layer="1"/>
-<wire x1="62.55140625" y1="40.08819375" x2="62.55140625" y2="38.79459375" width="0.3048" layer="1"/>
-<wire x1="74.83730625" y1="3.678796875" x2="74.83730625" y2="6.25730625" width="0.3048" layer="1"/>
-<wire x1="87.884" y1="13.462" x2="92.202" y2="17.78" width="0.3048" layer="1"/>
-<wire x1="92.202" y1="17.78" x2="92.202" y2="25.654" width="0.3048" layer="1"/>
-<wire x1="74.83730625" y1="6.25730625" x2="82.042" y2="13.462" width="0.3048" layer="1"/>
-<wire x1="82.042" y1="13.462" x2="87.884" y2="13.462" width="0.3048" layer="1"/>
-<wire x1="92.202" y1="25.654" x2="88.646" y2="29.21" width="0.3048" layer="1"/>
-<wire x1="70.104" y1="32.766" x2="70.358" y2="33.02" width="0.3048" layer="16"/>
-<wire x1="34.29" y1="32.766" x2="70.104" y2="32.766" width="0.3048" layer="16"/>
-<via x="77.724" y="29.21" extent="1-16" drill="0.508"/>
-<wire x1="88.646" y1="29.21" x2="77.724" y2="29.21" width="0.3048" layer="1"/>
-<wire x1="77.724" y1="29.21" x2="74.168" y2="29.21" width="0.3048" layer="16"/>
-<wire x1="74.168" y1="29.21" x2="70.358" y2="33.02" width="0.3048" layer="16"/>
+<via x="68.58" y="32.766" extent="1-16" drill="0.508"/>
+<wire x1="68.58" y1="32.766" x2="68.326" y2="32.766" width="0.3048" layer="1"/>
+<wire x1="68.326" y1="32.766" x2="62.55140625" y2="38.54059375" width="0.3048" layer="1"/>
+<wire x1="62.55140625" y1="40.08819375" x2="62.55140625" y2="38.54059375" width="0.3048" layer="1"/>
+<wire x1="34.29" y1="32.766" x2="68.58" y2="32.766" width="0.3048" layer="16"/>
 </signal>
 <signal name="V_BCKP">

Commit message: All the review changes done except a few which need to be discussed
Parts:
- removed ESD1: SOT95P275X110-6N, SOT95P275X110-6N:SOT95P275X110-6N
- removed IC2: MCP1826T-3302E_DC, MCP1826T-3302E_DC:SOT127P706X180-6N
- added IC3: MCP1826T-3302E_DC, MCP1826T-3302E_DC:SOT127P706X180-6N
- added IC6: TS3USB221ERSER, TS3USB221ERSER:TS3USB221ERSER
- added TP1, TP2, TP3: TPB1,27, testpad:B1,27
- IC1: value TS3USB221ERSER -> SOT95P275X110-6N; device TS3USB221ERSER:TS3USB221ERSER -> SOT95P275X110-6N:SOT95P275X110-6N
- moved J1 98.3 mm to (4.56, 44.4)
- moved IC1 74.4 mm to (17.6, 70.0), flipped to the bottom, turned to 0 degrees
- moved C21 7.37 mm to (55.7, 69.5), turned to 90 degrees
- moved JP3 7.37 mm to (79.8, 77.7)
- moved R17 7.01 mm to (25.4, 44.2), turned to 180 degrees
- moved SOLAR_CHARGER 6.61 mm to (2.81, 52.3)
- moved C8 6.10 mm to (11.7, 65.0)
- moved C4 6.06 mm to (40.2, 55.1), turned to 270 degrees
- moved J2 5.61 mm to (5.20, 61.0)
- moved R5 5.04 mm to (71.6, 21.6)
- moved TP5 4.20 mm to (46.5, 36.0)
- moved T1 4.20 mm to (23.0, 48.1)
- moved J3 4.10 mm to (16.3, 24.4)
- moved J4 4.10 mm to (20.1, 29.5)
- moved J5 4.10 mm to (12.4, 29.5)
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- renumbered U$1 to IC8, U2 to IC5, U4 to IC7
Connections:
- net GND: now also IC1.5, IC1.6, IC3.3, IC3.6; no longer ESD1.5, ESD1.6, IC2.3, IC2.6
- net MC_USB_D+: now also IC6.1; no longer IC1.1
- net MC_USB_D-: now also IC6.2; no longer IC1.2
- net M_USB_D+: now also IC6.3; no longer IC1.3
- net M_USB_D-: now also IC6.4; no longer IC1.4
- net N$2: now also IC3.5; no longer IC2.5
- net PWR_ON: now also IC1.1; no longer ESD1.1
- net RST: now also IC1.4; no longer ESD1.4
- net RXD: now also IC5.14; no longer IC5.13
- net SIM_DET: now also IC1.3; no longer ESD1.3
- net SIM_I/O: now also IC1.2; no longer ESD1.2
- net SW_EN: now also IC6.6; no longer IC1.6
- net SW_SEL: now also IC6.9; no longer IC1.9
- net TXD: now also IC5.13; no longer IC5.14
- net USB_D+: now also IC6.8; no longer IC1.8
- net USB_D-: now also IC6.7; no longer IC1.7
- net USB_GND: now also IC6.5; no longer IC1.5
- net V+: now also IC3.1, IC3.2; no longer IC2.1, IC2.2
- net VCC: now also IC6.10, TP2.TP, TP3.TP; no longer IC1.10
- net VDD: now also IC3.4, TP1.TP; no longer IC2.4
Routing:
- net N$6: track 88.7 -> 36.5 mm, vias 3 -> 0
- net V+: track 64.9 -> 74.8 mm
- net VDD: track 59.5 -> 66.6 mm
- net NET_STAT: track 59.9 -> 53.0 mm
- net M_USB_D+: track 20.0 -> 14.3 mm
- net SIM_RST: track 36.8 -> 31.1 mm
- net ANT_DET: track 61.6 -> 56.8 mm
- net VCC: track 116.6 -> 121.2 mm
- net CODEC_CLK: track 61.0 -> 56.8 mm
- net SIM_I/O: track 60.6 -> 56.6 mm
- net M_USB_D-: track 20.1 -> 16.3 mm
- net GPIO2: track 50.2 -> 46.7 mm
- net +5V: track 109.0 -> 105.8 mm
- net VUSB_DET: track 131.0 -> 127.9 mm
- net I2S_WA: track 32.9 -> 29.9 mm
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Other:
- board text added: "5V_EN"
- board text added: "5V_SUPPLY"
- board text added: "ANT_DET"
- board text added: "CODEC_CLK"
- board text added: "GND"
- board text added: "GPIO2"
- board text added: "GPIO3"
- board text added: "GPIO4"
- board text added: "I2S_CLK"
- board text added: "I2S_RXD"
- board text added: "I2S_TXD"
- board text added: "I2S_WA"
- board text added: "MC_USB_D+"
- board text added: "MC_USB_D-"
- board text added: "MIC_BCLK"
- board text added: "MIC_DOUT"
- board text added: "MIC_LRCLK"
- board text added: "SW_EN"
- board text added: "SW_SEL"
- board text added: "USB_GND"
- board text added: "V+"
- board text added: "VCC"
- board text added: "VDD"
- board text added: "VUSB_DET"
