File: SARA_U201_BREAKOUT_BOARD/SARA_U201.brd (EAGLE design)
At the start: 103.9 x 80 mm, 62 parts, among them IC1 SOT95P275X110-6N, IC3 MCP1826T-3302E_DC, IC5 TXB0106PWR, IC6 TS3USB221ERSER, IC7 SARA-U201-03B, IC8 TEENSY3_6--ALLPINS, J1 SMA_CONNECTOR, J2 B2B-PH-SM4-TB(LF)(SN), J3 61300211121, J4 61300311121, J5 61300311121, T1 BC847, X1 CCM03-3013LFT_R102

Commit message: Updated the BOM as well with the schematics and layout
Parts:
- removed LED2: (no value), led:CHIPLED_0603
- added LED3: SML-LX0805GC-TR, SML-LX0805GC-TR:LEDC2012X120N
- renumbered ESD2 to IC2, ESD3 to IC4
Connections:
- removed net N$11: LED2.C, T1.3
- new net N$8: LED3.C, T1.3
- net N$9: now also LED3.A; no longer LED2.A
Routing:
- net N$8: track 0.00 -> 4.54 mm
- net N$11: track 3.40 -> 0.00 mm
- net N$9: track 2.81 -> 3.66 mm
Changed lines of the file:
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@@
 <attribute name="NAME" x="20.612540625" y="49.1143625" size="0.8128" layer="25"/>
-</element>
-<element name="LED2" library="led" library_urn="urn:adsk.eagle:library:259" package="CHIPLED_0603" package3d_urn="urn:adsk.eagle:package:15822/2" value="" x="26.27780625" y="49.71340625" smashed="yes" rot="R180">
-<attribute name="NAME" x="26.98305" y="50.92498125" size="0.8128" layer="25" rot="R270"/>
-<attribute name="VALUE" x="24.37280625" y="50.98340625" size="1.27" layer="27" rot="R270"/>
 </element>
 <element name="R11" library="rcl" library_urn="urn:adsk.eagle:library:334" package="R0805" package3d_urn="urn:adsk.eagle:package:23553/2" value="470K" x="18.529746875" y="77.52176875" smashed="yes" rot="MR180">
@@
 </element>
 <element name="JP3" library="pinhead" library_urn="urn:adsk.eagle:library:325" package="1X09" package3d_urn="urn:adsk.eagle:package:22483/2" value="" x="79.84540625" y="77.72219375" smashed="yes" rot="R180">
-<attribute name="NAME" x="68.91020625" y="77.68639375" size="1.27" layer="25" ratio="10" rot="R90"/>
+<attribute name="NAME" x="67.89420625" y="75.90839375" size="1.27" layer="25" ratio="10" rot="R90"/>
 <attribute name="VALUE" x="91.27540625" y="80.89719375" size="1.27" layer="27" rot="R180"/>
 </element>
-<element name="ESD2" library="SOT95P275X110-6N" package="SOT95P275X110-6N" value="SOT95P275X110-6N" x="59.55140625" y="70.89219375" smashed="yes" rot="MR180">
+<element name="IC2" library="SOT95P275X110-6N" package="SOT95P275X110-6N" value="SOT95P275X110-6N" x="59.55140625" y="70.89219375" smashed="yes" rot="MR180">
 <attribute name="NAME" x="61.554409375" y="72.487053125" size="1.27" layer="26" ratio="10" rot="MR0"/>
 </element>
-<element name="ESD3" library="SOT95P275X110-6N" package="SOT95P275X110-6N" value="SOT95P275X110-6N" x="91.65340625" y="48.72619375" smashed="yes">
-<attribute name="NAME" x="89.61665625" y="50.562871875" size="1.27" layer="25" ratio="10"/>
+<element name="IC4" library="SOT95P275X110-6N" package="SOT95P275X110-6N" value="SOT95P275X110-6N" x="91.65340625" y="48.72619375" smashed="yes">
+<attribute name="NAME" x="90.37865625" y="50.562871875" size="1.27" layer="25" ratio="10"/>
 </element>
 <element name="IC1" library="SOT95P275X110-6N" package="SOT95P275X110-6N" value="SOT95P275X110-6N" x="17.61540625" y="70.03219375" smashed="yes" rot="MR0">
@@
 <attribute name="NAME" x="87.757" y="37.846" size="1.27" layer="25" ratio="10"/>
 <attribute name="TP_SIGNAL_NAME" value="" x="88.519" y="37.973" size="1" layer="37"/>
+</element>
+<element name="LED3" library="SML-LX0805GC-TR" package="LEDC2012X120N" value="SML-LX0805GC-TR" x="27.432" y="50.292" smashed="yes" rot="R90">
+<attribute name="DESCRIPTION" value=" Green 2 x 1.25 mm 0805 140° Water Clear 10 mcd 2.2 V LED SMT " x="27.432" y="50.292" size="1.778" layer="27" rot="R90" display="off"/>
+<attribute name="DIGI-KEY_PART_NUMBER" value="67-2188-1-ND" x="27.432" y="50.292" size="1.778" layer="27" rot="R90" display="off"/>
+<attribute name="DIGI-KEY_PURCHASE_URL" value="https://www.digikey.in/product-detail/en/lumex-opto-components-inc/SML-LX0805GC-TR/67-2188-1-ND/4172828?utm_source=snapeda&amp;utm_medium=aggregator&amp;utm_campaign=symbol" x="27.432" y="50.292" size="1.778" layer="27" rot="R90" display="off"/>
+<attribute name="MF" value="Lumex Opto/Components" x="27.432" y="50.292" size="1.778" layer="27" rot="R90" display="off"/>
+<attribute name="MP" value="SML-LX0805GC-TR" x="27.432" y="50.292" size="1.778" layer="27" rot="R90" display="off"/>
+<attribute name="NAME" x="28.681" y="51.504" size="0.8" layer="25" rot="R270"/>
+<attribute name="PACKAGE" value="0805 Lumex" x="27.432" y="50.292" size="1.778" layer="27" rot="R90" display="off"/>
 </element>
 </elements>
@@
 <contactref element="C19" pad="1"/>
 <contactref element="X1" pad="C5"/>
-<contactref element="ESD2" pad="5"/>
-<contactref element="ESD2" pad="6"/>
+<contactref element="IC2" pad="5"/>
+<contactref element="IC2" pad="6"/>
 <contactref element="IC1" pad="6"/>
 <contactref element="IC1" pad="5"/>
@@
 <contactref element="X1" pad="C3"/>
 <contactref element="C22" pad="2"/>
-<contactref element="ESD2" pad="3"/>
+<contactref element="IC2" pad="3"/>
 <contactref element="IC7" pad="38"/>
 <wire x1="52.13540625" y1="72.00619375" x2="48.708640625" y2="68.579428125" width="0.3048" layer="16"/>
@@
 <contactref element="X1" pad="C2"/>
 <contactref element="C21" pad="2"/>
-<contactref element="ESD2" pad="2"/>
+<contactref element="IC2" pad="2"/>
 <contactref element="IC7" pad="40"/>
 <wire x1="58.784303125" y1="70.892190625" x2="58.28140625" y2="70.89219375" width="0.3048" layer="16"/>
@@
 <contactref element="C20" pad="2"/>
 <contactref element="C6" pad="2"/>
-<contactref element="ESD2" pad="1"/>
+<contactref element="IC2" pad="1"/>
 <contactref element="IC7" pad="41"/>
 <wire x1="52.13540625" y1="66.92619375" x2="52.13540625" y2="61.5812375" width="0.3048" layer="16"/>
@@
 <contactref element="USB" pad="1"/>
 <contactref element="C9" pad="2"/>
-<contactref element="ESD3" pad="5"/>
-<contactref element="ESD3" pad="6"/>
+<contactref element="IC4" pad="5"/>
+<contactref element="IC4" pad="6"/>
 <contactref element="JP4" pad="4"/>
 <contactref element="IC7" pad="30"/>
@@
 <wire x1="24.433515625" y1="44.159653125" x2="26.333515625" y2="44.159653125" width="0" layer="19" extent="1-1"/>
 </signal>
-<signal name="N$9">
-<contactref element="LED2" pad="A"/>
-<contactref element="R15" pad="1"/>
-<wire x1="26.27780625" y1="50.46340625" x2="24.500765625" y2="52.240446875" width="0.3048" layer="1"/>
-<wire x1="24.202934375" y1="52.240446875" x2="24.500765625" y2="52.240446875" width="0.3048" layer="1"/>
-</signal>
-<signal name="N$11">
-<contactref element="T1" pad="3"/>
-<contactref element="LED2" pad="C"/>
-<wire x1="26.27780625" y1="48.96340625" x2="26.25099375" y2="48.96340625" width="0.3048" layer="1"/>
-<wire x1="26.25099375" y1="48.96340625" x2="26.02259375" y2="49.19180625" width="0.3048" layer="1"/>
-<wire x1="26.02259375" y1="49.19180625" x2="22.97459375" y2="49.19180625" width="0.3048" layer="1"/>
-</signal>
 <signal name="N$5">
-<contactref element="ESD2" pad="4"/>
+<contactref element="IC2" pad="4"/>
 <contactref element="R2" pad="2"/>
 <contactref element="X1" pad="SW1"/>
@@
 <contactref element="USB" pad="5"/>
 <contactref element="C9" pad="1"/>
-<contactref element="ESD3" pad="1"/>
+<contactref element="IC4" pad="1"/>
 <contactref element="JP4" pad="1"/>
 <contactref element="IC7" pad="17"/>
@@
 <signal name="M_USB_D-">
 <contactref element="USB" pad="4"/>
-<contactref element="ESD3" pad="2"/>
+<contactref element="IC4" pad="2"/>
 <contactref element="IC6" pad="4"/>
 <wire x1="88.01540625" y1="44.93019375" x2="88.00340625" y2="44.91819375" width="0.2032" layer="1"/>
@@
 <signal name="M_USB_D+">
 <contactref element="USB" pad="3"/>
-<contactref element="ESD3" pad="3"/>
+<contactref element="IC4" pad="3"/>
 <contactref element="IC6" pad="3"/>
 <wire x1="88.00740625" y1="44.42219375" x2="88.00340625" y2="44.41819375" width="0.2032" layer="1"/>
@@
 <wire x1="14.986" y1="46.736" x2="14.986" y2="24.384" width="0.6096" layer="16"/>
 </signal>
+<signal name="N$8">
+<contactref element="T1" pad="3"/>
+<contactref element="LED3" pad="C"/>
+<wire x1="22.97459375" y1="49.19180625" x2="23.1747875" y2="49.392" width="0.3048" layer="1"/>
+<wire x1="23.1747875" y1="49.392" x2="27.432" y2="49.392" width="0.3048" layer="1"/>
+</signal>
+<signal name="N$9">
+<contactref element="LED3" pad="A"/>
+<contactref element="R15" pad="1"/>
+<wire x1="24.202934375" y1="52.240446875" x2="26.383553125" y2="52.240446875" width="0.3048" layer="1"/>
+<wire x1="26.383553125" y1="52.240446875" x2="27.432" y2="51.192" width="0.3048" layer="1"/>
+</signal>
 </signals>
