File: SARA_U201_BREAKOUT_BOARD/SARA_U201.sch (EAGLE design)
At the start: 54 parts, among them J6 -, T1 BC847, U1 LT1764AEQ#PBF, U2 SN74AVC4T774, U3 SN74AVC4T774, X1 CCM03-3013LFT_R102

Commit message: Updated Layout with changed footprint for level shifters and SARA-U201
Parts:
- removed U$1: SARA_U201, SARA_U201:SARA_U201
- added U4: SARA-U201-03B, SARA-U201-03B:SARA-U201-03B
- C4: value 10uF -> 100nF
- R13: value 9K1 -> 6K8
- U2, U3: value SN74AVC4T774 -> SN74AVC4T774PW; device Arduino-ICs:SN74AVC4T774 -> SN74AVC4T774PW:SN74AVC4T774PW
Connections:
- removed net GND1: U2.DIR2, U2.DIR3, U2.DIR4
- removed net N$10: U$1.1_GND, U$1.3_GND, U$1.5_GND
- net ANT: now also U4.ATN; no longer U$1.ANT_56
- net ANT_DET: now also U4.ANT_DET; no longer U$1.ANT_DET_62
- net CODEC_CLK: now also U4.CODEC_CLK; no longer U$1.19_CODEC_CLK
- net CTS1: now also U4.CTS; no longer U$1.11_CTS
- net DCD1: now also U4.DCD; no longer U$1.8_DCD
- net DSR1: now also U4.DSR; no longer U$1.6_DSR
- net DTR1: now also U4.DTR; no longer U$1.9_DTR
- net GND: now also U2.DIR2, U2.DIR3, U2.DIR4, U2.GND, U2.~OE, U3.DIR1, U3.~OE, U4.GND_1, U4.GND_10, U4.GND_11, U4.GND_12, U4.GND_13, U4.GND_14, U4.GND_15, U4.GND_16, U4.GND_17, U4.GND_18, U4.GND_19, U4.GND_2, U4.GND_20, U4.GND_21, U4.GND_22, U4.GND_23, U4.GND_24, U4.GND_25, U4.GND_26, U4.GND_27, U4.GND_28, U4.GND_29, U4.GND_3, U4.GND_30, U4.GND_31, U4.GND_32, U4.GND_33, U4.GND_34, U4.GND_35, U4.GND_36, U4.GND_37, U4.GND_38, U4.GND_39, U4.GND_40, U4.GND_41, U4.GND_42, U4.GND_43, U4.GND_44, U4.GND_45, U4.GND_46, U4.GND_47, U4.GND_48, U4.GND_49, U4.GND_5, U4.GND_50, U4.GND_51, U4.GND_52, U4.GND_6, U4.GND_7, U4.GND_9, U4.RSVD_2; no longer U$1.20_GND, U$1.21_GND, U$1.22_GND, U$1.32_GND, U$1.33_RSVD, U$1.43_GND, U$1.GND_50, U$1.GND_54, U$1.GND_55, U$1.GND_57, U$1.GND_58, U$1.GND_59, U$1.GND_60, U$1.GND_61, U$1.GND_63, U$1.GND_64, U$1.GND_65, U$1.GND_66, U$1.GND_67, U$1.GND_68, U$1.GND_69, U$1.GND_70, U$1.GND_71, U$1.GND_72, U$1.GND_73, U$1.GND_74, U$1.GND_75, U$1.GND_76, U$1.GND_77, U$1.GND_78, U$1.GND_79, U$1.GND_80, U$1.GND_81, U$1.GND_82, U$1.GND_83, U$1.GND_84, U$1.GND_85, U$1.GND_86, U$1.GND_87, U$1.GND_88, U$1.GND_89, U$1.GND_90, U$1.GND_91, U$1.GND_92, U$1.GND_93, U$1.GND_94, U$1.GND_95, U$1.GND_96, U3.DIR2, U3.OE
- net GND2: now also U4.GND_4; no longer U$1.14_GND, U2.GND, U2.OE
- net GPIO2: now also U4.GPIO2; no longer U$1.23_GPIO2
- net GPIO3: now also U4.GPIO3; no longer U$1.24_GPIO3
- net GPIO4: now also U4.GPIO4; no longer U$1.25_GPIO4
- net I2S_CLK: now also U4.I2S_CLK; no longer U$1.36_I2S_CLK
- net I2S_RXD: now also U4.I2S_RXD; no longer U$1.37_I2S_RXD
- net I2S_TXD: now also U4.I2S_TXD; no longer U$1.35_I2S_TXD
- net I2S_WA: now also U4.I2S_WA; no longer U$1.34_I2S_WA
- net NET_STAT: now also U4.GPIO1; no longer U$1.16_GPIO1
- net PWR_ON: now also U4.PWR_ON; no longer U$1.15_PWR_ON
- net RI1: now also U4.RI; no longer U$1.7_RI
- net RST: now also U4.RESET_N; no longer U$1.18_RESET_N
- net RTS1: now also TP2.TP, U4.RTS; no longer TP3.TP, U$1.10_RTS
- net RXD: now also U3.A1; no longer U3.A2
- net RXD1: now also TP3.TP, U4.RXD; no longer TP2.TP, U$1.13_RXD
- net SCL: now also U4.SCL; no longer U$1.27_SCL
- net SDA: now also U4.SDA; no longer U$1.26_SDA
- net SIM_CLK: now also U4.SIM_CLK; no longer U$1.38_SIM_CLK
- net SIM_DET: now also U4.SIM_DET; no longer U$1.42_SIM_DET
- net SIM_I/O: now also U4.SIM_IO; no longer U$1.39_SIM_IO
- net SIM_RST: now also U4.SIM_RST; no longer U$1.40_SIM_RST
- net TXD: now also U3.A2; no longer U3.A1
- net TXD1: now also U4.TXD; no longer U$1.12_TXD
- net USB_D+: now also U4.USB_D+; no longer U$1.29_USB_D+
- net USB_D-: now also U4.USB_D-; no longer U$1.28_USB_D-
- net USB_GND: now also U4.GND_8; no longer U$1.30_GND
- net VCC: now also U3.DIR2, U4.VCC_1, U4.VCC_2, U4.VCC_3; no longer U$1.VCC_51, U$1.VCC_52, U$1.VCC_53, U3.DIR1
- net VCCINT: now also U4.V_INT; no longer U$1.4_V_INT
- net VSIM: now also U4.VSIM; no longer U$1.41_VSIM
- net VUSB_DET: now also U4.VUSB_DET; no longer U$1.17_VUSB_DET
- net V_BCKP: now also U4.V_BCKP; no longer U$1.2_V_BCKP
Other:
- note added: "VCC = 3.3V VCCINT = 1.8V"
- note removed: "SARA_U201"
- note removed: "SN74AVC4T774PWR"
- note removed: "VCC=3.3V VCCINT=1.4V"
- moved on the sheet: C1, C10, C16, C2, C3, C4, R20, TP1, TP2, TP3, TP4, TP5

Commit message: Added the USB switch and power LED
Parts:
- added IC1: TS3USB221ERSER, TS3USB221ERSER:TS3USB221ERSER
- added LED1: SML-LX0805GC-TR, SML-LX0805GC-TR:SML-LX0805GC-TR
- added R1: 470, rcl:R-EU_R0805
Connections:
- new net MC_USB_D+: IC1.1D+, JP4.3
- new net MC_USB_D-: IC1.1D-, JP4.2
- new net M_USB_D+: ESD3.ESD3, IC1.2D+, USB.3
- new net M_USB_D-: ESD3.ESD2, IC1.2D-, USB.4
- new net N$1: LED1.C, R1.2
- new net SW_EN: IC1.!OE, JP2.1
- new net SW_SEL: IC1.S, JP2.2
- new net USB_D+1: JP2.3
- new net USB_GND1: JP2.4
- net +5V: now also LED1.A
- net GND: now also R1.1; no longer JP2.2
- net SCL: no longer JP2.3
- net SDA: no longer JP2.4
- net USB_D+: now also IC1.D+; no longer ESD3.ESD3, JP4.3, USB.3
- net USB_D-: now also IC1.D-; no longer ESD3.ESD2, JP4.2, USB.4
- net USB_GND: now also IC1.GND
- net VCC: now also IC1.VCC
- net VCCINT: no longer JP2.1
Other:
- note added: "INDICATION LED's"
- note added: "SARA - U201 GSM Module"
- note added: "USB SWITCH"
- note removed: "I2C"
- note removed: "NETWORK STATUS"
- moved on the sheet: C1, C18, C19, C2, C20, C21, C22, C6, C7, C8, C9, J2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

Commit message: Changed the pad for L2 and used minimum no. of vias to connect to the USB switch
Parts:
- L2: device rcl:L-EUL1812 -> 490-15685-1-ND:SRR1260-470MLQW18AN39NJ8ZD
Connections:
- net GND: now also L2.1; no longer L2.2
- net N$7: now also L2.2; no longer L2.1
Changed lines of the file:
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@@
 <part name="C5" library="rcl" library_urn="urn:adsk.eagle:library:334" deviceset="C-EU" device="C0805" package3d_urn="urn:adsk.eagle:package:23617/2" value="15pF"/>
 <part name="C12" library="rcl" library_urn="urn:adsk.eagle:library:334" deviceset="C-EU" device="C0805" package3d_urn="urn:adsk.eagle:package:23617/2" value="33pF"/>
-<part name="L2" library="rcl" library_urn="urn:adsk.eagle:library:334" deviceset="L-EU" device="L1812" package3d_urn="urn:adsk.eagle:package:23494/2" value="39nH"/>
 <part name="JP1" library="pinhead" library_urn="urn:adsk.eagle:library:325" deviceset="PINHD-1X13" device="" package3d_urn="urn:adsk.eagle:package:22421/2"/>
 <part name="JP3" library="pinhead" library_urn="urn:adsk.eagle:library:325" deviceset="PINHD-1X9" device="" package3d_urn="urn:adsk.eagle:package:22483/2"/>
@@
 <part name="R1" library="rcl" library_urn="urn:adsk.eagle:library:334" deviceset="R-EU_" device="R0805" package3d_urn="urn:adsk.eagle:package:23553/2" value="470"/>
 <part name="GND28" library="supply1" library_urn="urn:adsk.eagle:library:371" deviceset="GND" device=""/>
+<part name="L2" library="490-15685-1-ND" deviceset="SRR1260-470M" device="LQW18AN39NJ8ZD" value="39nH"/>
 </parts>
 <sheets>
@@
 <attribute name="NAME" x="330.2" y="325.12" size="1.778" layer="104"/>
 </instance>
-<instance part="GND20" gate="1" x="307.34" y="297.18" smashed="yes">
-<attribute name="VALUE" x="304.8" y="294.64" size="1.778" layer="96"/>
+<instance part="GND20" gate="1" x="307.34" y="289.56" smashed="yes">
+<attribute name="VALUE" x="304.8" y="287.02" size="1.778" layer="96"/>
 </instance>
 <instance part="GND21" gate="1" x="337.82" y="297.18" smashed="yes">
@@
 <attribute name="NAME" x="312.039" y="319.024" size="1.778" layer="95" rot="R90"/>
 <attribute name="VALUE" x="317.119" y="319.024" size="1.778" layer="96" rot="R90"/>
-</instance>
-<instance part="L2" gate="G$1" x="307.34" y="307.34" smashed="yes">
-<attribute name="NAME" x="305.8414" y="303.53" size="1.778" layer="95" rot="R90"/>
-<attribute name="VALUE" x="310.642" y="303.53" size="1.778" layer="96" rot="R90"/>
 </instance>
 <instance part="JP1" gate="A" x="322.58" y="233.68" smashed="yes">
@@
 <instance part="GND28" gate="1" x="228.6" y="203.962" smashed="yes">
 <attribute name="VALUE" x="226.06" y="201.422" size="1.778" layer="96"/>
+</instance>
+<instance part="L2" gate="G$1" x="307.34" y="302.26" smashed="yes">
+<attribute name="NAME" x="309.37585" y="308.113059375" size="1.781359375" layer="95"/>
+<attribute name="VALUE" x="309.12101875" y="294.627040625" size="1.78101875" layer="96"/>
 </instance>
 </instances>
@@
 </segment>
 <segment>
-<pinref part="L2" gate="G$1" pin="2"/>
 <pinref part="GND20" gate="1" pin="GND"/>
-<wire x1="307.34" y1="302.26" x2="307.34" y2="299.72" width="0.1524" layer="91"/>
+<wire x1="307.34" y1="294.64" x2="307.34" y2="292.1" width="0.1524" layer="91"/>
+<pinref part="L2" gate="G$1" pin="1"/>
 </segment>
 <segment>
@@
 <pinref part="C5" gate="G$1" pin="2"/>
 <pinref part="C12" gate="G$1" pin="1"/>
-<pinref part="L2" gate="G$1" pin="1"/>
 <wire x1="307.34" y1="317.5" x2="304.8" y2="317.5" width="0.1524" layer="91"/>
-<wire x1="307.34" y1="312.42" x2="307.34" y2="317.5" width="0.1524" layer="91"/>
+<wire x1="307.34" y1="309.88" x2="307.34" y2="317.5" width="0.1524" layer="91"/>
 <junction x="307.34" y="317.5"/>
-</segment>
-</net>
+<pinref part="L2" gate="G$1" pin="2"/>
+</segment>
+</net>

Commit message: Added Teensy, MIC, Boost connectors along with some layout changes with USB switch and rerouting all the connections
Parts:
- removed C1, C2: 100nF, rcl:C-EUC0805
- removed H1, H2, H3, H4: MOUNT-HOLE3.0, holes:MOUNT-HOLE3.0
- removed J6: -, Arduino-connectors:UFL
- removed JP1: (no value), pinhead:PINHD-1X13
- removed TP1, TP2, TP3, TP4: TPB1,27, testpad:TPB1,27
- removed U1: LT1764AEQ#PBF, LT1764AEQ_PBF:LT1764AEQ#PBF
- removed U3: SN74AVC4T774PW, SN74AVC4T774PW:SN74AVC4T774PW
- added C11, C13: (no value), rcl:C-USC0805
- added IC2: MCP1826T-3302E_DC, MCP1826T-3302E_DC:MCP1826T-3302E_DC
- added J1: SMA_CONNECTOR, SMA_CONNECTOR:SMA_CONNECTOR
- added J3, SOLAR_CHARGER: 61300211121, 61300211121:61300211121
- added J4, J5: 61300311121, 61300311121:61300311121
- added R3: 100K, rcl:R-EU_R0805
- added R4, R5, R6: 0R, adafruit:R-US_M0805
- added SWITCH: GSM Power, EG1218:EG1218
- added U$1: TEENSY3_6--ALLPINS, Teensy_3_6:TEENSY3_6--ALLPINS
- added WILDLY_5V_1A_BOOST: (no value), adafruit:PINHD-1X8BIG
- added WILDLY_I2S_MIC: (no value), adafruit:PINHD-1X6
- C7: value 10uF -> 2.2uF
- J2: value (none) -> B2B-PH-SM4-TB(LF)(SN); device SparkFun-Connectors:JST_2MM_MALE -> B2B-PH-SM4-TB_LF__SN_:B2B-PH-SM4-TB(LF)(SN)
- R13: value 6K8 -> 10K
- R14: value 3K9 -> 1K
- U2: value SN74AVC4T774PW -> TXB0106PWR; device SN74AVC4T774PW:SN74AVC4T774PW -> TXB0106PWR:TXB0106PWR
Connections:
- removed net DCD: JP1.8, U2.A4
- removed net DSR: JP1.6, U2.A2
- removed net DTR: JP1.5, U2.A1
- new net 5V_EN: SWITCH.1, WILDLY_5V_1A_BOOST.5
- new net 5V_SUPPLY: R4.2, WILDLY_5V_1A_BOOST.1
- new net FUEL_GAUGE_SCL: J4.2, U$1.19/A5/PWM/T/SCL0
- new net FUEL_GAUGE_SDA: J4.1, U$1.18/A4/PWM/T/SDA0
- new net LB: WILDLY_5V_1A_BOOST.3
- new net MIC_BCLK: U$1.9/PWM/RX2/CS0-1, WILDLY_I2S_MIC.3
- new net MIC_DOUT: U$1.13/LED/ALT-PWM/SCK0, WILDLY_I2S_MIC.4
- new net MIC_LRCLK: U$1.23/A9/PWM/T, WILDLY_I2S_MIC.5
- new net N$2: IC2.PWRGD, R13.2, R3.1
- new net N$4: WILDLY_5V_1A_BOOST.6
- new net STAT: U$1.24, U2.B1
- new net V+: C8.1, IC2.!SHDN, IC2.VIN, J2.1, J3.1, SOLAR_CHARGER.1, WILDLY_5V_1A_BOOST.7
- new net VDD: C4.2, C7.1, IC2.VOUT, R15.2, R3.2, U4.VCC_1, U4.VCC_2, U4.VCC_3
- net +5V: now also C11.1, C13.1, R4.1, U$1.VIN; no longer C8.1, J2.+, JP1.10, U1.*SHDN, U1.IN
- net CTS: now also U$1.33/A14/CAN1TX/TX5/ALT-SCL0, U2.B4; no longer JP1.4, U3.A4
- net CTS1: now also U2.A4; no longer TP4.TP, U3.B4
- net DCD1: no longer U2.B4
- net DSR1: no longer U2.B2
- net DTR1: no longer U2.B1
- net GND: now also C11.2, C13.2, IC2.GND, IC2.GND_(TAB), J1.GND, J2.2, J3.2, SOLAR_CHARGER.2, SWITCH.COM, U$1.GND, WILDLY_5V_1A_BOOST.2, WILDLY_5V_1A_BOOST.4, WILDLY_I2S_MIC.2; no longer C1.2, C2.2, J2.-, J6.GND, JP1.9, U1.GND, U1.GND_2, U2.DIR2, U2.DIR3, U2.DIR4, U2.~OE, U3.DIR1, U3.DIR4, U3.GND, U3.~OE
- net MC_USB_D+: now also U$1.D+
- net MC_USB_D-: now also U$1.D-
- net N$3: no longer U1.ADJ
- net N$6: now also J1.SIG; no longer J6.SIG
- net NET_STAT: now also U2.A1
- net PWR_ON: now also U$1.35/A16/PWM; no longer JP1.11
- net RI: now also U$1.17/A3/PWM/T/ALT-SDA0, U2.B6; no longer JP1.7, U2.A3
- net RI1: now also U2.A6; no longer U2.B3
- net RST: now also U$1.20/A6/PWM/CS0-2/ALT-SCK1; no longer JP1.12
- net RTS: now also U$1.34/A15/CAN1RX/RX5/ALT-SDA0, U2.B5; no longer JP1.3, U3.A3
- net RTS1: now also U2.A5; no longer TP2.TP, U3.B3
- net RXD: now also R6.1, R6.2, U$1.1/TX1/MISO1/T, U2.B3; no longer JP1.2, U3.A1
- net RXD1: now also U2.A2; no longer TP3.TP, U3.B2
- net TXD: now also R5.1, R5.2, U$1.0/RX1/MOSI1/T, U2.B2; no longer JP1.1, U3.A2
- net TXD1: now also U2.A3; no longer TP1.TP, U3.B1
- net VCC: now also U$1.3V3, U2.VCCB, WILDLY_I2S_MIC.1; no longer C2.1, C4.2, C7.1, JP1.13, R13.2, R15.2, U1.OUT, U2.DIR1, U2.VCCA, U3.DIR2, U3.DIR3, U3.VCCA, U4.VCC_1, U4.VCC_2, U4.VCC_3
- net VCCINT: now also U2.OE, U2.VCCA; no longer C1.1, U2.VCCB, U3.VCCB
- net VUSB_DET: now also U$1.VUSB
Other:
- note added: "5V"
- note added: "5V Boost 1A"
- note added: "5V Out EN - Transmitter On/Off"
- note added: "Adafruit I2S Microphone SPH0645LM4H"
- note added: "EN"
- note added: "Fuel Gauge"
- note added: "GND"
- note added: "LB"
- note added: "Solar Charger"
- note added: "VBAT"
- note added: "VDD = 4.14V VCCINT = 1.8V VCC = 3.3V"
- note added: "VS"
- note added: "VUSB"
- note removed: "VCC = 3.3V VCCINT = 1.8V"
- moved on the sheet: C10, C3, C7, C8, JP2, JP4, R13, R14, TP5, U2

Commit message: Removed the RST pin connection from Teensy as it requires a level shifter
Connections:
- net RST: no longer U$1.20/A6/PWM/CS0-2/ALT-SCK1
Changed lines of the file:
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@@
 <label x="406.4" y="332.74" size="1.778" layer="95"/>
-</segment>
-<segment>
-<pinref part="U$1" gate="G$1" pin="20/A6/PWM/CS0-2/ALT-SCK1"/>
-<wire x1="426.72" y1="134.62" x2="411.48" y2="134.62" width="0.1524" layer="91"/>
-<label x="411.48" y="134.62" size="1.778" layer="95"/>
 </segment>
 </net>

Commit message: All the review changes done except a few which need to be discussed
Parts:
- removed ESD1: SOT95P275X110-6N, SOT95P275X110-6N:SOT95P275X110-6N
- removed U$1: TEENSY3_6--ALLPINS, Teensy_3_6:TEENSY3_6--ALLPINS
- removed U2: TXB0106PWR, TXB0106PWR:TXB0106PWR
- removed U4: SARA-U201-03B, SARA-U201-03B:SARA-U201-03B
- added IC5: TXB0106PWR, TXB0106PWR:TXB0106PWR
- added IC6: TS3USB221ERSER, TS3USB221ERSER:TS3USB221ERSER
- added IC7: SARA-U201-03B, SARA-U201-03B:SARA-U201-03B
- added IC8: TEENSY3_6--ALLPINS, Teensy_3_6:TEENSY3_6--ALLPINS
- added TP1, TP2, TP3: TPB1,27, testpad:TPB1,27
- IC1: value TS3USB221ERSER -> SOT95P275X110-6N; device TS3USB221ERSER:TS3USB221ERSER -> SOT95P275X110-6N:SOT95P275X110-6N
- renumbered IC2 to IC3
Connections:
- net +5V: now also IC8.VIN; no longer U$1.VIN
- net ANT: now also IC7.ATN; no longer U4.ATN
- net ANT_DET: now also IC7.ANT_DET; no longer U4.ANT_DET
- net CODEC_CLK: now also IC7.CODEC_CLK; no longer U4.CODEC_CLK
- net CTS: now also IC5.B4, IC8.33/A14/CAN1TX/TX5/ALT-SCL0; no longer U$1.33/A14/CAN1TX/TX5/ALT-SCL0, U2.B4
- net CTS1: now also IC5.A4, IC7.CTS; no longer U2.A4, U4.CTS
- net DCD1: now also IC7.DCD; no longer U4.DCD
- net DSR1: now also IC7.DSR; no longer U4.DSR
- net DTR1: now also IC7.DTR; no longer U4.DTR
- net FUEL_GAUGE_SCL: now also IC8.19/A5/PWM/T/SCL0; no longer U$1.19/A5/PWM/T/SCL0
- net FUEL_GAUGE_SDA: now also IC8.18/A4/PWM/T/SDA0; no longer U$1.18/A4/PWM/T/SDA0
- net GND: now also IC1.GND_A, IC1.GND_B, IC5.GND, IC7.GND_1, IC7.GND_10, IC7.GND_11, IC7.GND_12, IC7.GND_13, IC7.GND_14, IC7.GND_15, IC7.GND_16, IC7.GND_17, IC7.GND_18, IC7.GND_19, IC7.GND_2, IC7.GND_20, IC7.GND_21, IC7.GND_22, IC7.GND_23, IC7.GND_24, IC7.GND_25, IC7.GND_26, IC7.GND_27, IC7.GND_28, IC7.GND_29, IC7.GND_3, IC7.GND_30, IC7.GND_31, IC7.GND_32, IC7.GND_33, IC7.GND_34, IC7.GND_35, IC7.GND_36, IC7.GND_37, IC7.GND_38, IC7.GND_39, IC7.GND_40, IC7.GND_41, IC7.GND_42, IC7.GND_43, IC7.GND_44, IC7.GND_45, IC7.GND_46, IC7.GND_47, IC7.GND_48, IC7.GND_49, IC7.GND_5, IC7.GND_50, IC7.GND_51, IC7.GND_52, IC7.GND_6, IC7.GND_7, IC7.GND_9, IC7.RSVD_2, IC8.GND; no longer ESD1.GND_A, ESD1.GND_B, U$1.GND, U2.GND, U4.GND_1, U4.GND_10, U4.GND_11, U4.GND_12, U4.GND_13, U4.GND_14, U4.GND_15, U4.GND_16, U4.GND_17, U4.GND_18, U4.GND_19, U4.GND_2, U4.GND_20, U4.GND_21, U4.GND_22, U4.GND_23, U4.GND_24, U4.GND_25, U4.GND_26, U4.GND_27, U4.GND_28, U4.GND_29, U4.GND_3, U4.GND_30, U4.GND_31, U4.GND_32, U4.GND_33, U4.GND_34, U4.GND_35, U4.GND_36, U4.GND_37, U4.GND_38, U4.GND_39, U4.GND_40, U4.GND_41, U4.GND_42, U4.GND_43, U4.GND_44, U4.GND_45, U4.GND_46, U4.GND_47, U4.GND_48, U4.GND_49, U4.GND_5, U4.GND_50, U4.GND_51, U4.GND_52, U4.GND_6, U4.GND_7, U4.GND_9, U4.RSVD_2
- net GND2: now also IC7.GND_4; no longer U4.GND_4
- net GPIO2: now also IC7.GPIO2; no longer U4.GPIO2
- net GPIO3: now also IC7.GPIO3; no longer U4.GPIO3
- net GPIO4: now also IC7.GPIO4; no longer U4.GPIO4
- net I2S_CLK: now also IC7.I2S_CLK; no longer U4.I2S_CLK
- net I2S_RXD: now also IC7.I2S_RXD; no longer U4.I2S_RXD
- net I2S_TXD: now also IC7.I2S_TXD; no longer U4.I2S_TXD
- net I2S_WA: now also IC7.I2S_WA; no longer U4.I2S_WA
- net MC_USB_D+: now also IC6.1D+, IC8.D+; no longer IC1.1D+, U$1.D+
- net MC_USB_D-: now also IC6.1D-, IC8.D-; no longer IC1.1D-, U$1.D-
- net MIC_BCLK: now also IC8.9/PWM/RX2/CS0-1; no longer U$1.9/PWM/RX2/CS0-1
- net MIC_DOUT: now also IC8.13/LED/ALT-PWM/SCK0; no longer U$1.13/LED/ALT-PWM/SCK0
- net MIC_LRCLK: now also IC8.23/A9/PWM/T; no longer U$1.23/A9/PWM/T
- net M_USB_D+: now also IC6.2D+; no longer IC1.2D+
- net M_USB_D-: now also IC6.2D-; no longer IC1.2D-
- net NET_STAT: now also IC5.A1, IC7.GPIO1; no longer U2.A1, U4.GPIO1
- net PWR_ON: now also IC1.ESD1, IC7.PWR_ON, IC8.35/A16/PWM; no longer ESD1.ESD1, U$1.35/A16/PWM, U4.PWR_ON
- net RI: now also IC5.B6, IC8.17/A3/PWM/T/ALT-SDA0; no longer U$1.17/A3/PWM/T/ALT-SDA0, U2.B6
- net RI1: now also IC5.A6, IC7.RI; no longer U2.A6, U4.RI
- net RST: now also IC1.ESD4, IC7.RESET_N; no longer ESD1.ESD4, U4.RESET_N
- net RTS: now also IC5.B5, IC8.34/A15/CAN1RX/RX5/ALT-SDA0; no longer U$1.34/A15/CAN1RX/RX5/ALT-SDA0, U2.B5
- net RTS1: now also IC5.A5, IC7.RTS; no longer U2.A5, U4.RTS
- net RXD: now also IC5.B2, IC8.1/TX1/MISO1/T; no longer U$1.1/TX1/MISO1/T, U2.B3
- net RXD1: now also IC5.A2, IC7.RXD; no longer U2.A2, U4.RXD
- net SCL: now also IC7.SCL; no longer U4.SCL
- net SDA: now also IC7.SDA; no longer U4.SDA
- net SIM_CLK: now also IC7.SIM_CLK; no longer U4.SIM_CLK
- net SIM_DET: now also IC1.ESD3, IC7.SIM_DET; no longer ESD1.ESD3, U4.SIM_DET
- net SIM_I/O: now also IC1.ESD2, IC7.SIM_IO; no longer ESD1.ESD2, U4.SIM_IO
- net SIM_RST: now also IC7.SIM_RST; no longer U4.SIM_RST
- net STAT: now also IC5.B1, IC8.24; no longer U$1.24, U2.B1
- net SW_EN: now also IC6.!OE; no longer IC1.!OE
- net SW_SEL: now also IC6.S; no longer IC1.S
- net TXD: now also IC5.B3, IC8.0/RX1/MOSI1/T; no longer U$1.0/RX1/MOSI1/T, U2.B2
- net TXD1: now also IC5.A3, IC7.TXD; no longer U2.A3, U4.TXD
- net USB_D+: now also IC6.D+, IC7.USB_D+; no longer IC1.D+, U4.USB_D+
- net USB_D-: now also IC6.D-, IC7.USB_D-; no longer IC1.D-, U4.USB_D-
- net USB_GND: now also IC6.GND, IC7.GND_8; no longer IC1.GND, U4.GND_8
- net VCC: now also IC5.VCCB, IC6.VCC, IC8.3V3, TP2.TP, TP3.TP; no longer IC1.VCC, U$1.3V3, U2.VCCB
- net VCCINT: now also IC5.OE, IC5.VCCA, IC7.V_INT; no longer U2.OE, U2.VCCA, U4.V_INT
- net VDD: now also IC7.VCC_1, IC7.VCC_2, IC7.VCC_3, TP1.TP; no longer U4.VCC_1, U4.VCC_2, U4.VCC_3
- net VSIM: now also IC7.VSIM; no longer U4.VSIM
- net VUSB_DET: now also IC7.VUSB_DET, IC8.VUSB; no longer U$1.VUSB, U4.VUSB_DET
- net V_BCKP: now also IC7.V_BCKP; no longer U4.V_BCKP
Other:
- note added: "I2S Microphone"
- note added: "IC1"
- note added: "IC2"
- note added: "IC4"
- note added: "IC8 Teensy uC"
- note added: "On/Off Switch"
- note added: "Power-Boost"
- note added: "TEENSY 3.6 - uC Module"
- note added: "UART LEVEL SHIFTER"
- note removed: "ESD1"
- note removed: "ESD2"
- note removed: "ESD3"
- note removed: "UART"
- moved on the sheet: C10, C11, C13, C16, C3, C4, J3, J4, J5, R18, R19, R20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
