File: SARA_U201_BREAKOUT_BOARD/SARA_U201.sch (EAGLE design)
At the start: 62 parts, among them IC1 SOT95P275X110-6N, IC3 MCP1826T-3302E_DC, IC5 TXB0106PWR, IC6 TS3USB221ERSER, IC7 SARA-U201-03B, IC8 TEENSY3_6--ALLPINS, J1 SMA_CONNECTOR, J2 B2B-PH-SM4-TB(LF)(SN), J3 61300211121, J4 61300311121, J5 61300311121, T1 BC847, X1 CCM03-3013LFT_R102

Commit message: Updated the BOM as well with the schematics and layout
Parts:
- removed LED2: (no value), led:LEDCHIPLED_0603
- added LED3: SML-LX0805GC-TR, SML-LX0805GC-TR:SML-LX0805GC-TR
- renumbered ESD2 to IC2, ESD3 to IC4
Connections:
- removed net N$11: LED2.C, T1.C
- new net N$8: LED3.C, T1.C
- net N$9: now also LED3.A; no longer LED2.A
Other:
- note removed: "LTST-C190KRKT"
- moved on the sheet: R15
Changed lines of the file:
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@@
 <part name="T1" library="transistor" library_urn="urn:adsk.eagle:library:402" deviceset="BC847" device="" package3d_urn="urn:adsk.eagle:package:29904/2"/>
 <part name="GND44" library="supply1" library_urn="urn:adsk.eagle:library:371" deviceset="GND" device=""/>
-<part name="LED2" library="led" library_urn="urn:adsk.eagle:library:259" deviceset="LED" device="CHIPLED_0603" package3d_urn="urn:adsk.eagle:package:15822/2"/>
 <part name="R11" library="rcl" library_urn="urn:adsk.eagle:library:334" deviceset="R-EU_" device="R0805" package3d_urn="urn:adsk.eagle:package:23553/2" value="470K"/>
 <part name="R13" library="rcl" library_urn="urn:adsk.eagle:library:334" deviceset="R-EU_" device="R0805" package3d_urn="urn:adsk.eagle:package:23553/2" value="10K"/>
@@
 <part name="JP3" library="pinhead" library_urn="urn:adsk.eagle:library:325" deviceset="PINHD-1X9" device="" package3d_urn="urn:adsk.eagle:package:22483/2"/>
 <part name="LOGO1" library="logo" library_urn="urn:adsk.eagle:library:264" deviceset="ESD_10.00" device=""/>
-<part name="ESD2" library="SOT95P275X110-6N" deviceset="SOT95P275X110-6N" device=""/>
-<part name="ESD3" library="SOT95P275X110-6N" deviceset="SOT95P275X110-6N" device=""/>
+<part name="IC2" library="SOT95P275X110-6N" deviceset="SOT95P275X110-6N" device=""/>
+<part name="IC4" library="SOT95P275X110-6N" deviceset="SOT95P275X110-6N" device=""/>
 <part name="IC1" library="SOT95P275X110-6N" deviceset="SOT95P275X110-6N" device=""/>
 <part name="JP4" library="pinhead" library_urn="urn:adsk.eagle:library:325" deviceset="PINHD-1X4" device="" package3d_urn="urn:adsk.eagle:package:22407/2"/>
@@
 <part name="TP2" library="testpad" library_urn="urn:adsk.eagle:library:385" deviceset="TP" device="B1,27" package3d_urn="urn:adsk.eagle:package:27944/1"/>
 <part name="TP3" library="testpad" library_urn="urn:adsk.eagle:library:385" deviceset="TP" device="B1,27" package3d_urn="urn:adsk.eagle:package:27944/1"/>
+<part name="LED3" library="SML-LX0805GC-TR" deviceset="SML-LX0805GC-TR" device=""/>
 </parts>
 <sheets>
@@
 <wire x1="127" y1="274.32" x2="5.08" y2="274.32" width="0.4064" layer="94" style="shortdash"/>
 <wire x1="5.08" y1="190.5" x2="78.74" y2="190.5" width="0.4064" layer="94" style="shortdash"/>
-<text x="195.58" y="228.6" size="1.778" layer="95" rot="R90">LTST-C190KRKT</text>
 <text x="172.72" y="264.16" size="5.08" layer="94">INDICATION LED's</text>
 <wire x1="78.74" y1="190.5" x2="127" y2="190.5" width="0.4064" layer="94" style="shortdash"/>
@@
 </instance>
 <instance part="T1" gate="G$1" x="182.88" y="223.52" smashed="yes">
-<attribute name="NAME" x="172.72" y="231.14" size="1.778" layer="95"/>
-<attribute name="VALUE" x="172.72" y="228.6" size="1.778" layer="96"/>
+<attribute name="NAME" x="174.498" y="228.854" size="1.778" layer="95"/>
+<attribute name="VALUE" x="174.752" y="226.06" size="1.778" layer="96"/>
 </instance>
 <instance part="GND44" gate="1" x="172.72" y="203.2" smashed="yes">
 <attribute name="VALUE" x="170.18" y="200.66" size="1.778" layer="96"/>
-</instance>
-<instance part="LED2" gate="G$1" x="185.42" y="236.22" smashed="yes">
-<attribute name="NAME" x="188.976" y="231.648" size="1.778" layer="95" rot="R90"/>
-<attribute name="VALUE" x="191.135" y="231.648" size="1.778" layer="96" rot="R90"/>
 </instance>
 <instance part="R11" gate="G$1" x="30.48" y="373.38" smashed="yes" rot="R90">
@@
 <attribute name="VALUE" x="216.408" y="372.11" size="1.778" layer="96" rot="R90"/>
 </instance>
-<instance part="R15" gate="G$1" x="185.42" y="246.38" smashed="yes" rot="R90">
-<attribute name="NAME" x="183.9214" y="242.57" size="1.778" layer="95" rot="R90"/>
-<attribute name="VALUE" x="188.722" y="242.57" size="1.778" layer="96" rot="R90"/>
+<instance part="R15" gate="G$1" x="185.42" y="251.46" smashed="yes" rot="R90">
+<attribute name="NAME" x="183.9214" y="249.428" size="1.778" layer="95" rot="R90"/>
+<attribute name="VALUE" x="188.468" y="248.412" size="1.778" layer="96" rot="R90"/>
 </instance>
 <instance part="R16" gate="G$1" x="172.72" y="213.36" smashed="yes" rot="R90">
@@
 </instance>
 <instance part="LOGO1" gate="G$1" x="454.66" y="25.4" smashed="yes"/>
-<instance part="ESD2" gate="G$1" x="73.66" y="370.84" smashed="yes"/>
-<instance part="ESD3" gate="G$1" x="294.64" y="383.54" smashed="yes"/>
+<instance part="IC2" gate="G$1" x="73.66" y="370.84" smashed="yes"/>
+<instance part="IC4" gate="G$1" x="294.64" y="383.54" smashed="yes"/>
 <instance part="IC1" gate="G$1" x="40.64" y="365.76" smashed="yes"/>
 <instance part="JP4" gate="A" x="327.66" y="238.76" smashed="yes">
@@
 <attribute name="VALUE" x="497.84" y="396.24" size="1.778" layer="96" rot="R90"/>
 </instance>
-<instance part="VDD3" gate="G$1" x="185.42" y="256.54" smashed="yes">
-<attribute name="VALUE" x="182.88" y="254" size="1.778" layer="96" rot="R90"/>
+<instance part="VDD3" gate="G$1" x="185.42" y="261.62" smashed="yes">
+<attribute name="VALUE" x="182.88" y="259.08" size="1.778" layer="96" rot="R90"/>
 </instance>
 <instance part="P+1" gate="VCC" x="139.7" y="170.18" smashed="yes">
@@
 <attribute name="NAME" x="97.79" y="229.87" size="1.778" layer="95"/>
 <attribute name="TP_SIGNAL_NAME" x="100.33" y="227.33" size="1.778" layer="97"/>
+</instance>
+<instance part="LED3" gate="G$1" x="185.42" y="236.22" smashed="yes" rot="R90">
+<attribute name="NAME" x="181.60373125" y="235.45486875" size="1.780740625" layer="95" rot="R90"/>
+<attribute name="VALUE" x="191.77315" y="229.10631875" size="1.77946875" layer="96" rot="R90"/>
 </instance>
 </instances>
@@
 </segment>
 <segment>
-<pinref part="ESD2" gate="G$1" pin="GND_A"/>
+<pinref part="IC2" gate="G$1" pin="GND_A"/>
 <pinref part="GND12" gate="1" pin="GND"/>
 <wire x1="73.66" y1="350.52" x2="73.66" y2="347.98" width="0.1524" layer="91"/>
@@
 </segment>
 <segment>
-<pinref part="ESD2" gate="G$1" pin="GND_B"/>
+<pinref part="IC2" gate="G$1" pin="GND_B"/>
 <pinref part="GND13" gate="1" pin="GND"/>
 <wire x1="76.2" y1="350.52" x2="76.2" y2="347.98" width="0.1524" layer="91"/>
@@
 <wire x1="111.76" y1="396.24" x2="111.76" y2="383.54" width="0.1524" layer="91"/>
 <junction x="111.76" y="383.54"/>
-<pinref part="ESD2" gate="G$1" pin="ESD3"/>
+<pinref part="IC2" gate="G$1" pin="ESD3"/>
 <wire x1="76.2" y1="378.46" x2="76.2" y2="383.54" width="0.1524" layer="91"/>
 <junction x="76.2" y="383.54"/>
@@
 <wire x1="104.14" y1="396.24" x2="104.14" y2="386.08" width="0.1524" layer="91"/>
 <junction x="104.14" y="386.08"/>
-<pinref part="ESD2" gate="G$1" pin="ESD2"/>
+<pinref part="IC2" gate="G$1" pin="ESD2"/>
 <wire x1="73.66" y1="378.46" x2="73.66" y2="386.08" width="0.1524" layer="91"/>
 <junction x="73.66" y="386.08"/>
@@
 <wire x1="88.9" y1="396.24" x2="88.9" y2="388.62" width="0.1524" layer="91"/>
 <junction x="88.9" y="388.62"/>
-<pinref part="ESD2" gate="G$1" pin="ESD1"/>
+<pinref part="IC2" gate="G$1" pin="ESD1"/>
 <wire x1="71.12" y1="378.46" x2="71.12" y2="388.62" width="0.1524" layer="91"/>
 <junction x="71.12" y="388.62"/>
@@
 <wire x1="307.34" y1="365.76" x2="307.34" y2="360.68" width="0.1524" layer="91"/>
 <junction x="307.34" y="360.68"/>
-<pinref part="ESD3" gate="G$1" pin="GND_A"/>
+<pinref part="IC4" gate="G$1" pin="GND_A"/>
 <wire x1="294.64" y1="363.22" x2="294.64" y2="360.68" width="0.1524" layer="91"/>
-<pinref part="ESD3" gate="G$1" pin="GND_B"/>
+<pinref part="IC4" gate="G$1" pin="GND_B"/>
 <wire x1="297.18" y1="363.22" x2="297.18" y2="360.68" width="0.1524" layer="91"/>
 <junction x="297.18" y="360.68"/>
@@
 </segment>
 </net>
-<net name="N$9" class="0">
-<segment>
-<pinref part="LED2" gate="G$1" pin="A"/>
-<pinref part="R15" gate="G$1" pin="1"/>
-<wire x1="185.42" y1="241.3" x2="185.42" y2="238.76" width="0.1524" layer="91"/>
-</segment>
-</net>
-<net name="N$11" class="0">
-<segment>
-<pinref part="T1" gate="G$1" pin="C"/>
-<wire x1="185.42" y1="228.6" x2="185.42" y2="231.14" width="0.1524" layer="91"/>
-<pinref part="LED2" gate="G$1" pin="C"/>
-</segment>
-</net>
 <net name="N$5" class="0">
 <segment>
-<pinref part="ESD2" gate="G$1" pin="ESD4"/>
+<pinref part="IC2" gate="G$1" pin="ESD4"/>
 <wire x1="78.74" y1="378.46" x2="78.74" y2="381" width="0.1524" layer="91"/>
 <pinref part="R2" gate="G$1" pin="2"/>
@@
 <pinref part="SUPPLY1" gate="+5V" pin="+5V"/>
 <pinref part="C9" gate="G$1" pin="1"/>
-<pinref part="ESD3" gate="G$1" pin="ESD1"/>
+<pinref part="IC4" gate="G$1" pin="ESD1"/>
 <wire x1="292.1" y1="391.16" x2="292.1" y2="401.32" width="0.1524" layer="91"/>
 <junction x="292.1" y="401.32"/>
@@
 <wire x1="279.4" y1="398.78" x2="294.64" y2="398.78" width="0.1524" layer="91"/>
 <label x="314.96" y="398.78" size="1.778" layer="95"/>
-<pinref part="ESD3" gate="G$1" pin="ESD2"/>
+<pinref part="IC4" gate="G$1" pin="ESD2"/>
 <wire x1="294.64" y1="398.78" x2="320.04" y2="398.78" width="0.1524" layer="91"/>
 <wire x1="294.64" y1="391.16" x2="294.64" y2="398.78" width="0.1524" layer="91"/>
@@
 <wire x1="279.4" y1="396.24" x2="297.18" y2="396.24" width="0.1524" layer="91"/>
 <label x="314.96" y="396.24" size="1.778" layer="95"/>
-<pinref part="ESD3" gate="G$1" pin="ESD3"/>
+<pinref part="IC4" gate="G$1" pin="ESD3"/>
 <wire x1="297.18" y1="396.24" x2="320.04" y2="396.24" width="0.1524" layer="91"/>
 <wire x1="297.18" y1="391.16" x2="297.18" y2="396.24" width="0.1524" layer="91"/>
@@
 <segment>
 <pinref part="R15" gate="G$1" pin="2"/>
-<wire x1="185.42" y1="251.46" x2="185.42" y2="254" width="0.1524" layer="91"/>
+<wire x1="185.42" y1="256.54" x2="185.42" y2="259.08" width="0.1524" layer="91"/>
 <pinref part="VDD3" gate="G$1" pin="VDD"/>
 </segment>
@@
 </segment>
 </net>
+<net name="N$8" class="0">
+<segment>
+<pinref part="T1" gate="G$1" pin="C"/>
+<pinref part="LED3" gate="G$1" pin="C"/>
+</segment>
+</net>
+<net name="N$9" class="0">
+<segment>
+<pinref part="LED3" gate="G$1" pin="A"/>
+<pinref part="R15" gate="G$1" pin="1"/>
+</segment>
+</net>
