File: MCP73871-Solar Charger/Adafruit MCP73871 Solar Charger v4.sch (EAGLE design)
At the start: 35 parts, among them CN1 DCIN, IC1 MCP73871

Commit message: Fix Silkscreen issues with Solar board
Parts:
- renumbered IC1 to U1
Other:
- moved on the sheet: R10, R8, R9
Changed lines of the file:
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@@
 <?xml version="1.0" encoding="utf-8"?>
 <!DOCTYPE eagle SYSTEM "eagle.dtd">
-<eagle version="9.3.0">
+<eagle version="9.3.2">
 <drawing>
 <settings>
@@
 </classes>
 <parts>
-<part name="IC1" library="adafruit" deviceset="MCP73871" device=""/>
+<part name="U1" library="adafruit" deviceset="MCP73871" device=""/>
 <part name="GND1" library="supply1" deviceset="GND" device=""/>
 <part name="P+1" library="supply1" deviceset="VCC" device=""/>
@@
 </plain>
 <instances>
-<instance part="IC1" gate="G$1" x="160.02" y="96.52" smashed="yes"/>
+<instance part="U1" gate="G$1" x="160.02" y="96.52" smashed="yes"/>
 <instance part="GND1" gate="1" x="162.56" y="68.58" smashed="yes">
 <attribute name="VALUE" x="160.02" y="66.04" size="1.778" layer="96"/>
@@
 <attribute name="VALUE" x="93.98" y="111.506" size="1.27" layer="96"/>
 </instance>
-<instance part="R8" gate="G$1" x="99.06" y="127" smashed="yes" rot="R90">
-<attribute name="NAME" x="97.5614" y="123.19" size="1.778" layer="95" rot="R90"/>
-<attribute name="VALUE" x="102.362" y="123.19" size="1.778" layer="96" rot="R90"/>
-</instance>
-<instance part="R9" gate="G$1" x="109.22" y="127" smashed="yes" rot="R90">
-<attribute name="NAME" x="107.7214" y="123.19" size="1.778" layer="95" rot="R90"/>
-<attribute name="VALUE" x="112.522" y="123.19" size="1.778" layer="96" rot="R90"/>
-</instance>
-<instance part="R10" gate="G$1" x="119.38" y="127" smashed="yes" rot="R90">
-<attribute name="NAME" x="117.8814" y="123.19" size="1.778" layer="95" rot="R90"/>
-<attribute name="VALUE" x="122.682" y="123.19" size="1.778" layer="96" rot="R90"/>
-</instance>
-<instance part="P+4" gate="VCC" x="99.06" y="137.16" smashed="yes">
-<attribute name="VALUE" x="96.52" y="134.62" size="1.778" layer="96" rot="R90"/>
+<instance part="R8" gate="G$1" x="93.98" y="127" smashed="yes" rot="R90">
+<attribute name="NAME" x="92.4814" y="123.19" size="1.778" layer="95" rot="R90"/>
+<attribute name="VALUE" x="97.282" y="123.19" size="1.778" layer="96" rot="R90"/>
+</instance>
+<instance part="R9" gate="G$1" x="104.14" y="127" smashed="yes" rot="R90">
+<attribute name="NAME" x="102.6414" y="123.19" size="1.778" layer="95" rot="R90"/>
+<attribute name="VALUE" x="107.442" y="123.19" size="1.778" layer="96" rot="R90"/>
+</instance>
+<instance part="R10" gate="G$1" x="114.3" y="127" smashed="yes" rot="R90">
+<attribute name="NAME" x="112.8014" y="123.19" size="1.778" layer="95" rot="R90"/>
+<attribute name="VALUE" x="117.602" y="123.19" size="1.778" layer="96" rot="R90"/>
+</instance>
+<instance part="P+4" gate="VCC" x="93.98" y="137.16" smashed="yes">
+<attribute name="VALUE" x="91.44" y="134.62" size="1.778" layer="96" rot="R90"/>
 </instance>
 <instance part="C1" gate="G$1" x="213.36" y="111.76" smashed="yes">
@@
 <instance part="D1" gate="G$1" x="53.34" y="124.46" smashed="yes">
 <attribute name="NAME" x="50.8" y="127" size="1.27" layer="95"/>
-<attribute name="VALUE" x="50.8" y="120.65" size="1.27" layer="96"/>
+<attribute name="VALUE" x="48.26" y="120.65" size="1.27" layer="96"/>
 </instance>
 <instance part="GND9" gate="1" x="48.26" y="109.22" smashed="yes">
@@
 <wire x1="165.1" y1="71.12" x2="162.56" y2="71.12" width="0.1524" layer="91"/>
 <junction x="162.56" y="71.12"/>
-<pinref part="IC1" gate="G$1" pin="GND1"/>
+<pinref part="U1" gate="G$1" pin="GND1"/>
 <pinref part="GND1" gate="1" pin="GND"/>
-<pinref part="IC1" gate="G$1" pin="GND2"/>
-<pinref part="IC1" gate="G$1" pin="GND3"/>
+<pinref part="U1" gate="G$1" pin="GND2"/>
+<pinref part="U1" gate="G$1" pin="GND3"/>
 </segment>
 <segment>
@@
 <wire x1="160.02" y1="121.92" x2="160.02" y2="119.38" width="0.1524" layer="91"/>
 <junction x="160.02" y="119.38"/>
-<pinref part="IC1" gate="G$1" pin="IN2"/>
-<pinref part="IC1" gate="G$1" pin="IN1"/>
+<pinref part="U1" gate="G$1" pin="IN2"/>
+<pinref part="U1" gate="G$1" pin="IN1"/>
 <pinref part="P+1" gate="VCC" pin="VCC"/>
 </segment>
@@
 <junction x="127" y="96.52"/>
 <pinref part="P+3" gate="VCC" pin="VCC"/>
-<pinref part="IC1" gate="G$1" pin="CE"/>
-<pinref part="IC1" gate="G$1" pin="SEL"/>
-<pinref part="IC1" gate="G$1" pin="PROG2"/>
-<pinref part="IC1" gate="G$1" pin="/TE"/>
+<pinref part="U1" gate="G$1" pin="CE"/>
+<pinref part="U1" gate="G$1" pin="SEL"/>
+<pinref part="U1" gate="G$1" pin="PROG2"/>
+<pinref part="U1" gate="G$1" pin="/TE"/>
 </segment>
 <segment>
@@
 </segment>
 <segment>
-<wire x1="109.22" y1="132.08" x2="119.38" y2="132.08" width="0.1524" layer="91"/>
-<wire x1="109.22" y1="132.08" x2="99.06" y2="132.08" width="0.1524" layer="91"/>
-<wire x1="99.06" y1="134.62" x2="99.06" y2="132.08" width="0.1524" layer="91"/>
-<junction x="109.22" y="132.08"/>
-<junction x="99.06" y="132.08"/>
+<wire x1="104.14" y1="132.08" x2="114.3" y2="132.08" width="0.1524" layer="91"/>
+<wire x1="104.14" y1="132.08" x2="93.98" y2="132.08" width="0.1524" layer="91"/>
+<wire x1="93.98" y1="134.62" x2="93.98" y2="132.08" width="0.1524" layer="91"/>
+<junction x="104.14" y="132.08"/>
+<junction x="93.98" y="132.08"/>
 <pinref part="R10" gate="G$1" pin="2"/>
 <pinref part="R9" gate="G$1" pin="2"/>
@@
 <pinref part="R2" gate="G$1" pin="1"/>
 <pinref part="R3" gate="G$1" pin="1"/>
-<pinref part="IC1" gate="G$1" pin="VPCC"/>
+<pinref part="U1" gate="G$1" pin="VPCC"/>
 </segment>
 </net>
 <net name="N$1" class="0">
 <segment>
-<wire x1="139.7" y1="106.68" x2="119.38" y2="106.68" width="0.1524" layer="91"/>
-<wire x1="119.38" y1="106.68" x2="121.92" y2="114.3" width="0.1524" layer="91"/>
+<wire x1="139.7" y1="106.68" x2="121.92" y2="106.68" width="0.1524" layer="91"/>
 <pinref part="PWR" gate="G$1" pin="C"/>
-<pinref part="IC1" gate="G$1" pin="/PG"/>
+<pinref part="U1" gate="G$1" pin="/PG"/>
+<wire x1="121.92" y1="114.3" x2="121.92" y2="106.68" width="0.1524" layer="91"/>
 </segment>
 </net>
 <net name="N$4" class="0">
 <segment>
-<wire x1="139.7" y1="104.14" x2="109.22" y2="104.14" width="0.1524" layer="91"/>
-<wire x1="109.22" y1="104.14" x2="111.76" y2="114.3" width="0.1524" layer="91"/>
+<wire x1="139.7" y1="104.14" x2="111.76" y2="104.14" width="0.1524" layer="91"/>
+<wire x1="111.76" y1="104.14" x2="109.22" y2="104.14" width="0.1524" layer="91"/>
 <wire x1="109.22" y1="104.14" x2="109.22" y2="93.98" width="0.1524" layer="91"/>
 <wire x1="91.44" y1="93.98" x2="109.22" y2="93.98" width="0.1524" layer="91"/>
-<junction x="109.22" y="104.14"/>
-<pinref part="IC1" gate="G$1" pin="STAT2"/>
+<pinref part="U1" gate="G$1" pin="STAT2"/>
 <pinref part="DONE" gate="G$1" pin="C"/>
 <pinref part="JP5" gate="A" pin="3"/>
+<wire x1="111.76" y1="114.3" x2="111.76" y2="104.14" width="0.1524" layer="91"/>
+<junction x="111.76" y="104.14"/>
 </segment>
 </net>
 <net name="N$11" class="0">
 <segment>
-<wire x1="139.7" y1="101.6" x2="99.06" y2="101.6" width="0.1524" layer="91"/>
-<wire x1="99.06" y1="101.6" x2="101.6" y2="114.3" width="0.1524" layer="91"/>
+<wire x1="139.7" y1="101.6" x2="101.6" y2="101.6" width="0.1524" layer="91"/>
+<wire x1="101.6" y1="101.6" x2="99.06" y2="101.6" width="0.1524" layer="91"/>
 <wire x1="99.06" y1="101.6" x2="99.06" y2="88.9" width="0.1524" layer="91"/>
-<junction x="99.06" y="101.6"/>
-<pinref part="IC1" gate="G$1" pin="STAT1/LBO"/>
+<pinref part="U1" gate="G$1" pin="STAT1/LBO"/>
 <pinref part="CHRG/LBO" gate="G$1" pin="C"/>
 <pinref part="JP5" gate="A" pin="1"/>
 <wire x1="91.44" y1="88.9" x2="99.06" y2="88.9" width="0.1524" layer="91"/>
+<wire x1="101.6" y1="114.3" x2="101.6" y2="101.6" width="0.1524" layer="91"/>
+<junction x="101.6" y="101.6"/>
 </segment>
 </net>
 <net name="N$12" class="0">
 <segment>
-<wire x1="99.06" y1="121.92" x2="93.98" y2="114.3" width="0.1524" layer="91"/>
+<wire x1="93.98" y1="121.92" x2="93.98" y2="114.3" width="0.1524" layer="91"/>
 <pinref part="CHRG/LBO" gate="G$1" pin="A"/>
 <pinref part="R8" gate="G$1" pin="1"/>
@@
 <net name="N$13" class="0">
 <segment>
-<wire x1="104.14" y1="114.3" x2="109.22" y2="121.92" width="0.1524" layer="91"/>
+<wire x1="104.14" y1="114.3" x2="104.14" y2="121.92" width="0.1524" layer="91"/>
 <pinref part="DONE" gate="G$1" pin="A"/>
 <pinref part="R9" gate="G$1" pin="1"/>
@@
 <net name="N$14" class="0">
 <segment>
-<wire x1="114.3" y1="114.3" x2="119.38" y2="121.92" width="0.1524" layer="91"/>
+<wire x1="114.3" y1="114.3" x2="114.3" y2="121.92" width="0.1524" layer="91"/>
 <pinref part="PWR" gate="G$1" pin="A"/>
 <pinref part="R10" gate="G$1" pin="1"/>
@@
 <net name="N$15" class="0">
 <segment>
-<pinref part="IC1" gate="G$1" pin="PROG3"/>
+<pinref part="U1" gate="G$1" pin="PROG3"/>
 <pinref part="R12" gate="G$1" pin="2"/>
 </segment>
@@
 <segment>
 <wire x1="139.7" y1="83.82" x2="132.08" y2="83.82" width="0.1524" layer="91"/>
-<pinref part="IC1" gate="G$1" pin="PROG1"/>
+<pinref part="U1" gate="G$1" pin="PROG1"/>
 <pinref part="R11" gate="G$1" pin="2"/>
 </segment>
@@
 <junction x="182.88" y="109.22"/>
 <junction x="213.36" y="116.84"/>
-<pinref part="IC1" gate="G$1" pin="OUT2"/>
-<pinref part="IC1" gate="G$1" pin="OUT1"/>
+<pinref part="U1" gate="G$1" pin="OUT2"/>
+<pinref part="U1" gate="G$1" pin="OUT1"/>
 <pinref part="LOAD" gate="G$1" pin="2"/>
 <pinref part="C1" gate="G$1" pin="1"/>
@@
 <segment>
 <wire x1="182.88" y1="86.36" x2="185.42" y2="86.36" width="0.1524" layer="91"/>
-<pinref part="IC1" gate="G$1" pin="THERM"/>
+<pinref part="U1" gate="G$1" pin="THERM"/>
 <pinref part="R5" gate="G$1" pin="1"/>
 </segment>
@@
 <pinref part="BATT" gate="G$1" pin="2"/>
 <pinref part="C2" gate="G$1" pin="1"/>
-<pinref part="IC1" gate="G$1" pin="VBAT1"/>
-<pinref part="IC1" gate="G$1" pin="VBAT2"/>
-<pinref part="IC1" gate="G$1" pin="VBAT3"/>
+<pinref part="U1" gate="G$1" pin="VBAT1"/>
+<pinref part="U1" gate="G$1" pin="VBAT2"/>
+<pinref part="U1" gate="G$1" pin="VBAT3"/>
 <pinref part="JP4" gate="G$1" pin="1"/>
 </segment>
