File: Teensy_Recorder/wildly_teensy_proto.brd (EAGLE design)
At the start: 60.7 x 77.5 mm, 40 parts, among them J1 61300211121, J2 61300311121, J3 61300311121, T1 BC847BLT1G, T2 BC847BLT1G, T3 BC847BLT1G, T4 BC847BLT1G

Commit message: Minor changes done like the net name changed
Parts:
- moved SOLAR_CHARGER 1.27 mm to (50.2, 2.79)
Connections:
- net N$13 renamed VCCIO
Routing:
- net VCC: track 49.4 -> 50.0 mm
Changed lines of the file:
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@@
 <drawing>
 <settings>
-<setting alwaysvectorfont="no"/>
+<setting alwaysvectorfont="yes"/>
 <setting verticaltext="up"/>
 </settings>
@@
 <hole x="2.921" y="2.667" drill="3.048"/>
 <dimension x1="0" y1="-1.27" x2="60.706" y2="-1.27" x3="30.353" y3="-3.81" textsize="1.778" layer="1"/>
-<wire x1="0" y1="77.47" x2="60.706" y2="77.47" width="0.1524" layer="20"/>
-<wire x1="60.706" y1="77.47" x2="60.706" y2="0" width="0.1524" layer="20"/>
-<wire x1="60.706" y1="0" x2="0" y2="0" width="0.1524" layer="20"/>
-<wire x1="0" y1="0" x2="0" y2="77.47" width="0.1524" layer="20"/>
 <text x="12.192" y="68.199" size="0.508" layer="25" rot="R90">MIC_LRCLK</text>
 <text x="14.605" y="68.58" size="0.508" layer="25" rot="R90">MIC_DOUT</text>
@@
 <text x="53.975" y="54.356" size="0.508" layer="25">GND</text>
 <text x="54.61" y="51.816" size="0.508" layer="25">5V</text>
-<text x="47.879" y="4.445" size="0.6096" layer="25" rot="R90">GND</text>
-<text x="50.419" y="4.445" size="0.6096" layer="25" rot="R90">VCC</text>
-<text x="47.244" y="4.445" size="0.6096" layer="26" rot="MR90">GND</text>
-<text x="49.784" y="4.445" size="0.6096" layer="26" rot="MR90">VCC</text>
+<text x="49.149" y="4.445" size="0.6096" layer="25" rot="R90">GND</text>
+<text x="51.689" y="4.445" size="0.6096" layer="25" rot="R90">VCC</text>
+<text x="48.514" y="4.445" size="0.6096" layer="26" rot="MR90">GND</text>
+<text x="51.054" y="4.445" size="0.6096" layer="26" rot="MR90">VCC</text>
 <dimension x1="-2.54" y1="77.47" x2="-2.54" y2="0" x3="-3.81" y3="38.735" textsize="1.778" layer="1"/>
 <text x="18.034" y="7.366" size="2.1844" layer="26" rot="MR90">Wildly_Listen_Proto_V1</text>
@@
 <wire x1="60.706" y1="0" x2="60.706" y2="77.47" width="0.3048" layer="51"/>
 <wire x1="60.706" y1="77.47" x2="0" y2="77.47" width="0.3048" layer="51"/>
+<wire x1="0" y1="77.47" x2="60.706" y2="77.47" width="0.1524" layer="20"/>
+<wire x1="60.706" y1="77.47" x2="60.706" y2="0" width="0.1524" layer="20"/>
+<wire x1="60.706" y1="0" x2="0" y2="0" width="0.1524" layer="20"/>
+<wire x1="0" y1="0" x2="0" y2="77.47" width="0.1524" layer="20"/>
 </plain>
 <attributes>
@@
 <attribute name="VALUE" x="19.431" y="67.31" size="1.27" layer="27" rot="R270"/>
 </element>
-<element name="SOLAR_CHARGER" library="61300211121" package="61300211121" value="61300211121" x="48.895" y="2.794" smashed="yes" rot="R180">
-<attribute name="AVAILABILITY" value="Unavailable" x="48.895" y="2.794" size="1.778" layer="27" rot="R180" display="off"/>
-<attribute name="DESCRIPTION" value=" Board-To-Board Connector, Vertical, WR-PHD Series, Through Hole, Header, 2, 2.54 mm " x="48.895" y="2.794" size="1.778" layer="27" rot="R180" display="off"/>
-<attribute name="MF" value="Wurth Electronics" x="48.895" y="2.794" size="1.778" layer="27" rot="R180" display="off"/>
-<attribute name="MP" value="61300211121" x="48.895" y="2.794" size="1.778" layer="27" rot="R180" display="off"/>
-<attribute name="NAME" x="48.6462" y="1.1089" size="0.8128" layer="25" rot="R180" align="bottom-center"/>
-<attribute name="PACKAGE" value="None" x="48.895" y="2.794" size="1.778" layer="27" rot="R180" display="off"/>
-<attribute name="PRICE" value="None" x="48.895" y="2.794" size="1.778" layer="27" rot="R180" display="off"/>
-<attribute name="VALUE" x="51.0502" y="5.3342" size="0.8128" layer="27" rot="R180"/>
+<element name="SOLAR_CHARGER" library="61300211121" package="61300211121" value="61300211121" x="50.165" y="2.794" smashed="yes" rot="R180">
+<attribute name="AVAILABILITY" value="Unavailable" x="50.165" y="2.794" size="1.778" layer="27" rot="R180" display="off"/>
+<attribute name="DESCRIPTION" value=" Board-To-Board Connector, Vertical, WR-PHD Series, Through Hole, Header, 2, 2.54 mm " x="50.165" y="2.794" size="1.778" layer="27" rot="R180" display="off"/>
+<attribute name="MF" value="Wurth Electronics" x="50.165" y="2.794" size="1.778" layer="27" rot="R180" display="off"/>
+<attribute name="MP" value="61300211121" x="50.165" y="2.794" size="1.778" layer="27" rot="R180" display="off"/>
+<attribute name="NAME" x="49.9162" y="1.1089" size="0.8128" layer="25" rot="R180" align="bottom-center"/>
+<attribute name="PACKAGE" value="None" x="50.165" y="2.794" size="1.778" layer="27" rot="R180" display="off"/>
+<attribute name="PRICE" value="None" x="50.165" y="2.794" size="1.778" layer="27" rot="R180" display="off"/>
+<attribute name="VALUE" x="52.3202" y="5.3342" size="0.8128" layer="27" rot="R180"/>
 </element>
 <element name="SWITCH" library="EG1218" package="3PIN_SLIDE_SWITCH" value="GSM Power" x="42.418" y="73.914" smashed="yes">
@@
 <attribute name="MF" value="Wurth Electronics" x="54.483" y="30.099" size="1.778" layer="27" display="off"/>
 <attribute name="MP" value="61300211121" x="54.483" y="30.099" size="1.778" layer="27" display="off"/>
-<attribute name="NAME" x="54.4778" y="31.9111" size="0.8128" layer="25" align="bottom-center"/>
 <attribute name="PACKAGE" value="None" x="54.483" y="30.099" size="1.778" layer="27" display="off"/>
 <attribute name="PRICE" value="None" x="54.483" y="30.099" size="1.778" layer="27" display="off"/>
@@
 <attribute name="MF" value="Wurth Electronics" x="50.673" y="35.179" size="1.778" layer="27" rot="R90" display="off"/>
 <attribute name="MP" value="61300311121" x="50.673" y="35.179" size="1.778" layer="27" rot="R90" display="off"/>
-<attribute name="NAME" x="48.6609" y="35.2738" size="0.8128" layer="25" rot="R90" align="bottom-center"/>
 <attribute name="PACKAGE" value="None" x="50.673" y="35.179" size="1.778" layer="27" rot="R90" display="off"/>
 <attribute name="PRICE" value="None" x="50.673" y="35.179" size="1.778" layer="27" rot="R90" display="off"/>
@@
 <attribute name="MF" value="Wurth Electronics" x="58.293" y="35.179" size="1.778" layer="27" rot="R270" display="off"/>
 <attribute name="MP" value="61300311121" x="58.293" y="35.179" size="1.778" layer="27" rot="R270" display="off"/>
-<attribute name="NAME" x="60.3051" y="35.0842" size="0.8128" layer="25" rot="R270" align="bottom-center"/>
 <attribute name="PACKAGE" value="None" x="58.293" y="35.179" size="1.778" layer="27" rot="R270" display="off"/>
 <attribute name="PRICE" value="None" x="58.293" y="35.179" size="1.778" layer="27" rot="R270" display="off"/>
@@
 <contactref element="SOLAR_CHARGER" pad="1"/>
 <wire x1="49.53" y1="14.986" x2="49.53" y2="26.924" width="0.6096" layer="1"/>
-<wire x1="49.53" y1="14.986" x2="49.53" y2="3.429" width="0.6096" layer="1"/>
-<wire x1="50.165" y1="2.794" x2="49.53" y2="3.429" width="0.6096" layer="1"/>
+<wire x1="49.53" y1="14.986" x2="49.53" y2="4.699" width="0.6096" layer="1"/>
+<wire x1="51.435" y1="2.794" x2="49.53" y2="4.699" width="0.6096" layer="1"/>
 <contactref element="BATT" pad="1"/>
 <wire x1="49.53" y1="14.986" x2="51.324" y2="13.192" width="0.6096" layer="1"/>
@@
 <wire x1="55.626" y1="40.386" x2="55.626" y2="42.926" width="0.6096" layer="1"/>
 </signal>
-<signal name="N$13">
+<signal name="VCCIO">
+<contactref element="JP2" pad="2"/>
 <contactref element="WILDLY_5V_1A_BOOST" pad="7"/>
 <contactref element="JP3" pad="1"/>
@@
 <wire x1="56.896" y1="67.183" x2="56.896" y2="67.31" width="0.6096" layer="1"/>
 <wire x1="56.896" y1="67.183" x2="51.181" y2="61.468" width="0.6096" layer="1"/>
-<contactref element="JP2" pad="2"/>
-<wire x1="51.054" y1="45.466" x2="55.626" y2="45.466" width="0.6096" layer="1"/>
+<wire x1="55.626" y1="45.466" x2="51.308" y2="45.466" width="0.6096" layer="1"/>
+<wire x1="51.308" y1="45.466" x2="51.181" y2="45.593" width="0.6096" layer="1"/>
 </signal>
 </signals>

Commit message: Rework recroder board to be more compact, remove unnecessary components etc
Parts:
- removed 5V_INPUT: 61300211121, 61300211121:61300211121
- removed JP2, JP3: (no value), jumper:JP1
- removed NETSTATLED: (no value), adafruit:CHIP-LED0805
- removed R12: 870R, adafruit:M0805
- removed R4: 0R, adafruit:M0805
- removed R9: 1.65KR, adafruit:M0805
- removed SWITCH: GSM Power, EG1218:3PIN_SLIDE_SWITCH
- removed T4: BC847BLT1G, BC847BLT1G:SOT96P237X111-3N
- removed WILDLY_5V_1A_BOOST: (no value), adafruit:1X08-BIG
- added ON-OFF-SWITCH: Power, EG1218:3PIN_SLIDE_SWITCH
- moved WILDLY_I2S_MIC 19.3 mm to (35.1, 74.3)
- moved J2 17.8 mm to (50.4, 53.0)
- moved J3 17.8 mm to (58.0, 53.0)
- moved J1 17.8 mm to (54.2, 47.9)
- moved R10 4.93 mm to (9.91, 44.7)
- moved R14 4.44 mm to (13.0, 35.1)
- moved T3 4.10 mm to (14.4, 44.5)
- moved R2 3.57 mm to (18.8, 54.4)
- moved R13 3.05 mm to (18.7, 41.9)
- moved R3 2.09 mm to (18.8, 62.2)
- moved RECLED 2.05 mm to (9.91, 50.7), turned to 0 degrees
- moved T1 2.03 mm to (14.0, 63.0)
- moved JP1 1.98 mm to (14.4, 29.6)
- moved ERRLED 1.44 mm to (9.91, 59.6), turned to 0 degrees
- moved SDLED 1.37 mm to (10.2, 39.2), turned to 0 degrees
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Connections:
- removed net +5V: 5V_INPUT.1, C1.1, C2.1, R4.1, TEENSY_PIN_5.1, U$1.VIN
- removed net 5V_EN: SWITCH.1, WILDLY_5V_1A_BOOST.5
- removed net 5V_SUPPLY: R4.2, WILDLY_5V_1A_BOOST.1
- removed net LB: WILDLY_5V_1A_BOOST.3
- removed net N$12: J3.1, JP2.1
- removed net N$16: NETSTATLED.A, R12.1
- removed net N$5: NETSTATLED.C, T3.3
- removed net N$6: WILDLY_5V_1A_BOOST.6
- removed net N$7: R9.2, T3.1
- removed net VCCIO: JP2.2, JP3.1, WILDLY_5V_1A_BOOST.7
- new net VIN: C1.1, C2.1, J1.1, ON-OFF-SWITCH.2, TEENSY_PIN_5.1, U$1.VIN
- net +3V3: no longer R12.2
- net GND: no longer 5V_INPUT.2, SWITCH.2, T4.2, WILDLY_5V_1A_BOOST.2, WILDLY_5V_1A_BOOST.4
- net N$1: now also T3.3; no longer T4.3
- net N$11: now also T3.1; no longer T4.1
- net NETSTATLED: no longer R9.1
- net VCC: now also ON-OFF-SWITCH.1; no longer J1.1, JP3.2
Routing:
- net +5V: track 65.4 -> 0.00 mm
- net VIN: track 0.00 -> 52.7 mm
- net VCCIO: track 28.8 -> 0.00 mm
- net 5V_EN: track 28.6 -> 0.00 mm
- net 5V_SUPPLY: track 21.7 -> 0.00 mm, vias 1 -> 0
- net VCC: track 50.0 -> 33.3 mm
- net MIC_LRCLK: track 41.7 -> 26.2 mm, vias 2 -> 0
- net MIC_DOUT: track 61.9 -> 49.7 mm, vias 1 -> 0
- net 3V3: track 42.8 -> 30.8 mm
- net FUEL_GAUGE_SDA: track 19.8 -> 10.7 mm
- net FUEL_GAUGE_SCL: track 19.3 -> 10.7 mm
- net MIC_BCLK: track 44.4 -> 51.9 mm
- net N$12: track 6.31 -> 0.00 mm
- net N$7: track 5.66 -> 0.00 mm
- net N$16: track 3.75 -> 0.00 mm
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Other:
- board size 60.7 x 77.5 mm -> 55.4 x 78.2 mm
- board text added: "NC"
- board text added: "VBAT"
- board text added: "VIN"
- board text added: "Wildly_Listen_Recorder_V1"
- board text removed: "5V"
- board text removed: "5V_EN"
- board text removed: "Wildly_Listen_Proto_V1"

Commit message: Add GSM pinouts, clean signals and silk screen, etc
Parts:
- removed R10, R11, R14: 870R, adafruit:M0805
- removed R13: 1.65KR, adafruit:M0805
- added R1: 1.65KR, adafruit:M0805
- added R4, R5, R6: 870R, adafruit:M0805
- added R7, R8: 0R, adafruit:M0805
- added WIILDLY_GSM: (no value), pinhead:1X10
- moved ERRLED 8.73 mm to (11.2, 68.2)
- moved T1 7.17 mm to (16.8, 69.6)
- moved RECLED 5.86 mm to (11.7, 56.3)
- moved SDLED 5.06 mm to (11.7, 44.1)
- moved T3 4.58 mm to (15.9, 48.8)
- moved JP1 4.58 mm to (14.1, 34.2)
- moved T2 2.50 mm to (14.9, 57.7)
- moved R3 1.27 mm to (18.0, 63.2), turned to 90 degrees
Connections:
- net MIC_BCLK renamed PWM
- net MIC_DOUT renamed RST
- net MIC_LRCLK renamed RX
- net POWER_CONTRL renamed POWER_CONTROL
- new net N$10: R7.1, WIILDLY_GSM.3
- new net N$12: R8.1, WIILDLY_GSM.4
- new net NETSTAT: U$1.24, WIILDLY_GSM.9
- new net POWER_CNTROL: WIILDLY_GSM.10
- new net RESET_OF_GSM: WIILDLY_GSM.7
- net +3V3: now also R4.2, R5.2, R6.2; no longer R10.2, R11.2, R14.2
- net 3V3: now also WIILDLY_GSM.1
- net CTS_OF_GSM: now also WIILDLY_GSM.6
- net GND: now also WIILDLY_GSM.2
- net N$11: now also R1.2; no longer R13.2
- net N$14: now also R6.1; no longer R10.1
- net N$15: now also R5.1; no longer R11.1
- net N$9: now also R4.1; no longer R14.1
- net NET_STAT: no longer U$1.24
- net PWM_SARA: now also WIILDLY_GSM.8
- net RTS_OF_GSM: now also WIILDLY_GSM.5
- net RX_OF_GSM: now also R7.2
- net SDLED: now also R1.1; no longer R13.1
- net TX_OF_GSM: now also R8.2
Routing:
- net PWM_SARA: track 3.81 -> 48.4 mm, vias 0 -> 2
- net 3V3: track 30.8 -> 58.4 mm
- net NETSTAT: track 0.00 -> 17.1 mm, vias 0 -> 1
- net N$12: track 0.00 -> 12.6 mm
- net N$10: track 0.00 -> 10.2 mm
- net +3V3: track 41.5 -> 36.7 mm
- net N$2: track 5.95 -> 2.12 mm
- net NET_STAT: track 3.81 -> 0.00 mm
- net ERRLED: track 58.1 -> 60.4 mm
- net N$8: track 2.76 -> 4.55 mm
- net N$11: track 2.82 -> 4.45 mm
- net N$9: track 5.05 -> 3.71 mm
- net N$14: track 5.31 -> 4.24 mm
- net SDLED: track 49.0 -> 49.9 mm
- net N$1: track 5.40 -> 4.89 mm
Other:
- board text added: "3V"
- board text added: "CTS"
- board text added: "NETSTAT"
- board text added: "POWER_CONTROL"
- board text added: "PWM"
- board text added: "RESET"
- board text added: "RTS"
- board text added: "RX"
- board text added: "TX"

Commit message: Add GSM signals, rerouting for space efficiency and minor changes for fabrication
Parts:
- removed JP1: (no value), jumper:JP1
- added LED_JUMPER: (no value), jumper:JP1
- moved R4 5.18 mm to (10.7, 43.4), turned to 180 degrees
- moved R8 5.14 mm to (17.3, 20.1)
- moved T2 4.20 mm to (16.6, 61.5)
- moved R7 4.13 mm to (17.3, 16.8)
- moved SDLED 3.56 mm to (11.7, 47.6)
- moved R3 3.05 mm to (18.0, 66.3)
- moved R6 2.55 mm to (10.2, 53.1), turned to 180 degrees
- moved T1 2.54 mm to (16.8, 72.1)
- moved RECLED 1.85 mm to (11.2, 58.0)
- moved R1 1.63 mm to (17.7, 44.2)
- moved T3 1.48 mm to (16.6, 50.0)
- moved R2 1.27 mm to (17.8, 55.1), turned to 90 degrees
- moved R5 1.08 mm to (10.2, 63.5), turned to 180 degrees
Connections:
- removed net POWER_CNTROL: WIILDLY_GSM.10
- removed net RESET_OF_GSM: WIILDLY_GSM.7
- net +3V3: now also LED_JUMPER.1; no longer JP1.1
- net 3V3: now also LED_JUMPER.2; no longer JP1.2
- net NETSTATLED: no longer U$1.38
- net POWER_CONTROL: now also WIILDLY_GSM.10
- net RESET_GSM: now also WIILDLY_GSM.7
Routing:
- net POWER_CONTROL: track 3.81 -> 85.0 mm
- net RX_OF_GSM: track 3.81 -> 58.6 mm, vias 0 -> 2
- net RESET_GSM: track 3.81 -> 58.3 mm, vias 0 -> 2
- net TX_OF_GSM: track 3.81 -> 53.2 mm, vias 0 -> 1
- net RTS_OF_GSM: track 3.81 -> 50.0 mm
- net NETSTATLED: track 46.2 -> 0.00 mm, vias 1 -> 0
- net CTS_OF_GSM: track 3.81 -> 48.7 mm
- net 3V3: track 58.4 -> 71.0 mm
- net N$12: track 12.6 -> 7.99 mm
- net N$2: track 2.12 -> 5.52 mm
- net N$10: track 10.2 -> 7.57 mm
- net RECLED: track 60.5 -> 62.7 mm
- net SDLED: track 49.9 -> 51.6 mm
- net N$4: track 4.53 -> 5.92 mm
- net N$3: track 3.09 -> 4.47 mm
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Other:
- board size 55.4 x 78.2 mm -> 55.1 x 78 mm
