File: Teensy_Recorder/wildly_teensy_proto.brd (EAGLE design)
At the start: 55.1 x 78 mm, 34 parts, among them J1 61300211121, J2 61300311121, J3 61300311121, T1 BC847BLT1G, T2 BC847BLT1G, T3 BC847BLT1G

Commit message: Add RTC pinouts and associated silkscreen
Parts:
- added WILDLY_RTC: (no value), con-lstb:MA04-1
Connections:
- removed net 3V3: LED_JUMPER.2, TEENSY_PIN_3.3, TEENSY_PIN_5.3, U$1.3V3(1), U$1.3V3(2), U$1.3V3(3), U$1.3V3(4), WIILDLY_GSM.1, WILDLY_I2S_MIC.1
- removed net FUEL_GAUGE_SCL: J2.2, TEENSY_PIN_6.2, U$1.19
- removed net FUEL_GAUGE_SDA: J2.1, TEENSY_PIN_6.3, U$1.18
- new net 3V: LED_JUMPER.2, TEENSY_PIN_3.3, TEENSY_PIN_5.3, U$1.3V3(1), U$1.3V3(2), U$1.3V3(3), U$1.3V3(4), WIILDLY_GSM.1, WILDLY_I2S_MIC.1, WILDLY_RTC.1
- new net SCL: J2.2, TEENSY_PIN_6.2, U$1.19, WILDLY_RTC.3
- new net SDA: J2.1, TEENSY_PIN_6.3, U$1.18, WILDLY_RTC.4
- net GND: now also WILDLY_RTC.2
Routing:
- net 3V: track 0.00 -> 115.4 mm
- net 3V3: track 71.0 -> 0.00 mm
- net SCL: track 0.00 -> 23.0 mm
- net SDA: track 0.00 -> 16.1 mm
- net FUEL_GAUGE_SCL: track 10.7 -> 0.00 mm
- net FUEL_GAUGE_SDA: track 10.7 -> 0.00 mm
- net VIN: track 52.7 -> 51.8 mm
Other:
- board text added: "SCL"
- board text added: "SDA"
Changed lines of the file:
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@@
 <?xml version="1.0" encoding="utf-8"?>
 <!DOCTYPE eagle SYSTEM "eagle.dtd">
-<eagle version="9.3.2">
+<eagle version="9.3.0">
 <drawing>
 <settings>
-<setting alwaysvectorfont="yes"/>
+<setting alwaysvectorfont="no"/>
 <setting verticaltext="up"/>
 </settings>
@@
 <text x="51.943" y="11.43" size="0.6096" layer="25" rot="R180">GND</text>
 <text x="51.943" y="13.462" size="0.6096" layer="25" rot="R180">VCC</text>
-<text x="58.166" y="44.45" size="1.016" layer="25" rot="R180">FUEL_GAUGE</text>
+<text x="58.928" y="58.674" size="1.016" layer="25" rot="R180">FUEL_GAUGE</text>
 <wire x1="5.588" y1="77.216" x2="5.588" y2="-0.508" width="0.3048" layer="51"/>
 <wire x1="5.588" y1="-0.508" x2="60.706" y2="-0.508" width="0.3048" layer="51"/>
@@
 <text x="57.277" y="33.655" size="1.778" layer="26" rot="MR0">OFF</text>
 <text x="56.642" y="18.923" size="1.778" layer="26" rot="MR0">ON</text>
+<text x="53.721" y="38.862" size="0.6096" layer="25" rot="R180">GND</text>
+<text x="53.213" y="36.322" size="0.6096" layer="25" rot="R180">3V</text>
+<text x="53.467" y="35.814" size="0.508" layer="26" rot="MR0">3V3</text>
+<text x="53.467" y="38.354" size="0.508" layer="26" rot="MR0">GND</text>
+<text x="53.721" y="44.196" size="0.6096" layer="25" rot="R180">SDA</text>
+<text x="53.467" y="41.402" size="0.6096" layer="25" rot="R180">SCL</text>
+<text x="53.467" y="40.894" size="0.508" layer="26" rot="MR0">SCL</text>
+<text x="53.467" y="43.688" size="0.508" layer="26" rot="MR0">SDA</text>
 </plain>
 <attributes>
@@
 <param name="mdViaViaSameLayer" value="8mil"/>
 <param name="mnLayersViaInSmd" value="2"/>
-<param name="mdCopperDimension" value="8mil"/>
+<param name="mdCopperDimension" value="10mil"/>
 <param name="mdDrill" value="8mil"/>
 <param name="mdSmdStop" value="0mil"/>
@@
 <param name="mlMinCreamFrame" value="0mil"/>
 <param name="mlMaxCreamFrame" value="0mil"/>
-<param name="mlViaStopLimit" value="20mil"/>
+<param name="mlViaStopLimit" value="25mil"/>
 <param name="srRoundness" value="0"/>
 <param name="srMinRoundness" value="0mil"/>
@@
 <attribute name="PACKAGE" value="None" x="54.229" y="47.879" size="1.778" layer="27" display="off"/>
 <attribute name="PRICE" value="None" x="54.229" y="47.879" size="1.778" layer="27" display="off"/>
-<attribute name="VALUE" x="52.0738" y="45.3388" size="0.8128" layer="27"/>
 </element>
 <element name="J2" library="61300311121" package="61300311121" value="61300311121" x="50.419" y="52.959" smashed="yes" rot="R90">
@@
 <attribute name="PACKAGE" value="None" x="50.419" y="52.959" size="1.778" layer="27" rot="R90" display="off"/>
 <attribute name="PRICE" value="None" x="50.419" y="52.959" size="1.778" layer="27" rot="R90" display="off"/>
-<attribute name="VALUE" x="52.9592" y="50.8038" size="0.8128" layer="27" rot="R90"/>
 </element>
 <element name="J3" library="61300311121" package="61300311121" value="61300311121" x="58.039" y="52.959" smashed="yes" rot="R270">
@@
 <attribute name="PACKAGE" value="None" x="58.039" y="52.959" size="1.778" layer="27" rot="R270" display="off"/>
 <attribute name="PRICE" value="None" x="58.039" y="52.959" size="1.778" layer="27" rot="R270" display="off"/>
-<attribute name="VALUE" x="55.4988" y="55.1142" size="0.8128" layer="27" rot="R270"/>
 </element>
 <element name="WIILDLY_GSM" library="pinhead" library_urn="urn:adsk.eagle:library:325" package="1X10" package3d_urn="urn:adsk.eagle:package:22406/2" value="" x="9.906" y="20.066" smashed="yes" rot="R90">
@@
 <attribute name="NAME" x="16.256" y="21.082" size="0.8128" layer="25"/>
 <attribute name="VALUE" x="16.51" y="18.034" size="0.8128" layer="27"/>
+</element>
+<element name="WILDLY_RTC" library="con-lstb" library_urn="urn:adsk.eagle:library:162" package="MA04-1" package3d_urn="urn:adsk.eagle:package:8337/1" value="" x="50.038" y="39.878" smashed="yes" rot="R90">
+<attribute name="MF" value="" x="50.038" y="39.878" size="1.778" layer="27" rot="R90" display="off"/>
+<attribute name="MPN" value="" x="50.038" y="39.878" size="1.778" layer="27" rot="R90" display="off"/>
+<attribute name="NAME" x="46.863" y="34.544" size="1.27" layer="26" ratio="10" rot="MR90"/>
+<attribute name="OC_FARNELL" value="unknown" x="50.038" y="39.878" size="1.778" layer="27" rot="R90" display="off"/>
+<attribute name="OC_NEWARK" value="unknown" x="50.038" y="39.878" size="1.778" layer="27" rot="R90" display="off"/>
+<attribute name="VALUE" x="48.387" y="40.513" size="1.27" layer="27" ratio="10" rot="R90"/>
 </element>
 </elements>
@@
 </polygon>
 <contactref element="WIILDLY_GSM" pad="2"/>
+<contactref element="WILDLY_RTC" pad="2"/>
 </signal>
 <signal name="TX_OF_GSM">
@@
 <wire x1="17.837" y1="45.14975625" x2="17.653" y2="45.146" width="0.508" layer="1"/>
 </signal>
-<signal name="3V3">
+<signal name="3V">
 <contactref element="U$1" pad="3V3(1)"/>
 <contactref element="U$1" pad="3V3(2)"/>
@@
 <wire x1="16.383" y1="38.735" x2="16.383" y2="38.227" width="0.3048" layer="1"/>
 <wire x1="16.383" y1="38.227" x2="16.256" y2="38.1" width="0.3048" layer="1"/>
-<wire x1="16.383" y1="38.735" x2="40.378" y2="61.222" width="0" layer="19" extent="1-16"/>
+<contactref element="WILDLY_RTC" pad="1"/>
+<wire x1="45.466" y1="60.96" x2="57.404" y2="60.96" width="0.4064" layer="16"/>
+<wire x1="56.642" y1="40.894" x2="56.642" y2="38.608" width="0.4064" layer="16"/>
+<wire x1="56.642" y1="38.608" x2="54.102" y2="36.068" width="0.4064" layer="16"/>
+<wire x1="54.102" y1="36.068" x2="50.038" y2="36.068" width="0.4064" layer="16"/>
+<wire x1="57.404" y1="60.96" x2="59.944" y2="58.42" width="0.4064" layer="16"/>
+<wire x1="59.944" y1="58.42" x2="59.944" y2="44.196" width="0.4064" layer="16"/>
+<wire x1="59.944" y1="44.196" x2="56.642" y2="40.894" width="0.4064" layer="16"/>
+<wire x1="26.8589" y1="30.48" x2="50.038" y2="36.068" width="0" layer="19" extent="16-16"/>
 <wire x1="31.496" y1="20.32" x2="26.8589" y2="30.48" width="0" layer="19" extent="16-16"/>
 <wire x1="36.576" y1="7.62" x2="31.496" y2="20.32" width="0" layer="19" extent="1-1"/>
@@
 <contactref element="TEENSY_PIN_7" pad="5"/>
 <wire x1="45.466" y1="25.4" x2="41.656" y2="25.4" width="0.6096" layer="16"/>
-</signal>
-<signal name="FUEL_GAUGE_SDA">
-<contactref element="U$1" pad="18"/>
-<contactref element="TEENSY_PIN_6" pad="3"/>
-<wire x1="41.656" y1="45.72" x2="45.466" y2="45.72" width="0.3048" layer="16"/>
-<contactref element="J2" pad="1"/>
-<wire x1="50.419" y1="50.419" x2="45.72" y2="45.72" width="0.3048" layer="1"/>
-<wire x1="45.466" y1="45.72" x2="45.72" y2="45.72" width="0.3048" layer="1"/>
-</signal>
-<signal name="FUEL_GAUGE_SCL">
-<contactref element="U$1" pad="19"/>
-<contactref element="TEENSY_PIN_6" pad="2"/>
-<wire x1="41.656" y1="48.26" x2="45.466" y2="48.26" width="0.3048" layer="16"/>
-<contactref element="J2" pad="2"/>
-<wire x1="50.419" y1="52.959" x2="45.72" y2="48.26" width="0.3048" layer="1"/>
-<wire x1="45.466" y1="48.26" x2="45.72" y2="48.26" width="0.3048" layer="1"/>
 </signal>
 <signal name="VCC">
@@
 <wire x1="52.959" y1="57.531" x2="52.959" y2="47.879" width="0.6096" layer="1"/>
 <wire x1="52.959" y1="47.879" x2="53.721" y2="47.117" width="0.6096" layer="1"/>
-<wire x1="53.721" y1="47.117" x2="53.721" y2="27.051" width="0.6096" layer="1"/>
-<wire x1="53.721" y1="27.051" x2="55.245" y2="27.051" width="0.508" layer="1"/>
-<wire x1="55.245" y1="27.051" x2="55.372" y2="27.178" width="0.508" layer="1"/>
+<wire x1="53.721" y1="47.117" x2="53.721" y2="28.448" width="0.6096" layer="1"/>
 <wire x1="51.435" y1="66.128" x2="51.977" y2="65.586" width="0.508" layer="1"/>
 <wire x1="51.977" y1="65.586" x2="52.39541875" y2="65.586" width="0.508" layer="1"/>
@@
 <wire x1="54.102" y1="58.674" x2="52.959" y2="57.531" width="0.508" layer="1"/>
 <wire x1="54.102" y1="63.87941875" x2="54.102" y2="58.674" width="0.508" layer="1"/>
+<wire x1="53.721" y1="28.448" x2="54.991" y2="27.178" width="0.508" layer="1"/>
+<wire x1="54.991" y1="27.178" x2="55.372" y2="27.178" width="0.508" layer="1"/>
 </signal>
 <signal name="N$10">
@@
 <wire x1="17.018" y1="27.94" x2="20.818971875" y2="27.949028125" width="0.4064" layer="16"/>
 </signal>
+<signal name="SDA">
+<contactref element="WILDLY_RTC" pad="4"/>
+<contactref element="U$1" pad="18"/>
+<contactref element="J2" pad="1"/>
+<contactref element="TEENSY_PIN_6" pad="3"/>
+<wire x1="41.656" y1="45.72" x2="45.466" y2="45.72" width="0.4064" layer="16"/>
+<wire x1="45.466" y1="45.72" x2="50.165" y2="50.419" width="0.4064" layer="16"/>
+<wire x1="50.165" y1="50.419" x2="50.419" y2="50.419" width="0.4064" layer="16"/>
+<wire x1="45.466" y1="45.72" x2="47.498" y2="43.688" width="0.4064" layer="1"/>
+<wire x1="47.498" y1="43.688" x2="50.038" y2="43.688" width="0.4064" layer="1"/>
+</signal>
+<signal name="SCL">
+<contactref element="WILDLY_RTC" pad="3"/>
+<contactref element="U$1" pad="19"/>
+<contactref element="J2" pad="2"/>
+<contactref element="TEENSY_PIN_6" pad="2"/>
+<wire x1="41.656" y1="48.26" x2="45.466" y2="48.26" width="0.4064" layer="16"/>
+<wire x1="45.466" y1="48.26" x2="45.72" y2="48.26" width="0.4064" layer="16"/>
+<wire x1="45.72" y1="48.26" x2="50.419" y2="52.959" width="0.4064" layer="16"/>
+<wire x1="45.466" y1="48.26" x2="48.768" y2="44.958" width="0.4064" layer="1"/>
+<wire x1="48.768" y1="44.958" x2="51.37685625" y2="44.958" width="0.4064" layer="1"/>
+<wire x1="51.37685625" y1="44.958" x2="52.1208" y2="44.21405625" width="0.4064" layer="1"/>
+<wire x1="52.1208" y1="44.21405625" x2="52.1208" y2="43.16194375" width="0.4064" layer="1"/>
+<wire x1="52.1208" y1="43.16194375" x2="51.37685625" y2="42.418" width="0.4064" layer="1"/>
+<wire x1="51.37685625" y1="42.418" x2="51.308" y2="42.418" width="0.4064" layer="1"/>
+<wire x1="51.308" y1="42.418" x2="50.038" y2="41.148" width="0.4064" layer="1"/>
+</signal>
 </signals>
