File: Teensy_Recorder/wildly_teensy_proto.sch (EAGLE design)
At the start: 40 parts, among them J1 61300211121, J2 61300311121, J3 61300311121, T1 BC847BLT1G, T2 BC847BLT1G, T3 BC847BLT1G, T4 BC847BLT1G

Commit message: Minor changes done like the net name changed
Connections:
- net N$13 renamed VCCIO
Changed lines of the file:
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@@
 </segment>
 </net>
-<net name="N$13" class="0">
+<net name="VCCIO" class="0">
+<segment>
+<pinref part="JP2" gate="A" pin="2"/>
+<wire x1="189.738" y1="135.89" x2="200.66" y2="135.89" width="0.1524" layer="91"/>
+<label x="193.548" y="135.89" size="1.778" layer="95"/>
+</segment>
 <segment>
 <pinref part="WILDLY_5V_1A_BOOST" gate="G$1" pin="7"/>
@@
 <label x="-68.58" y="73.66" size="1.778" layer="95"/>
 </segment>
-<segment>
-<pinref part="JP2" gate="A" pin="2"/>
-<wire x1="189.738" y1="135.89" x2="200.66" y2="135.89" width="0.1524" layer="91"/>
-<label x="193.548" y="135.89" size="1.778" layer="95"/>
-</segment>
 </net>

Commit message: Rework recroder board to be more compact, remove unnecessary components etc
Parts:
- removed 5V_INPUT: 61300211121, 61300211121:61300211121
- removed JP2, JP3: (no value), jumper:JP1Q
- removed NETSTATLED: (no value), adafruit:LEDCHIP-LED0805
- removed R12: 870R, adafruit:R-US_M0805
- removed R4: 0R, adafruit:R-US_M0805
- removed R9: 1.65KR, adafruit:R-US_M0805
- removed T4: BC847BLT1G, BC847BLT1G:BC847BLT1G
- removed WILDLY_5V_1A_BOOST: (no value), adafruit:PINHD-1X8BIG
- ON-OFF-SWITCH: value GSM Power -> Power
- renumbered SWITCH to ON-OFF-SWITCH
Connections:
- removed net +5V: 5V_INPUT.1, C1.1, C2.1, R4.1, TEENSY_PIN_5.1, U$1.VIN
- removed net 5V_EN: ON-OFF-SWITCH.1, WILDLY_5V_1A_BOOST.5
- removed net 5V_SUPPLY: R4.2, WILDLY_5V_1A_BOOST.1
- removed net LB: WILDLY_5V_1A_BOOST.3
- removed net N$12: J3.1, JP2.1
- removed net N$16: NETSTATLED.A, R12.1
- removed net N$5: NETSTATLED.C, T3.C
- removed net N$6: WILDLY_5V_1A_BOOST.6
- removed net N$7: R9.2, T3.B
- removed net VCCIO: JP2.2, JP3.1, WILDLY_5V_1A_BOOST.7
- new net VIN: C1.1, C2.1, J1.1, ON-OFF-SWITCH.COM, TEENSY_PIN_5.1, U$1.VIN
- net +3V3: no longer R12.2
- net GND: no longer 5V_INPUT.2, ON-OFF-SWITCH.COM, T4.E, WILDLY_5V_1A_BOOST.2, WILDLY_5V_1A_BOOST.4
- net N$1: now also T3.C; no longer T4.C
- net N$11: now also T3.B; no longer T4.B
- net NETSTATLED: no longer R9.1
- net VCC: now also ON-OFF-SWITCH.1; no longer J1.1, JP3.2
Other:
- note added: "ON/OFF"
- note removed: "5V"
- note removed: "5V - SUPPLY"
- note removed: "5V Boost 1A"
- note removed: "5V Out EN - Transmitter On/Off"
- note removed: "EN"
- note removed: "GND"
- note removed: "LB"
- note removed: "VBAT"
- note removed: "VS"
- note removed: "VUSB"
- moved on the sheet: T3

Commit message: Add GSM pinouts, clean signals and silk screen, etc
Parts:
- added R7, R8: 0R, adafruit:R-US_M0805
- added WIILDLY_GSM: (no value), pinhead:PINHD-1X10
- renumbered R10 to R6, R11 to R5, R13 to R1, R14 to R4
Connections:
- net MIC_BCLK renamed PWM
- net MIC_DOUT renamed RST
- net MIC_LRCLK renamed RX
- net POWER_CONTRL renamed POWER_CONTROL
- new net N$10: R7.1, WIILDLY_GSM.3
- new net N$12: R8.1, WIILDLY_GSM.4
- new net NETSTAT: U$1.24, WIILDLY_GSM.9
- new net POWER_CNTROL: WIILDLY_GSM.10
- new net RESET_OF_GSM: WIILDLY_GSM.7
- net 3V3: now also WIILDLY_GSM.1
- net CTS_OF_GSM: now also WIILDLY_GSM.6
- net GND: now also WIILDLY_GSM.2
- net NET_STAT: no longer U$1.24
- net PWM_SARA: now also WIILDLY_GSM.8
- net RTS_OF_GSM: now also WIILDLY_GSM.5
- net RX_OF_GSM: now also R7.2
- net TX_OF_GSM: now also R8.2
Other:
- note added: "Wildly UBLOX GSM Board"

Commit message: Add GSM signals, rerouting for space efficiency and minor changes for fabrication
Parts:
- renumbered JP1 to LED_JUMPER
Connections:
- removed net POWER_CNTROL: WIILDLY_GSM.10
- removed net RESET_OF_GSM: WIILDLY_GSM.7
- net NETSTATLED: no longer U$1.38/A19/PWM/SDA1
- net POWER_CONTROL: now also WIILDLY_GSM.10
- net RESET_GSM: now also WIILDLY_GSM.7
Changed lines of the file:
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@@
 <grid distance="0.1" unitdist="inch" unit="inch" style="lines" multiple="1" display="no" altdistance="0.01" altunitdist="inch" altunit="inch"/>
 <layers>
-<layer number="1" name="Top" color="4" fill="1" visible="yes" active="no"/>
-<layer number="16" name="Bottom" color="1" fill="1" visible="yes" active="no"/>
-<layer number="17" name="Pads" color="2" fill="1" visible="yes" active="no"/>
-<layer number="18" name="Vias" color="2" fill="1" visible="yes" active="no"/>
-<layer number="19" name="Unrouted" color="6" fill="1" visible="yes" active="no"/>
-<layer number="20" name="Dimension" color="24" fill="1" visible="yes" active="no"/>
-<layer number="21" name="tPlace" color="7" fill="1" visible="yes" active="no"/>
-<layer number="22" name="bPlace" color="7" fill="1" visible="yes" active="no"/>
-<layer number="23" name="tOrigins" color="15" fill="1" visible="yes" active="no"/>
-<layer number="24" name="bOrigins" color="15" fill="1" visible="yes" active="no"/>
-<layer number="25" name="tNames" color="7" fill="1" visible="yes" active="no"/>
-<layer number="26" name="bNames" color="7" fill="1" visible="yes" active="no"/>
-<layer number="27" name="tValues" color="7" fill="1" visible="yes" active="no"/>
-<layer number="28" name="bValues" color="7" fill="1" visible="yes" active="no"/>
+<layer number="1" name="Top" color="4" fill="1" visible="no" active="no"/>
+<layer number="16" name="Bottom" color="1" fill="1" visible="no" active="no"/>
+<layer number="17" name="Pads" color="2" fill="1" visible="no" active="no"/>
+<layer number="18" name="Vias" color="2" fill="1" visible="no" active="no"/>
+<layer number="19" name="Unrouted" color="6" fill="1" visible="no" active="no"/>
+<layer number="20" name="Dimension" color="24" fill="1" visible="no" active="no"/>
+<layer number="21" name="tPlace" color="7" fill="1" visible="no" active="no"/>
+<layer number="22" name="bPlace" color="7" fill="1" visible="no" active="no"/>
+<layer number="23" name="tOrigins" color="15" fill="1" visible="no" active="no"/>
+<layer number="24" name="bOrigins" color="15" fill="1" visible="no" active="no"/>
+<layer number="25" name="tNames" color="7" fill="1" visible="no" active="no"/>
+<layer number="26" name="bNames" color="7" fill="1" visible="no" active="no"/>
+<layer number="27" name="tValues" color="7" fill="1" visible="no" active="no"/>
+<layer number="28" name="bValues" color="7" fill="1" visible="no" active="no"/>
 <layer number="29" name="tStop" color="7" fill="3" visible="no" active="no"/>
 <layer number="30" name="bStop" color="7" fill="6" visible="no" active="no"/>
@@
 <layer number="35" name="tGlue" color="7" fill="4" visible="no" active="no"/>
 <layer number="36" name="bGlue" color="7" fill="5" visible="no" active="no"/>
-<layer number="37" name="tTest" color="7" fill="1" visible="yes" active="no"/>
-<layer number="38" name="bTest" color="7" fill="1" visible="yes" active="no"/>
+<layer number="37" name="tTest" color="7" fill="1" visible="no" active="no"/>
+<layer number="38" name="bTest" color="7" fill="1" visible="no" active="no"/>
 <layer number="39" name="tKeepout" color="4" fill="11" visible="no" active="no"/>
 <layer number="40" name="bKeepout" color="1" fill="11" visible="no" active="no"/>
@@
 <layer number="44" name="Drills" color="7" fill="1" visible="no" active="no"/>
 <layer number="45" name="Holes" color="7" fill="1" visible="no" active="no"/>
-<layer number="46" name="Milling" color="3" fill="1" visible="yes" active="no"/>
-<layer number="47" name="Measures" color="7" fill="1" visible="yes" active="no"/>
-<layer number="48" name="Document" color="7" fill="1" visible="yes" active="no"/>
-<layer number="49" name="Reference" color="7" fill="1" visible="yes" active="no"/>
-<layer number="50" name="dxf" color="7" fill="1" visible="yes" active="no"/>
-<layer number="51" name="tDocu" color="7" fill="1" visible="yes" active="no"/>
-<layer number="52" name="bDocu" color="7" fill="1" visible="yes" active="no"/>
-<layer number="53" name="tPadExt" color="7" fill="1" visible="yes" active="no"/>
-<layer number="54" name="bPadExt" color="1" fill="1" visible="yes" active="no"/>
-<layer number="56" name="wert" color="7" fill="1" visible="yes" active="no"/>
-<layer number="57" name="tCAD" color="7" fill="1" visible="yes" active="no"/>
-<layer number="59" name="tCarbon" color="7" fill="1" visible="yes" active="no"/>
-<layer number="60" name="bCarbon" color="7" fill="1" visible="yes" active="no"/>
+<layer number="46" name="Milling" color="3" fill="1" visible="no" active="no"/>
+<layer number="47" name="Measures" color="7" fill="1" visible="no" active="no"/>
+<layer number="48" name="Document" color="7" fill="1" visible="no" active="no"/>
+<layer number="49" name="Reference" color="7" fill="1" visible="no" active="no"/>
+<layer number="50" name="dxf" color="7" fill="1" visible="no" active="no"/>
+<layer number="51" name="tDocu" color="7" fill="1" visible="no" active="no"/>
+<layer number="52" name="bDocu" color="7" fill="1" visible="no" active="no"/>
+<layer number="53" name="tPadExt" color="7" fill="1" visible="no" active="no"/>
+<layer number="54" name="bPadExt" color="1" fill="1" visible="no" active="no"/>
+<layer number="56" name="wert" color="7" fill="1" visible="no" active="no"/>
+<layer number="57" name="tCAD" color="7" fill="1" visible="no" active="no"/>
+<layer number="59" name="tCarbon" color="7" fill="1" visible="no" active="no"/>
+<layer number="60" name="bCarbon" color="7" fill="1" visible="no" active="no"/>
 <layer number="88" name="SimResults" color="9" fill="1" visible="yes" active="yes"/>
 <layer number="89" name="SimProbes" color="9" fill="1" visible="yes" active="yes"/>
@@
 <part name="P+1" library="supply1" library_urn="urn:adsk.eagle:library:371" deviceset="VCC" device="" value="V_BATT"/>
 <part name="P+4" library="supply1" library_urn="urn:adsk.eagle:library:371" deviceset="VCC" device="" value="V_BATT"/>
-<part name="JP1" library="jumper" library_urn="urn:adsk.eagle:library:252" deviceset="JP1Q" device="" package3d_urn="urn:adsk.eagle:package:15455/1"/>
+<part name="LED_JUMPER" library="jumper" library_urn="urn:adsk.eagle:library:252" deviceset="JP1Q" device="" package3d_urn="urn:adsk.eagle:package:15455/1"/>
 <part name="T3" library="BC847BLT1G" deviceset="BC847BLT1G" device=""/>
 <part name="T1" library="BC847BLT1G" deviceset="BC847BLT1G" device=""/>
@@
 <attribute name="VALUE" x="81.28" y="137.16" size="1.778" layer="96" rot="R90"/>
 </instance>
-<instance part="JP1" gate="A" x="-5.08" y="91.44" smashed="yes" rot="R270">
+<instance part="LED_JUMPER" gate="A" x="-5.08" y="91.44" smashed="yes" rot="R270">
 <attribute name="NAME" x="-7.62" y="93.98" size="1.778" layer="95"/>
 <attribute name="VALUE" x="-10.16" y="86.995" size="1.778" layer="96"/>
@@
 <label x="162.56" y="-7.62" size="1.778" layer="95"/>
 </segment>
+<segment>
+<pinref part="WIILDLY_GSM" gate="A" pin="7"/>
+<wire x1="-99.06" y1="-35.56" x2="-127" y2="-35.56" width="0.1524" layer="91"/>
+<label x="-127" y="-35.56" size="1.778" layer="95"/>
+</segment>
 </net>
 <net name="CTS_OF_GSM" class="0">
@@
 </net>
 <net name="NETSTATLED" class="0">
-<segment>
-<pinref part="U$1" gate="G$1" pin="38/A19/PWM/SDA1"/>
-<wire x1="99.06" y1="-2.54" x2="119.38" y2="-2.54" width="0.1524" layer="91"/>
-<label x="101.6" y="-2.54" size="1.778" layer="95"/>
-</segment>
 <segment>
 <pinref part="TEENSY_PIN_8" gate="A" pin="1"/>
@@
 <label x="223.52" y="-15.24" size="1.778" layer="95"/>
 </segment>
+<segment>
+<pinref part="WIILDLY_GSM" gate="A" pin="10"/>
+<wire x1="-99.06" y1="-43.18" x2="-127" y2="-43.18" width="0.1524" layer="91"/>
+<label x="-127" y="-43.18" size="1.778" layer="95"/>
+</segment>
 </net>
 <net name="N$14" class="0">
@@
 <label x="-84.328" y="2.794" size="1.778" layer="95" rot="R180"/>
 <wire x1="30.48" y1="91.44" x2="2.54" y2="91.44" width="0.1524" layer="91"/>
-<pinref part="JP1" gate="A" pin="2"/>
+<pinref part="LED_JUMPER" gate="A" pin="2"/>
 </segment>
 <segment>
@@
 <net name="+3V3" class="0">
 <segment>
-<pinref part="JP1" gate="A" pin="1"/>
+<pinref part="LED_JUMPER" gate="A" pin="1"/>
 <wire x1="-12.7" y1="91.44" x2="-20.32" y2="91.44" width="0.1524" layer="91"/>
 <pinref part="+3V3" gate="G$1" pin="+3V3"/>
@@
 </segment>
 </net>
-<net name="RESET_OF_GSM" class="0">
-<segment>
-<pinref part="WIILDLY_GSM" gate="A" pin="7"/>
-<wire x1="-99.06" y1="-35.56" x2="-127" y2="-35.56" width="0.1524" layer="91"/>
-<label x="-127" y="-35.56" size="1.778" layer="95"/>
-</segment>
-</net>
 <net name="NETSTAT" class="0">
 <segment>
@@
 </segment>
 </net>
-<net name="POWER_CNTROL" class="0">
-<segment>
-<pinref part="WIILDLY_GSM" gate="A" pin="10"/>
-<wire x1="-99.06" y1="-43.18" x2="-127" y2="-43.18" width="0.1524" layer="91"/>
-<label x="-127" y="-43.18" size="1.778" layer="95"/>
-</segment>
-</net>

Commit message: Add RTC pinouts and associated silkscreen
Parts:
- added WILDLY_RTC: (no value), con-lstb:MA04-1
Connections:
- removed net 3V3: LED_JUMPER.2, TEENSY_PIN_3.3, TEENSY_PIN_5.3, U$1.3V3, WIILDLY_GSM.1, WILDLY_I2S_MIC.1
- removed net FUEL_GAUGE_SCL: J2.2, TEENSY_PIN_6.2, U$1.19/A5/PWM/T/SCL0
- removed net FUEL_GAUGE_SDA: J2.1, TEENSY_PIN_6.3, U$1.18/A4/PWM/T/SDA0
- new net 3V: LED_JUMPER.2, TEENSY_PIN_3.3, TEENSY_PIN_5.3, U$1.3V3, WIILDLY_GSM.1, WILDLY_I2S_MIC.1, WILDLY_RTC.1
- new net SCL: J2.2, TEENSY_PIN_6.2, U$1.19/A5/PWM/T/SCL0, WILDLY_RTC.3
- new net SDA: J2.1, TEENSY_PIN_6.3, U$1.18/A4/PWM/T/SDA0, WILDLY_RTC.4
- net GND: now also WILDLY_RTC.2
Other:
- note added: "Wildly I2S Microphone SPH0645LM4H"
- note added: "Wildly RTC"
- note removed: "Adafruit I2S Microphone SPH0645LM4H"
Changed lines of the file:
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@@
 <?xml version="1.0" encoding="utf-8"?>
 <!DOCTYPE eagle SYSTEM "eagle.dtd">
-<eagle version="9.3.2">
+<eagle version="9.3.0">
 <drawing>
 <settings>
@@
 <part name="R7" library="adafruit" library_urn="urn:adsk.eagle:library:420" deviceset="R-US_" device="M0805" package3d_urn="urn:adsk.eagle:package:6240587/1" value="0R"/>
 <part name="R8" library="adafruit" library_urn="urn:adsk.eagle:library:420" deviceset="R-US_" device="M0805" package3d_urn="urn:adsk.eagle:package:6240587/1" value="0R"/>
+<part name="WILDLY_RTC" library="con-lstb" library_urn="urn:adsk.eagle:library:162" deviceset="MA04-1" device="" package3d_urn="urn:adsk.eagle:package:8337/1"/>
 </parts>
 <sheets>
 <sheet>
 <plain>
-<text x="-91.44" y="-5.08" size="1.778" layer="91">Adafruit I2S Microphone SPH0645LM4H </text>
 <text x="27.94" y="142.24" size="1.778" layer="91">ON/OFF</text>
 <text x="93.98" y="139.7" size="1.778" layer="91">Solar Charger</text>
@@
 <text x="152.4" y="149.86" size="2.54" layer="91">Fuel Gauge</text>
 <text x="-121.92" y="-53.34" size="1.778" layer="91">Wildly UBLOX GSM Board</text>
+<text x="-96.52" y="-5.08" size="1.778" layer="91">Wildly I2S Microphone SPH0645LM4H </text>
+<text x="-144.78" y="-5.08" size="1.778" layer="91">Wildly RTC</text>
 </plain>
 <instances>
@@
 <attribute name="NAME" x="-135.6614" y="-29.21" size="1.778" layer="95" rot="R270"/>
 <attribute name="VALUE" x="-135.382" y="-34.29" size="1.778" layer="96" rot="R270"/>
+</instance>
+<instance part="WILDLY_RTC" gate="1" x="-134.62" y="10.16" smashed="yes" rot="MR0">
+<attribute name="VALUE" x="-133.35" y="0" size="1.778" layer="96" rot="MR0"/>
+<attribute name="NAME" x="-130.81" y="-1.778" size="1.778" layer="95" rot="MR0"/>
 </instance>
 </instances>
@@
 <pinref part="GND4" gate="1" pin="GND"/>
 </segment>
+<segment>
+<pinref part="WILDLY_RTC" gate="1" pin="2"/>
+<wire x1="-142.24" y1="7.62" x2="-147.32" y2="7.62" width="0.1524" layer="91"/>
+<label x="-147.32" y="7.62" size="1.778" layer="95"/>
+</segment>
+<segment>
+<label x="-125.984" y="7.874" size="1.778" layer="95" rot="R180"/>
+</segment>
 </net>
 <net name="TX_OF_GSM" class="0">
@@
 <wire x1="-73.66" y1="12.7" x2="-58.42" y2="12.7" width="0.1524" layer="91"/>
 <label x="-58.42" y="12.7" size="1.778" layer="95"/>
-<label x="-94.996" y="11.938" size="1.778" layer="95"/>
+<label x="-84.836" y="11.938" size="1.778" layer="95"/>
 </segment>
 <segment>
@@
 </segment>
 </net>
-<net name="3V3" class="0">
+<net name="3V" class="0">
 <segment>
 <pinref part="U$1" gate="G$1" pin="3V3"/>
@@
 <label x="-142.24" y="-20.32" size="1.778" layer="95"/>
 </segment>
+<segment>
+<pinref part="WILDLY_RTC" gate="1" pin="1"/>
+<wire x1="-142.24" y1="5.08" x2="-147.32" y2="5.08" width="0.1524" layer="91"/>
+<label x="-147.32" y="5.08" size="1.778" layer="95"/>
+</segment>
+<segment>
+<label x="-127.508" y="5.334" size="1.778" layer="95" rot="R180"/>
+</segment>
 </net>
 <net name="NET_STAT" class="0">
@@
 <wire x1="215.9" y1="-17.78" x2="200.66" y2="-17.78" width="0.1524" layer="91"/>
 <label x="200.66" y="-17.78" size="1.778" layer="95"/>
-</segment>
-</net>
-<net name="FUEL_GAUGE_SDA" class="0">
-<segment>
-<pinref part="U$1" gate="G$1" pin="18/A4/PWM/T/SDA0"/>
-<wire x1="30.48" y1="40.64" x2="12.7" y2="40.64" width="0.1524" layer="91"/>
-<label x="2.54" y="40.64" size="1.778" layer="95"/>
-</segment>
-<segment>
-<pinref part="TEENSY_PIN_6" gate="A" pin="3"/>
-<wire x1="182.88" y1="-12.7" x2="167.64" y2="-12.7" width="0.1524" layer="91"/>
-<label x="154.94" y="-12.7" size="1.778" layer="95"/>
-</segment>
-<segment>
-<pinref part="J2" gate="G$1" pin="1"/>
-<wire x1="155.702" y1="140.716" x2="142.24" y2="140.716" width="0.1524" layer="91"/>
-<label x="131.826" y="140.716" size="1.778" layer="95"/>
-</segment>
-</net>
-<net name="FUEL_GAUGE_SCL" class="0">
-<segment>
-<pinref part="U$1" gate="G$1" pin="19/A5/PWM/T/SCL0"/>
-<wire x1="30.48" y1="38.1" x2="12.7" y2="38.1" width="0.1524" layer="91"/>
-<label x="2.54" y="38.1" size="1.778" layer="95"/>
-</segment>
-<segment>
-<pinref part="TEENSY_PIN_6" gate="A" pin="2"/>
-<wire x1="182.88" y1="-10.16" x2="167.64" y2="-10.16" width="0.1524" layer="91"/>
-<label x="154.94" y="-10.16" size="1.778" layer="95"/>
-</segment>
-<segment>
-<pinref part="J2" gate="G$1" pin="2"/>
-<wire x1="155.702" y1="138.176" x2="142.24" y2="138.176" width="0.1524" layer="91"/>
-<label x="131.826" y="138.176" size="1.778" layer="95"/>
 </segment>
 </net>
@@
 </segment>
 </net>
+<net name="SDA" class="0">
+<segment>
+<pinref part="WILDLY_RTC" gate="1" pin="4"/>
+<wire x1="-142.24" y1="12.7" x2="-147.32" y2="12.7" width="0.1524" layer="91"/>
+<label x="-147.32" y="12.7" size="1.778" layer="95"/>
+</segment>
+<segment>
+<pinref part="U$1" gate="G$1" pin="18/A4/PWM/T/SDA0"/>
+<wire x1="30.48" y1="40.64" x2="12.7" y2="40.64" width="0.1524" layer="91"/>
+<label x="2.54" y="40.64" size="1.778" layer="95"/>
+</segment>
+<segment>
+<pinref part="J2" gate="G$1" pin="1"/>
+<wire x1="155.702" y1="140.716" x2="142.24" y2="140.716" width="0.1524" layer="91"/>
+<label x="141.986" y="140.716" size="1.778" layer="95"/>
+</segment>
+<segment>
+<pinref part="TEENSY_PIN_6" gate="A" pin="3"/>
+<wire x1="182.88" y1="-12.7" x2="167.64" y2="-12.7" width="0.1524" layer="91"/>
+<label x="162.56" y="-12.7" size="1.778" layer="95"/>
+</segment>
+<segment>
+<label x="-130.556" y="11.938" size="1.778" layer="95"/>
+</segment>
+</net>
+<net name="SCL" class="0">
+<segment>
+<pinref part="WILDLY_RTC" gate="1" pin="3"/>
+<wire x1="-142.24" y1="10.16" x2="-147.32" y2="10.16" width="0.1524" layer="91"/>
+<label x="-147.32" y="10.16" size="1.778" layer="95"/>
+</segment>
+<segment>
+<pinref part="U$1" gate="G$1" pin="19/A5/PWM/T/SCL0"/>
+<wire x1="30.48" y1="38.1" x2="12.7" y2="38.1" width="0.1524" layer="91"/>
+<label x="2.54" y="38.1" size="1.778" layer="95"/>
+</segment>
+<segment>
+<pinref part="J2" gate="G$1" pin="2"/>
+<wire x1="155.702" y1="138.176" x2="142.24" y2="138.176" width="0.1524" layer="91"/>
+<label x="141.986" y="138.176" size="1.778" layer="95"/>
+</segment>
+<segment>
+<pinref part="TEENSY_PIN_6" gate="A" pin="2"/>
+<wire x1="182.88" y1="-10.16" x2="167.64" y2="-10.16" width="0.1524" layer="91"/>
+<label x="162.56" y="-10.16" size="1.778" layer="95"/>
+</segment>
+<segment>
+<label x="-125.222" y="10.668" size="1.778" layer="95" rot="R180"/>
+</segment>
+</net>
