File: PowerBoost - BASIC/Adafruit PowerBoost 1000 Basic.brd (EAGLE design)
At the start: 29.2 x 22.9 mm, 33 parts, among them CN1 USBA_FEMALE, T1 MMUN2133LT1G, U1 TPS61030RSAR, X2 3.5mm

Commit message: REmove Silkscreen and other placement issues in Powerboost basic
Parts:
- removed CN1: USBA_FEMALE, microbuilder:USB_HOST-PTH
- removed FID1, FID2, FID3: FIDUCIAL"", microbuilder:FIDUCIAL_1MM
- removed R10, R12: 49.9K 1%, microbuilder:0805-NO
- removed R11: 75K 1%, microbuilder:0805-NO
- removed R9: 43K 1%, microbuilder:0805-NO
- moved U$26 3.99 mm to (24.9, 13.5)
- moved U$25 3.86 mm to (24.9, 10.0)
- moved JP2 3.20 mm to (13.6, 21.5)
- moved LED1 0.52 mm to (3.90, 5.56)
- moved R3 0.40 mm to (10.8, 2.03)
- moved R13 0.25 mm to (10.0, 8.16)
- moved C1 0.13 mm to (11.8, 15.1)
- moved R4 0.13 mm to (10.0, 5.84)
Connections:
- removed net D+: CN1.D+, R11.1, R12.1
- removed net D-: CN1.D-, R10.1, R9.1
- net 5.0V: no longer CN1.VBUS, R11.2, R9.2
- net GND: no longer CN1.GND, R10.2, R12.2
Routing:
- net D+: track 12.7 -> 0.00 mm
- net 5.0V: track 29.7 -> 41.8 mm
- net D-: track 5.78 -> 0.00 mm
- net LBO: track 27.7 -> 31.1 mm
- net GND: track 8.02 -> 5.32 mm, vias 19 -> 0
- net N$2: track 2.01 -> 2.56 mm
Other:
- board text removed: "adafruit"
