File: PowerBoost - BASIC/Adafruit PowerBoost 1000 Basic.sch (EAGLE design)
At the start: 29 parts, among them CN1 USBA_FEMALE, T1 MMUN2133LT1G, U1 TPS61030RSAR, X2 3.5mm

Commit message: REmove Silkscreen and other placement issues in Powerboost basic
Parts:
- removed CN1: USBA_FEMALE, microbuilder:USB_TYPEAPTHFML
- removed FID1, FID2, FID3: FIDUCIAL"", microbuilder:FIDUCIAL""
- removed R10, R12: 49.9K 1%, microbuilder:RESISTOR0805_NOOUTLINE
- removed R11: 75K 1%, microbuilder:RESISTOR0805_NOOUTLINE
- removed R9: 43K 1%, microbuilder:RESISTOR0805_NOOUTLINE
Connections:
- removed net D+: CN1.D+, R11.1, R12.1
- removed net D-: CN1.D-, R10.1, R9.1
- net 5.0V: no longer CN1.VBUS, R11.2, R9.2
- net GND: no longer CN1.GND, R10.2, R12.2
Changed lines of the file:
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@@
 <?xml version="1.0" encoding="utf-8"?>
 <!DOCTYPE eagle SYSTEM "eagle.dtd">
-<eagle version="9.3.0">
+<eagle version="9.3.2">
 <drawing>
 <settings>
@@
 <part name="C2" library="microbuilder" deviceset="CAP_CERAMIC" device="0805-NOOUTLINE" value="2.2uF"/>
 <part name="U$7" library="microbuilder" deviceset="5.0V" device=""/>
-<part name="FID2" library="microbuilder" deviceset="FIDUCIAL" device="&quot;&quot;"/>
 <part name="X1" library="microbuilder" deviceset="TERMBLOCK_1X2" device=""/>
-<part name="R9" library="microbuilder" deviceset="RESISTOR" device="0805_NOOUTLINE" value="43K 1%"/>
-<part name="R10" library="microbuilder" deviceset="RESISTOR" device="0805_NOOUTLINE" value="49.9K 1%"/>
-<part name="R11" library="microbuilder" deviceset="RESISTOR" device="0805_NOOUTLINE" value="75K 1%"/>
-<part name="R12" library="microbuilder" deviceset="RESISTOR" device="0805_NOOUTLINE" value="49.9K 1%"/>
-<part name="CN1" library="microbuilder" deviceset="USB_TYPEA" device="PTHFML" value="USBA_FEMALE"/>
-<part name="U$15" library="microbuilder" deviceset="5.0V" device=""/>
-<part name="U$16" library="microbuilder" deviceset="5.0V" device=""/>
-<part name="U$17" library="microbuilder" deviceset="5.0V" device=""/>
 <part name="U$19" library="microbuilder" deviceset="VBAT" device=""/>
 <part name="LED1" library="microbuilder" deviceset="LED" device="0805_NOOUTLINE" value="RED"/>
@@
 <part name="U$9" library="microbuilder" deviceset="GND" device=""/>
 <part name="U$14" library="microbuilder" deviceset="GND" device=""/>
-<part name="U$18" library="microbuilder" deviceset="GND" device=""/>
-<part name="U$21" library="microbuilder" deviceset="GND" device=""/>
-<part name="U$22" library="microbuilder" deviceset="GND" device=""/>
 <part name="R2" library="microbuilder" deviceset="RESISTOR" device="_0805MP" value="340K"/>
 <part name="R1" library="microbuilder" deviceset="RESISTOR" device="_0805MP" value="1.87M"/>
@@
 <part name="C6" library="rcl" deviceset="C-US" device="C1210" value="100uF"/>
 <part name="X2" library="microbuilder" deviceset="TERMBLOCK_1X2" device="" value="3.5mm"/>
-<part name="FID1" library="microbuilder" deviceset="FIDUCIAL" device="&quot;&quot;">
-<attribute name="BOM" value="EXCLUDE"/>
-</part>
-<part name="FID3" library="microbuilder" deviceset="FIDUCIAL" device="&quot;&quot;">
-<attribute name="BOM" value="EXCLUDE"/>
-</part>
 <part name="JP2" library="microbuilder" deviceset="HEADER-1X8" device="ROUND"/>
 </parts>
@@
 <attribute name="VALUE" x="166.116" y="130.556" size="1.27" layer="96"/>
 </instance>
-<instance part="FID2" gate="G$1" x="246.38" y="43.18" smashed="yes"/>
 <instance part="X1" gate="G$1" x="182.88" y="106.68" smashed="yes" rot="MR180">
 <attribute name="VALUE" x="180.34" y="111.76" size="1.27" layer="96" rot="MR180"/>
 <attribute name="NAME" x="180.34" y="99.06" size="1.27" layer="95" rot="MR180"/>
 </instance>
-<instance part="R9" gate="G$1" x="231.14" y="109.22" smashed="yes">
-<attribute name="NAME" x="231.14" y="111.76" size="1.27" layer="95" font="vector" align="center"/>
-<attribute name="VALUE" x="231.14" y="109.22" size="1.016" layer="96" font="vector" ratio="15" align="center"/>
-</instance>
-<instance part="R10" gate="G$1" x="231.14" y="101.6" smashed="yes">
-<attribute name="NAME" x="231.14" y="104.14" size="1.27" layer="95" font="vector" align="center"/>
-<attribute name="VALUE" x="231.14" y="101.6" size="1.016" layer="96" font="vector" ratio="15" align="center"/>
-</instance>
-<instance part="R11" gate="G$1" x="231.14" y="88.9" smashed="yes">
-<attribute name="NAME" x="231.14" y="91.44" size="1.27" layer="95" font="vector" align="center"/>
-<attribute name="VALUE" x="231.14" y="88.9" size="1.016" layer="96" font="vector" ratio="15" align="center"/>
-</instance>
-<instance part="R12" gate="G$1" x="231.14" y="81.28" smashed="yes">
-<attribute name="NAME" x="231.14" y="83.82" size="1.27" layer="95" font="vector" align="center"/>
-<attribute name="VALUE" x="231.14" y="81.28" size="1.016" layer="96" font="vector" ratio="15" align="center"/>
-</instance>
-<instance part="CN1" gate="G$1" x="210.82" y="93.98" smashed="yes">
-<attribute name="NAME" x="200.66" y="102.616" size="1.27" layer="95"/>
-<attribute name="VALUE" x="200.66" y="83.82" size="1.27" layer="96"/>
-</instance>
-<instance part="U$15" gate="G$1" x="238.76" y="114.3" smashed="yes">
-<attribute name="VALUE" x="237.236" y="115.316" size="1.27" layer="96"/>
-</instance>
-<instance part="U$16" gate="G$1" x="238.76" y="93.98" smashed="yes">
-<attribute name="VALUE" x="237.236" y="94.996" size="1.27" layer="96"/>
-</instance>
-<instance part="U$17" gate="G$1" x="220.98" y="104.14" smashed="yes">
-<attribute name="VALUE" x="219.456" y="105.156" size="1.27" layer="96"/>
-</instance>
 <instance part="U$19" gate="G$1" x="81.28" y="111.76" smashed="yes">
 <attribute name="VALUE" x="79.756" y="112.776" size="1.27" layer="96"/>
@@
 <attribute name="VALUE" x="191.516" y="114.3" size="1.27" layer="96"/>
 </instance>
-<instance part="U$18" gate="G$1" x="238.76" y="99.06" smashed="yes">
-<attribute name="VALUE" x="237.236" y="96.52" size="1.27" layer="96"/>
-</instance>
-<instance part="U$21" gate="G$1" x="238.76" y="76.2" smashed="yes">
-<attribute name="VALUE" x="237.236" y="73.66" size="1.27" layer="96"/>
-</instance>
-<instance part="U$22" gate="G$1" x="220.98" y="83.82" smashed="yes">
-<attribute name="VALUE" x="219.456" y="81.28" size="1.27" layer="96"/>
-</instance>
 <instance part="R2" gate="G$1" x="96.52" y="73.66" smashed="yes" rot="R90">
 <attribute name="NAME" x="93.98" y="73.66" size="1.27" layer="95" font="vector" rot="R90" align="center"/>
@@
 <attribute name="NAME" x="53.34" y="86.36" size="1.27" layer="95" rot="R180"/>
 </instance>
-<instance part="FID1" gate="G$1" x="243.84" y="50.8" smashed="yes"/>
-<instance part="FID3" gate="G$1" x="233.68" y="53.34" smashed="yes"/>
 <instance part="JP2" gate="A" x="160.02" y="127" smashed="yes">
 <attribute name="NAME" x="153.67" y="140.335" size="1.778" layer="95"/>
@@
 <pinref part="LED2" gate="G$1" pin="C"/>
 <wire x1="190.5" y1="121.92" x2="193.04" y2="121.92" width="0.1524" layer="91"/>
-</segment>
-<segment>
-<pinref part="R10" gate="G$1" pin="2"/>
-<wire x1="236.22" y1="101.6" x2="238.76" y2="101.6" width="0.1524" layer="91"/>
-<pinref part="U$18" gate="G$1" pin="GND"/>
-</segment>
-<segment>
-<pinref part="R12" gate="G$1" pin="2"/>
-<wire x1="236.22" y1="81.28" x2="238.76" y2="81.28" width="0.1524" layer="91"/>
-<wire x1="238.76" y1="81.28" x2="238.76" y2="78.74" width="0.1524" layer="91"/>
-<pinref part="U$21" gate="G$1" pin="GND"/>
-</segment>
-<segment>
-<pinref part="CN1" gate="G$1" pin="GND"/>
-<wire x1="220.98" y1="88.9" x2="220.98" y2="86.36" width="0.1524" layer="91"/>
-<pinref part="U$22" gate="G$1" pin="GND"/>
 </segment>
 <segment>
@@
 </segment>
 <segment>
-<pinref part="R9" gate="G$1" pin="2"/>
-<pinref part="U$15" gate="G$1" pin="5.0V"/>
-<wire x1="236.22" y1="109.22" x2="238.76" y2="109.22" width="0.1524" layer="91"/>
-<wire x1="238.76" y1="109.22" x2="238.76" y2="111.76" width="0.1524" layer="91"/>
-</segment>
-<segment>
-<pinref part="R11" gate="G$1" pin="2"/>
-<pinref part="U$16" gate="G$1" pin="5.0V"/>
-<wire x1="236.22" y1="88.9" x2="238.76" y2="88.9" width="0.1524" layer="91"/>
-<wire x1="238.76" y1="88.9" x2="238.76" y2="91.44" width="0.1524" layer="91"/>
-</segment>
-<segment>
-<pinref part="CN1" gate="G$1" pin="VBUS"/>
-<pinref part="U$17" gate="G$1" pin="5.0V"/>
-<wire x1="220.98" y1="99.06" x2="220.98" y2="101.6" width="0.1524" layer="91"/>
-</segment>
-<segment>
 <pinref part="JP2" gate="A" pin="8"/>
 <wire x1="157.48" y1="119.38" x2="134.62" y2="119.38" width="0.1524" layer="91"/>
@@
 </segment>
 </net>
-<net name="D+" class="0">
-<segment>
-<wire x1="223.52" y1="88.9" x2="226.06" y2="88.9" width="0.1524" layer="91"/>
-<wire x1="220.98" y1="93.98" x2="223.52" y2="93.98" width="0.1524" layer="91"/>
-<wire x1="223.52" y1="93.98" x2="223.52" y2="88.9" width="0.1524" layer="91"/>
-<wire x1="223.52" y1="88.9" x2="223.52" y2="81.28" width="0.1524" layer="91"/>
-<wire x1="223.52" y1="81.28" x2="226.06" y2="81.28" width="0.1524" layer="91"/>
-<junction x="223.52" y="88.9"/>
-<pinref part="R11" gate="G$1" pin="1"/>
-<pinref part="R12" gate="G$1" pin="1"/>
-<pinref part="CN1" gate="G$1" pin="D+"/>
-</segment>
-</net>
-<net name="D-" class="0">
-<segment>
-<wire x1="223.52" y1="109.22" x2="226.06" y2="109.22" width="0.1524" layer="91"/>
-<wire x1="223.52" y1="101.6" x2="226.06" y2="101.6" width="0.1524" layer="91"/>
-<wire x1="223.52" y1="101.6" x2="223.52" y2="109.22" width="0.1524" layer="91"/>
-<wire x1="220.98" y1="96.52" x2="223.52" y2="96.52" width="0.1524" layer="91"/>
-<wire x1="223.52" y1="96.52" x2="223.52" y2="101.6" width="0.1524" layer="91"/>
-<junction x="223.52" y="101.6"/>
-<pinref part="R9" gate="G$1" pin="1"/>
-<pinref part="R10" gate="G$1" pin="1"/>
-<pinref part="CN1" gate="G$1" pin="D-"/>
-</segment>
-</net>
