File: Wildly_Multi_Lipo_Charger/Wildly_4Lipo_Charge.sch (EAGLE design)
At the start: 61 parts, among them CN1 JSTPH, CN2 JSTPH, CN3 JSTPH, CN4 JSTPH, CN5 DCIN, U1 MCP73831T-2ACI/OT, U2 MCP73831T-2ACI/OT, U3 MCP73831T-2ACI/OT, U4 MCP73831T-2ACI/OT

Commit message: Remove gorund plane and connect grounds directly, add reverse current protection, add jumpers to isolate individual batteries and main power if needed
Parts:
- added D2, D3, D4, D5: MBR120VLSFT1G, microbuilder:DIODESOD-123
- added JP5, JP6, JP7, JP8: (no value), jumper:JP1Q
Connections:
- new net N$10: D3.C, JP7.2, JP8.1, R3.1
- new net N$15: D2.A, X2.VBUS
- new net N$20: C1.+, C2.1, D5.C, DCIN_6V.2, JP5.1
- new net N$22: D3.A, X3.VBUS
- new net N$23: D2.C, JP6.2, JP7.1, R2.1
- new net N$24: D4.A, X4.VBUS
- new net N$27: D4.C, JP8.2, R4.1
- new net N$3: D1.A, X1.VBUS
- net N$21: now also D5.A; no longer D1.A
- net VCC: now also JP5.2, JP6.1; no longer C1.+, C2.1, DCIN_6V.2, R2.1, R3.1, R4.1, X1.VBUS, X2.VBUS, X3.VBUS, X4.VBUS
Other:
- moved on the sheet: C1, C11, C2, C21, C31, C41, CN5, D1, DCIN_6V, JP1, JP2, JP3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

Commit message: Remove jupers and place diode appropriately to prevent reverse current, remove ground looping
Parts:
- removed D5: MBR120VLSFT1G, microbuilder:DIODESOD-123
- removed JP5, JP6, JP7, JP8: (no value), jumper:JP1Q
- added D6: MBR120VLSFT1G, microbuilder:DIODESOD-123
Connections:
- removed net N$15: D2.A, X2.VBUS
- removed net N$20: C1.+, C2.1, D5.C, DCIN_6V.2, JP5.1
- removed net N$22: D3.A, X3.VBUS
- removed net N$23: D2.C, JP6.2, JP7.1, R2.1
- removed net N$24: D4.A, X4.VBUS
- removed net N$3: D1.A, X1.VBUS
- new net N$25: D2.C, R2.1, X2.VBUS
- new net N$26: D1.C, R1.1, X1.VBUS
- net N$10: now also X3.VBUS; no longer JP7.2, JP8.1
- net N$21: now also C1.+, C2.1, D6.A, DCIN_6V.2; no longer D5.A
- net N$27: now also X4.VBUS; no longer JP8.2
- net VCC: now also D1.A, D2.A, D3.A, D4.A, D6.C; no longer D1.C, JP5.2, JP6.1, R1.1
Other:
- moved on the sheet: D1, D2, D3, D4
