File: Wildly_Multi_Lipo_Charger/Wildly_4Lipo_Charge.brd (EAGLE design)
At the start: 81 x 44.4 mm, 61 parts, among them CN1 JSTPH, CN2 JSTPH, CN3 JSTPH, CN4 JSTPH, CN5 DCIN, U1 MCP73831T-2ACI/OT, U2 MCP73831T-2ACI/OT, U3 MCP73831T-2ACI/OT, U4 MCP73831T-2ACI/OT

Commit message: Remove gorund plane and connect grounds directly, add reverse current protection, add jumpers to isolate individual batteries and main power if needed
Parts:
- added D2, D3, D4, D5: MBR120VLSFT1G, microbuilder:SOD-123
- added JP5, JP6, JP7, JP8: (no value), jumper:JP1
- moved D1 18.3 mm to (34.3, 8.89), turned to 0 degrees
- moved JP3 5.24 mm to (69.8, 14.0)
- moved JP1 5.24 mm to (36.8, 14.0)
- moved JP2 5.24 mm to (53.3, 14.0)
- moved JP4 5.24 mm to (86.4, 14.0)
- moved C2 3.59 mm to (22.9, 22.9)
- moved X1 2.54 mm to (38.1, 2.54)
- moved X2 2.54 mm to (54.6, 2.54)
- moved X3 2.54 mm to (71.1, 2.54)
- moved X4 2.54 mm to (87.6, 2.54)
- moved JP11 2.54 mm to (38.1, 19.1)
- moved JP22 2.54 mm to (54.6, 19.1)
- moved JP33 2.54 mm to (71.1, 19.1)
- moved JP44 2.54 mm to (87.6, 19.1)
- moved C1 1.27 mm to (22.9, 31.8)
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Connections:
- new net N$10: D3.C, JP7.2, JP8.1, R3.1
- new net N$15: D2.A, X2.VBUS
- new net N$20: C1.+, C2.1, D5.C, DCIN_6V.2, JP5.1
- new net N$22: D3.A, X3.VBUS
- new net N$23: D2.C, JP6.2, JP7.1, R2.1
- new net N$24: D4.A, X4.VBUS
- new net N$27: D4.C, JP8.2, R4.1
- new net N$3: D1.A, X1.VBUS
- net N$21: now also D5.A; no longer D1.A
- net VCC: now also JP5.2, JP6.1; no longer C1.+, C2.1, DCIN_6V.2, R2.1, R3.1, R4.1, X1.VBUS, X2.VBUS, X3.VBUS, X4.VBUS
Routing:
- net GND: track 0.00 -> 500.3 mm, vias 0 -> 13
- net VCC: track 119.0 -> 31.2 mm
- net N$20: track 0.00 -> 29.6 mm
- net N$10: track 0.00 -> 24.5 mm
- net N$23: track 0.00 -> 21.4 mm
- net N$27: track 0.00 -> 10.3 mm
- net N$3: track 0.00 -> 2.44 mm
- net N$24: track 0.00 -> 2.44 mm
- net N$22: track 0.00 -> 2.44 mm
- net N$15: track 0.00 -> 2.44 mm
- net N$7: track 22.2 -> 19.8 mm
- net N$17: track 21.6 -> 19.9 mm
- net N$9: track 3.08 -> 1.81 mm
- net N$6: track 3.08 -> 1.81 mm
- net N$4: track 3.08 -> 1.81 mm
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- removed copper zone on layer 1, net GND
Other:
- board size 81 x 44.4 mm -> 81 x 47 mm

Commit message: Remove jupers and place diode appropriately to prevent reverse current, remove ground looping
Parts:
- removed D5: MBR120VLSFT1G, microbuilder:SOD-123
- removed JP5, JP6, JP7, JP8: (no value), jumper:JP1
- added D6: MBR120VLSFT1G, microbuilder:SOD-123
- moved JP3 5.24 mm to (74.9, 12.7)
- moved JP1 5.24 mm to (41.9, 12.7)
- moved JP2 5.24 mm to (58.4, 12.7)
- moved JP4 5.24 mm to (91.4, 12.7)
- moved D1 4.02 mm to (35.6, 12.7)
- moved D2 3.81 mm to (50.8, 12.7)
- moved D3 3.81 mm to (67.3, 12.7)
- moved D4 3.81 mm to (83.8, 12.7)
Connections:
- removed net N$15: D2.A, X2.VBUS
- removed net N$20: C1.+, C2.1, D5.C, DCIN_6V.2, JP5.1
- removed net N$22: D3.A, X3.VBUS
- removed net N$23: D2.C, JP6.2, JP7.1, R2.1
- removed net N$24: D4.A, X4.VBUS
- removed net N$3: D1.A, X1.VBUS
- new net N$25: D2.C, R2.1, X2.VBUS
- new net N$26: D1.C, R1.1, X1.VBUS
- net N$10: now also X3.VBUS; no longer JP7.2, JP8.1
- net N$21: now also C1.+, C2.1, D6.A, DCIN_6V.2; no longer D5.A
- net N$27: now also X4.VBUS; no longer JP8.2
- net VCC: now also D1.A, D2.A, D3.A, D4.A, D6.C; no longer D1.C, JP5.2, JP6.1, R1.1
Routing:
- net VCC: track 31.2 -> 85.1 mm, vias 0 -> 5
- net N$20: track 29.6 -> 0.00 mm
- net N$21: track 2.81 -> 31.6 mm
- net GND: track 500.3 -> 478.1 mm, vias 13 -> 8
- net N$23: track 21.4 -> 0.00 mm
- net N$25: track 0.00 -> 13.4 mm
- net N$26: track 0.00 -> 11.5 mm
- net N$10: track 24.5 -> 13.4 mm
- net N$27: track 10.3 -> 13.4 mm
- net N$3: track 2.44 -> 0.00 mm
- net N$24: track 2.44 -> 0.00 mm
- net N$22: track 2.44 -> 0.00 mm
- net N$15: track 2.44 -> 0.00 mm
- net VDD2: track 17.3 -> 16.3 mm
- net VDD1: track 17.3 -> 16.3 mm
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Other:
- board text added: "+"
- board text added: "-"

Commit message: Remove ground routing from under the diode, remove more ground looping near battery connectors
Routing:
- net GND: track 478.1 -> 400.4 mm
- net VCC: track 85.1 -> 87.0 mm
Changed lines of the file:
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@@
 <drawing>
 <settings>
-<setting alwaysvectorfont="yes"/>
+<setting alwaysvectorfont="no"/>
 <setting verticaltext="up"/>
 </settings>
@@
 <wire x1="25.4" y1="3.81" x2="24.98" y2="3.39" width="1.2192" layer="1"/>
 <wire x1="24.13" y1="41.91" x2="25.4" y2="40.64" width="1.2192" layer="1"/>
-<wire x1="25.4" y1="40.64" x2="25.4" y2="36.83" width="1.2192" layer="1"/>
-<wire x1="25.4" y1="36.83" x2="25.4" y2="31.75" width="1.2192" layer="1"/>
+<wire x1="25.4" y1="40.64" x2="25.4" y2="35.56" width="1.2192" layer="1"/>
+<wire x1="25.4" y1="35.56" x2="25.4" y2="31.75" width="1.2192" layer="1"/>
 <wire x1="23.86" y1="22.86" x2="25.4" y2="24.4" width="1.2192" layer="1"/>
 <wire x1="25.4" y1="24.4" x2="25.4" y2="31.75" width="1.2192" layer="1"/>
@@
 <wire x1="25.25" y1="0.15" x2="25.4" y2="0" width="1.2192" layer="1"/>
 <wire x1="25.4" y1="0" x2="25.94" y2="0.54" width="1.2192" layer="1"/>
-<wire x1="25.94" y1="0.54" x2="33.7" y2="0.54" width="1.2192" layer="1"/>
+<wire x1="25.94" y1="0.54" x2="31.75" y2="0.54" width="1.2192" layer="1"/>
+<wire x1="31.75" y1="0.54" x2="33.7" y2="0.54" width="1.2192" layer="1"/>
 <wire x1="42.5" y1="0.54" x2="50.21" y2="0.54" width="1.2192" layer="1"/>
 <wire x1="59.01" y1="0.54" x2="66.77" y2="0.54" width="1.2192" layer="1"/>
@@
 <wire x1="75.52" y1="0.54" x2="83.23" y2="0.54" width="1.2192" layer="1"/>
 <wire x1="38.1" y1="21.81" x2="38.1" y2="20.7528" width="0.6096" layer="1"/>
-<wire x1="34.56" y1="36.94" x2="35.6028" y2="37.9828" width="0.6096" layer="1"/>
-<wire x1="35.6028" y1="37.9828" x2="35.6028" y2="39.42938125" width="0.6096" layer="1"/>
-<wire x1="35.6028" y1="39.42938125" x2="35.87061875" y2="39.6972" width="0.6096" layer="1"/>
-<wire x1="35.87061875" y1="39.6972" x2="37.24938125" y2="39.6972" width="0.6096" layer="1"/>
-<wire x1="37.57658125" y1="39.37" x2="50.8" y2="39.37" width="0.6096" layer="1"/>
-<wire x1="37.24938125" y1="39.6972" x2="37.57658125" y2="39.37" width="0.6096" layer="1"/>
-<wire x1="50.8" y1="39.37" x2="50.8" y2="37.21" width="0.6096" layer="1"/>
-<wire x1="50.8" y1="37.21" x2="51.07" y2="36.94" width="0.6096" layer="1"/>
-<wire x1="52.38061875" y1="39.6972" x2="53.75938125" y2="39.6972" width="0.6096" layer="1"/>
-<wire x1="50.8" y1="39.37" x2="52.05341875" y2="39.37" width="0.6096" layer="1"/>
-<wire x1="54.08658125" y1="39.37" x2="68.58" y2="39.37" width="0.6096" layer="1"/>
-<wire x1="52.05341875" y1="39.37" x2="52.38061875" y2="39.6972" width="0.6096" layer="1"/>
-<wire x1="53.75938125" y1="39.6972" x2="54.08658125" y2="39.37" width="0.6096" layer="1"/>
-<wire x1="68.58" y1="39.37" x2="68.85" y2="39.1" width="0.6096" layer="1"/>
-<wire x1="68.85" y1="39.1" x2="68.85" y2="36.94" width="0.6096" layer="1"/>
-<wire x1="70.16061875" y1="39.6972" x2="71.53938125" y2="39.6972" width="0.6096" layer="1"/>
-<wire x1="68.58" y1="39.37" x2="69.83341875" y2="39.37" width="0.6096" layer="1"/>
-<wire x1="71.86658125" y1="39.37" x2="85.09" y2="39.37" width="0.6096" layer="1"/>
-<wire x1="69.83341875" y1="39.37" x2="70.16061875" y2="39.6972" width="0.6096" layer="1"/>
-<wire x1="71.53938125" y1="39.6972" x2="71.86658125" y2="39.37" width="0.6096" layer="1"/>
-<wire x1="85.09" y1="39.37" x2="85.09" y2="38.1" width="0.6096" layer="1"/>
 <wire x1="85.09" y1="38.1" x2="85.36" y2="37.83" width="0.6096" layer="1"/>
 <wire x1="85.36" y1="37.83" x2="85.36" y2="36.94" width="0.6096" layer="1"/>
-<wire x1="26.0756" y1="9.93614375" x2="26.0756" y2="7.84385625" width="1.2192" layer="1"/>
-<wire x1="26.0756" y1="7.84385625" x2="24.59614375" y2="6.3644" width="1.2192" layer="1"/>
-<wire x1="24.13" y1="41.91" x2="24.13" y2="16.54763125" width="1.2192" layer="1"/>
-<wire x1="22.0244" y1="6.3644" x2="19.05" y2="3.39" width="1.2192" layer="1"/>
-<wire x1="24.13" y1="16.54763125" x2="23.288" y2="15.70563125" width="1.2192" layer="1"/>
-<wire x1="24.59614375" y1="6.3644" x2="22.0244" y2="6.3644" width="1.2192" layer="1"/>
-<wire x1="23.288" y1="15.70563125" x2="23.288" y2="12.72374375" width="1.2192" layer="1"/>
-<wire x1="23.288" y1="12.72374375" x2="26.0756" y2="9.93614375" width="1.2192" layer="1"/>
 <wire x1="42.86" y1="15.24" x2="42.86" y2="13.02" width="0.9144" layer="1"/>
 <wire x1="42.86" y1="13.02" x2="43.18" y2="12.7" width="0.9144" layer="1"/>
@@
 <wire x1="92.39" y1="15.24" x2="92.39" y2="13.02" width="0.9144" layer="1"/>
 <wire x1="92.39" y1="13.02" x2="92.71" y2="12.7" width="0.9144" layer="1"/>
-<wire x1="34.29" y1="33.02" x2="29.21" y2="33.02" width="0.6096" layer="1"/>
-<wire x1="29.21" y1="33.02" x2="25.4" y2="36.83" width="0.6096" layer="1"/>
 <wire x1="39.7" y1="6.604" x2="39.7" y2="9.22" width="0.6096" layer="1"/>
 <wire x1="39.7" y1="9.22" x2="43.18" y2="12.7" width="0.6096" layer="1"/>
@@
 <wire x1="88.9" y1="20.32" x2="89.535" y2="20.32" width="0.6096" layer="16"/>
 <wire x1="89.535" y1="20.32" x2="91.44" y2="22.225" width="0.6096" layer="16"/>
+<wire x1="31.75" y1="16.9642125" x2="25.8542125" y2="22.86" width="0.9144" layer="1"/>
+<wire x1="23.86" y1="22.86" x2="25.8542125" y2="22.86" width="0.9144" layer="1"/>
+<wire x1="31.75" y1="16.9642125" x2="31.75" y2="0.54" width="0.9144" layer="1"/>
+<wire x1="25.4" y1="35.56" x2="27.94" y2="33.02" width="0.9144" layer="1"/>
+<wire x1="27.94" y1="33.02" x2="34.29" y2="33.02" width="0.9144" layer="1"/>
 <wire x1="68.58" y1="30.43789375" x2="68.9" y2="30.48" width="0" layer="19" extent="1-1"/>
+<wire x1="72.7796" y1="6.604" x2="72.72" y2="6.604" width="0" layer="19" extent="1-1"/>
+<wire x1="75.52" y1="0.54" x2="75.52" y2="6.04" width="0" layer="19" extent="1-1"/>
 <wire x1="38.1" y1="21.81" x2="38.1" y2="21.84789375" width="0" layer="19" extent="1-1"/>
-<wire x1="72.7796" y1="6.604" x2="72.72" y2="6.604" width="0" layer="19" extent="1-1"/>
-<wire x1="89.442" y1="6.604" x2="89.23" y2="6.604" width="0" layer="19" extent="1-1"/>
-<wire x1="56.422" y1="6.604" x2="56.21" y2="6.604" width="0" layer="19" extent="1-1"/>
 <wire x1="39.912" y1="6.604" x2="39.7" y2="6.604" width="0" layer="19" extent="1-1"/>
-<wire x1="25.25" y1="3.39" x2="24.98" y2="3.39" width="0" layer="19" extent="1-1"/>
+<wire x1="24.98" y1="3.39" x2="25.25" y2="3.39" width="0" layer="19" extent="1-1"/>
 <wire x1="34.61" y1="30.48" x2="34.29" y2="29.88210625" width="0" layer="19" extent="1-1"/>
+<wire x1="92.03" y1="6.04" x2="92.03" y2="0.54" width="0" layer="19" extent="1-1"/>
+<wire x1="89.23" y1="6.604" x2="89.442" y2="6.604" width="0" layer="19" extent="1-1"/>
+<wire x1="59.01" y1="6.04" x2="59.01" y2="0.54" width="0" layer="19" extent="1-1"/>
+<wire x1="56.21" y1="6.604" x2="56.422" y2="6.604" width="0" layer="19" extent="1-1"/>
 </signal>
 <signal name="N$1">
@@
 <contactref element="D4" pad="A"/>
 <contactref element="D6" pad="C"/>
-<wire x1="25.98" y1="17.78" x2="31.75" y2="12.01" width="1.2192" layer="1"/>
-<wire x1="31.75" y1="12.01" x2="31.75" y2="8.89" width="1.2192" layer="1"/>
-<via x="31.75" y="8.89" extent="1-16" drill="0.7818"/>
-<wire x1="31.75" y1="8.89" x2="38.1" y2="8.89" width="1.2192" layer="16"/>
 <wire x1="38.1" y1="8.89" x2="54.61" y2="8.89" width="1.2192" layer="16"/>
 <wire x1="54.61" y1="8.89" x2="71.12" y2="8.89" width="1.2192" layer="16"/>
@@
 <wire x1="85.67" y1="12.7" x2="87.63" y2="10.74" width="1.2192" layer="1"/>
 <wire x1="87.63" y1="10.74" x2="87.63" y2="8.89" width="1.2192" layer="1"/>
+<wire x1="38.1" y1="8.89" x2="29.845" y2="8.89" width="1.2192" layer="16"/>
+<via x="29.845" y="8.89" extent="1-16" drill="0.762"/>
+<wire x1="25.98" y1="17.78" x2="27.885" y2="15.875" width="1.2192" layer="1"/>
+<wire x1="27.885" y1="15.875" x2="29.21" y2="15.875" width="1.2192" layer="1"/>
+<wire x1="29.21" y1="15.875" x2="29.845" y2="15.24" width="1.2192" layer="1"/>
+<wire x1="29.845" y1="15.24" x2="29.845" y2="8.89" width="1.2192" layer="1"/>
 </signal>
 <signal name="N$21">
